File: mct2/mct2.kicad_sch (KiCad schematic)
At the start: 3 parts, among them J1 Bus_M.2_Socket_M, U1 TUSB7340

Commit message: July 7 2024
Parts:
- added C1: 470nF, symbol Device:C_Small
- added J2: Bus_M.2_Socket_E, symbol Connector:Bus_M.2_Socket_E
- added J3: Screw_Terminal_01x02, symbol Connector:Screw_Terminal_01x02
- added R1: 50m, symbol Device:R_Small
- added U2: BQ25700A, symbol mediacow:BQ25700A
- added U3: LTC2959, symbol mediacow:LTC2959
Connections:
- net GND: now also J3.1 (Pin_1)
- new net: J3.2 (Pin_2), R1.2, U3.5 (SENSEN)
- new net: R1.1, U3.2 (SENSEP)
- new net: C1.1, U3.3 (CFP)
- new net: C1.2, U3.4 (CFN)
- new net: J2.1 (GND), J2.18 (GND), J2.33 (GND), J2.39 (GND), J2.45 (GND), J2.51 (GND), J2.57 (GND), J2.63 (GND), J2.69 (GND), J2.7 (GND), J2.75 (GND)
- new net: J2.2 (3.3V), J2.4 (3.3V), J2.72 (3.3V), J2.74 (3.3V)
- new net SMB_SCL: U3.6 (SCL)
- new net SMB_SDA: U3.7 (SDA)
Other:
- moved on the sheet: J1

Commit message: block diagram and schematic update
Parts:
- removed C1: 470nF, symbol Device:C_Small
- removed J3: Screw_Terminal_01x02, symbol Connector:Screw_Terminal_01x02
- removed R1: 50m, symbol Device:R_Small
- removed U1: TUSB7340, Package_DFN_QFN:Texas_S-PWQFN-N100_EP5.5x5.5mm_ThermalVias, symbol Interface_USB:TUSB7340
- removed U3: LTC2959, symbol mediacow:LTC2959
- renumbered U2 to U1
Connections:
- net PROCHOT: now also U1.11 (PROCHOT)
Other:
- added sheet mct2_io (mct2_io.kicad_sch)
