File: mct2/mct2_io.kicad_sch (KiCad schematic)
At the start: 12 parts, among them J4 USB3_A_Stacked, J5 USB3_A_Stacked, J6 USB_A_Stacked, U1 TUSB7340, U4 TPS25221, U5 TPS25221, U6 TPS25221, U7 TPS25221

Commit message: figuring out USB3
Parts:
- removed R3, R4, R5: 80K, symbol Device:R_Small
- removed U5: TPS25221, symbol mediacow:TPS25221
- added C1, C2: 100nF, symbol Device:C_Small
- added LF1, LF2: ECMF2-40A100N6, symbol mediacow:ECMF2-40A100N6
- added R1: 9.09K 1%, symbol Device:R_Small
- added R6, R7: 80K, symbol Device:R_Small
- added U8: TPD2EUSB30, Package_TO_SOT_SMD:Texas_DRT-3, symbol Power_Protection:TPD2EUSB30
- renumbered U4 to U2
Connections:
- net XHCI_PCIE_REF_N is gone; now on net XHCI_PCIE_RX_N: U1.B41 (PCIE_REFCLKN)
- net XHCI_PCIE_REF_P is gone; now on net XHCI_PCIE_RX_P: U1.A45 (PCIE_REFCLKP)
- net GND: now also LF1.3 (GND), LF1.4 (GND), LF2.3 (GND), LF2.4 (GND), R6.2, R7.2, U8.3 (GND); no longer U6.2 (GND), U7.2 (GND)
- net USB_5V: no longer U6.1 (IN), U7.1 (IN)
- net at J6.1 (VBUS1): now also U6.6 (OUT)
- net at J6.5 (VBUS2): now also U7.6 (OUT)
- net at J5.10 (VBUS2): no longer U7.6 (OUT)
- net at U7.5 (ILIM): now also R7.1
- net at U1.A24 (R1EXT): now also R1.2
- net at U1.B23 (R1EXTRTN): now also R1.1
- net at J5.1 (VBUS1): no longer U6.6 (OUT)
- net at U6.5 (ILIM): now also R6.1
- net USBSS1_DN: no longer names the net of J4.2 (D1-)
- net USBSS1_DN: now also LF1.1; no longer U1.B18 (USB_DM_DN1)
- net USBSS1_DP: no longer names the net of J4.3 (D1+)
- net USBSS1_DP: now also LF1.2; no longer U1.A20 (USB_DP_DN1)
- net USBSS1_EN: no longer names the net of U1.B33 (PWRON1#)
- net USBSS1_EN: no longer U2.3 (EN)
- net USBSS1_OC: no longer names the net of U1.A36 (OVERCUR1#)
- net USBSS1_OC: no longer U2.4 (FAULT)
- net USBSS1_SSRXN renamed EUSBSS1_SSRXN
- net EUSBSS1_SSRXN: now also U8.2 (D-)
- net USBSS1_SSRXP renamed EUSBSS1_SSRXP
- net EUSBSS1_SSRXP: now also U8.1 (D+)
- net USBSS1_SSTXN: no longer names the net of J4.8 (SSTX1-)
- net USBSS1_SSTXN: now also LF2.1; no longer U1.B15 (USB_SSTXN_DN1)
- net USBSS1_SSTXP: no longer names the net of J4.9 (SSTX1+)
- net USBSS1_SSTXP: now also LF2.2; no longer U1.A17 (USB_SSTXP_DN1)
- net USBSS2_DN: no longer names the net of J4.11 (D2-)
- net USBSS2_DN: no longer U1.A13 (USB_DM_DN2)
- net USBSS2_DP: no longer names the net of J4.12 (D2+)
- net USBSS2_DP: no longer U1.B12 (USB_DP_DN2)
- net USBSS2_EN: no longer names the net of U1.B34 (PWRON2#)
- net USBSS2_OC: no longer names the net of U1.A37 (OVERCUR2#)
- net USBSS2_SSRXN: no longer names the net of J4.14 (SSRX2-)
- net USBSS2_SSRXN: no longer U1.A10 (USB_SSRXN_DN2)
- net USBSS2_SSRXP: no longer names the net of J4.15 (SSRX2+)
- net USBSS2_SSRXP: no longer U1.B9 (USB_SSRXP_DN2)
- net USBSS2_SSTXN: no longer names the net of J4.17 (SSTX2-)
- net USBSS2_SSTXN: no longer U1.B10 (USB_SSTXN_DN2)
- net USBSS2_SSTXP: no longer names the net of J4.18 (SSTX2+)
- net USBSS2_SSTXP: no longer U1.A11 (USB_SSTXP_DN2)
- net USBSS3_DN: no longer names the net of J5.2 (D1-)
- net USBSS3_DN: no longer U1.A27 (USB_DM_DN3)
- net USBSS3_DP: no longer names the net of J5.3 (D1+)
- net USBSS3_DP: no longer U1.B25 (USB_DP_DN3)
- net USBSS3_EN: no longer names the net of U1.A46 (PWRON3#)
- net USBSS3_EN: no longer U6.3 (EN)
- net USBSS3_OC: no longer names the net of U1.B43 (OVERCUR3#)
- net USBSS3_OC: no longer U6.4 (FAULT)
- net USBSS3_SSRXN: no longer names the net of J5.5 (SSRX1-)
- net USBSS3_SSRXN: no longer U1.A29 (USB_SSRXN_DN3)
- net USBSS3_SSRXP: no longer names the net of J5.6 (SSRX1+)
- net USBSS3_SSRXP: no longer U1.B27 (USB_SSRXP_DN3)
- net USBSS3_SSTXN: no longer names the net of J5.8 (SSTX1-)
- net USBSS3_SSTXN: no longer U1.A30 (USB_SSTXN_DN3)
- net USBSS3_SSTXP: no longer names the net of J5.9 (SSTX1+)
- net USBSS3_SSTXP: no longer U1.B28 (USB_SSTXP_DN3)
- net USBSS4_DN: no longer names the net of J5.11 (D2-)
- net USBSS4_DN: no longer U1.A5 (USB_DM_DN4)
- net USBSS4_DP: no longer names the net of J5.12 (D2+)
- net USBSS4_DP: no longer U1.B5 (USB_DP_DN4)
- net USBSS4_EN: no longer names the net of U7.3 (EN)
- net USBSS4_EN: no longer U1.A48 (PWRON4#)
- net USBSS4_OC: no longer names the net of U7.4 (FAULT)
- net USBSS4_OC: no longer U1.B45 (OVERCUR4#)
- net USBSS4_SSRXN: no longer names the net of J5.14 (SSRX2-)
- net USBSS4_SSRXN: no longer U1.A7 (USB_SSRXN_DN4)
- net USBSS4_SSRXP: no longer names the net of J5.15 (SSRX2+)
- net USBSS4_SSRXP: no longer U1.B6 (USB_SSRXP_DN4)
- net USBSS4_SSTXN: no longer names the net of J5.17 (SSTX2-)
- net USBSS4_SSTXN: no longer U1.A8 (USB_SSTXN_DN4)
- net USBSS4_SSTXP: no longer names the net of J5.18 (SSTX2+)
- net USBSS4_SSTXP: no longer U1.B7 (USB_SSTXP_DN4)
- new net: C2.2, LF2.5
- new net: C1.2, LF2.6
- new net EUSBSS1_DN: LF1.6, U1.B18 (USB_DM_DN1)
- new net EUSBSS1_DP: LF1.5, U1.A20 (USB_DP_DN1)
- new net EUSBSS1_EN: U2.3 (EN)
- new net EUSBSS1_OC: U2.4 (FAULT)
- new net EUSBSS1_SSTXN: C1.1, U1.B15 (USB_SSTXN_DN1)
- new net EUSBSS1_SSTXP: C2.1, U1.A17 (USB_SSTXP_DN1)
- new net EUSBSS2_DN: U1.A13 (USB_DM_DN2)
- new net EUSBSS2_DP: U1.B12 (USB_DP_DN2)
- new net EUSBSS2_SSRXN: U1.A10 (USB_SSRXN_DN2)
- new net EUSBSS2_SSRXP: U1.B9 (USB_SSRXP_DN2)
- new net EUSBSS2_SSTXN: U1.B10 (USB_SSTXN_DN2)
- new net EUSBSS2_SSTXP: U1.A11 (USB_SSTXP_DN2)
- new net EUSBSS3_DN: U1.A27 (USB_DM_DN3)
- new net EUSBSS3_DP: U1.B25 (USB_DP_DN3)
- new net EUSBSS3_SSRXN: U1.A29 (USB_SSRXN_DN3)
- new net EUSBSS3_SSRXP: U1.B27 (USB_SSRXP_DN3)
- new net EUSBSS3_SSTXN: U1.A30 (USB_SSTXN_DN3)
- new net EUSBSS3_SSTXP: U1.B28 (USB_SSTXP_DN3)
- new net EUSBSS4_DN: U1.A5 (USB_DM_DN4)
- new net EUSBSS4_DP: U1.B5 (USB_DP_DN4)
- new net EUSBSS4_SSRXN: U1.A7 (USB_SSRXN_DN4)
- new net EUSBSS4_SSRXP: U1.B6 (USB_SSRXP_DN4)
- new net EUSBSS4_SSTXN: U1.A8 (USB_SSTXN_DN4)
- new net EUSBSS4_SSTXP: U1.B7 (USB_SSTXP_DN4)
Other:
- moved on the sheet: J4A, J4B, J5A, J5B, J6, R2, U2
