File: circuits/mct2/mct2_power.kicad_sch (KiCad schematic)
At the start: 7 parts, among them J3 USB_C_Receptacle, J4 USB_C_Receptacle, U1 BQ25700A, U2 CYPD4225-40LQXI, U3 STM32L4A6RGTx, U4 TPD4EUSB30

Commit message: July 21, 2024
Parts:
- removed U2: CYPD4225-40LQXI, symbol mediacow:CYPD4225-40LQXIT
- removed U3: STM32L4A6RGTx, Package_QFP:LQFP-64_10x10mm_P0.5mm, symbol MCU_ST_STM32L4:STM32L4A6RGTx
- removed U4: TPD4EUSB30, Package_SON:USON-10_2.5x1.0mm_P0.5mm, symbol Power_Protection:TPD4EUSB30
- added C10, C11, C12, C13, C14, C15, C16, C2, C3, C4, C5, C6, C7, C8, C9: 220nF, Capacitor_SMD:C_0603_1608Metric, symbol Device:C_Small
- added C? (x2): 100nF, symbol Device:C_Small
- added C? (x2): 1uF, symbol Device:C_Small
- added R? (x2): 100K, symbol Device:R_Small
- added U4, U5, U6, U7: TPD4EUSB30, Package_SON:USON-10_2.5x1.0mm_P0.5mm, symbol mediacow:TPD4EUSB30
- added U9, U?: TPD6S300A, Package_DFN_QFN:WQFN-20-1EP_3x3mm_P0.4mm_EP1.7x1.7mm_ThermalVias, symbol Power_Protection:TPD6S300A
Connections:
- net TCP0_CC1: now also U?.4 (C_CC1); no longer J3.A5 (CC1)
- net TCP0_CC2: now also U?.5 (C_CC2); no longer J3.B5 (CC2)
- net TCP0_DN: now also U?.19 (D2)
- net TCP0_DP: now also U?.20 (D1)
- net TCP0_SBU1: now also U?.1 (C_SBU1); no longer J3.A8 (SBU1)
- net TCP0_SBU2: now also U?.2 (C_SBU2); no longer J3.B8 (SBU2)
- net TCP0_SSTX0_N: now also C6.1, U5.2 (D1-)
- net TCP0_SSTX0_P: now also C5.1, U5.1 (D1+)
- net TCP0_SSTX1_N: now also C2.1, U4.2 (D1-)
- net TCP0_SSTX1_P: now also C1.1, U4.1 (D1+)
- net TCP0_SSTXRX0_N: now also C8.1, U5.4 (D2-)
- net TCP0_SSTXRX0_P: now also C7.1, U5.3 (GND)
- net TCP0_SSTXRX1_N: now also C4.1, U4.4 (D2-)
- net TCP0_SSTXRX1_P: now also C3.1, U4.3 (GND)
- net TCP1_CC1: now also U9.4 (C_CC1); no longer J4.A5 (CC1)
- net TCP1_CC2: now also U9.5 (C_CC2); no longer J4.B5 (CC2)
- net TCP1_DN: now also U9.19 (D2)
- net TCP1_DP: now also U9.20 (D1)
- net TCP1_SBU1: now also U9.1 (C_SBU1); no longer J4.A8 (SBU1)
- net TCP1_SBU2: now also U9.2 (C_SBU2); no longer J4.B8 (SBU2)
- net TCP1_SSTX0_N: now also C14.1, U6.2 (D1-); no longer J4.A3 (TX1-)
- net TCP1_SSTX0_P: now also C13.1, U6.1 (D1+); no longer J4.A2 (TX1+)
- net TCP1_SSTX1_N: now also C10.1, U7.2 (D1-); no longer J4.B3 (TX2-)
- net TCP1_SSTX1_P: now also C9.1, U7.1 (D1+); no longer J4.B2 (TX2+)
- net TCP1_SSTXRX0_N: now also C16.1, U6.4 (D2-); no longer J4.B10 (RX1-)
- net TCP1_SSTXRX0_P: now also C15.1, U6.3 (GND); no longer J4.B11 (RX1+)
- net TCP1_SSTXRX1_N: now also C12.1, U7.4 (D2-); no longer J4.A10 (RX2-)
- net TCP1_SSTXRX1_P: now also C11.1, U7.3 (GND); no longer J4.A11 (RX2+)
- net at C1.2: now also J3.B2 (TX2+)
- net at J3.A10 (RX2-): now also C4.2
- net at J3.A11 (RX2+): now also C3.2
- net at J3.A2 (TX1+): now also C5.2
- net at J3.A3 (TX1-): now also C6.2
- net at J3.B10 (RX1-): now also C8.2
- net at J3.B11 (RX1+): now also C7.2
- net at J3.B3 (TX2-): now also C2.2
- new net: C?.1, U9.3 (VBIAS)
- new net: C11.2, J4.A11 (RX2+)
- new net: C10.2, J4.B3 (TX2-)
- new net: C14.2, J4.A3 (TX1-)
- new net: R?.2, U9.9 (~{FLT})
- new net: C?.1, U?.3 (VBIAS)
- new net: C15.2, J4.B11 (RX1+)
- new net: C16.2, J4.B10 (RX1-)
- new net: C12.2, J4.A10 (RX2-)
- new net: C13.2, J4.A2 (TX1+)
- new net: C9.2, J4.B2 (TX2+)
- new net: R?.2, U?.9 (~{FLT})
- new net GND: C?.2, C?.2, C?.2, C?.2, U4.3 (GND), U4.8 (GND), U5.3 (GND), U5.8 (GND), U6.3 (GND), U6.7 (NC), U6.8 (GND), U7.3 (GND), U7.8 (GND), U9.13 (GND), U9.16 (GND), U9.17 (GND), U9.18 (GND), U9.21 (GND), U9.8 (GND), U?.13 (GND), U?.16 (GND), U?.17 (GND), U?.18 (GND), U?.21 (GND), U?.8 (GND)
- new net TCP0_CC1_CN: J3.A5 (CC1), U?.12 (CC1), U?.7 (RPD_G1)
- new net TCP0_CC2_CN: J3.B5 (CC2), U?.11 (CC2), U?.6 (RPD_G2)
- new net TCP0_SBU1_CN: J3.A8 (SBU1), U?.15 (SBU1)
- new net TCP0_SBU2_CN: J3.B8 (SBU2), U?.14 (SBU2)
- new net TCP1_CC1_CN: J4.A5 (CC1), U9.12 (CC1), U9.7 (RPD_G1)
- new net TCP1_CC2_CN: J4.B5 (CC2), U9.11 (CC2), U9.6 (RPD_G2)
- new net TCP1_SBU1_CN: J4.B8 (SBU2), U9.15 (SBU1)
- new net TCP1_SBU2_CN: J4.A8 (SBU1), U9.14 (SBU2)
- new net TCP_LDO_3V3: C?.1, C?.1, R?.1, R?.1, U9.10 (VPWR), U?.10 (VPWR)
Other:
- moved on the sheet: C1, J3, J4

Commit message: July 23, 2024
Parts:
- removed C?: 100nF, symbol Device:C_Small
- removed C?: 1uF, symbol Device:C_Small
- removed R?: 100K, symbol Device:R_Small
- removed U?: TPD6S300A, Package_DFN_QFN:WQFN-20-1EP_3x3mm_P0.4mm_EP1.7x1.7mm_ThermalVias, symbol Power_Protection:TPD6S300A
- added C?: 100nF, symbol Device:C_Small
- added C? (x4): 220pF, symbol Device:C_Small
- added C? (x3): 10uF, symbol Device:C_Small
- added C?: 1uF, symbol Device:C_Small
- added Q? (x2): SiSF00DN, symbol mediacow:SiSF00DN
- added R?: 100K, symbol Device:R_Small
- added U?: TPD6S300A, Package_DFN_QFN:WQFN-20-1EP_3x3mm_P0.4mm_EP1.7x1.7mm_ThermalVias, symbol Power_Protection:TPD6S300A
- added U?: STM32L4A6RGTx, Package_QFP:LQFP-64_10x10mm_P0.5mm, symbol MCU_ST_STM32L4:STM32L4A6RGTx
- added U?: TPS65994ADRSLR, RSL0048B-IPC_A, symbol mediacow:TPS65994ADRSLR
Connections:
- net GND: now also C?.2, C?.2, C?.2, C?.2, C?.2, C?.2, C?.2, C?.2, C?.2, U?.12 (VSSA), U?.13 (GND), U?.16 (GND), U?.17 (GND), U?.18 (GND), U?.18 (VSS), U?.21 (GND), U?.31 (VSS), U?.36 (GND), U?.47 (VSS), U?.63 (VSS), U?.8 (GND)
- net TCP0_CC1: now also C?.1, U?.31 (PA_CC1), U?.4 (C_CC1)
- net TCP0_CC1_CN: now also U?.12 (CC1), U?.7 (RPD_G1)
- net TCP0_CC2: now also C?.1, U?.30 (PA_CC2), U?.5 (C_CC2)
- net TCP0_CC2_CN: now also U?.11 (CC2), U?.6 (RPD_G2)
- net TCP0_DN: now also U?.19 (D2)
- net TCP0_DP: now also U?.20 (D1)
- net TCP0_SBU1: now also U?.1 (C_SBU1)
- net TCP0_SBU1_CN: now also U?.15 (SBU1)
- net TCP0_SBU2: now also U?.2 (C_SBU2)
- net TCP0_SBU2_CN: now also U?.14 (SBU2)
- net TCP0_VBUS: now also Q?.7 (S1), Q?.8 (S1), U?.21 (PA_VBUS), U?.22 (PA_VBUS), U?.23 (PA_VBUS), U?.24 (PA_VBUS)
- net TCP1_CC1: now also C?.1, U?.6 (PB_CC1)
- net TCP1_CC2: now also C?.1, U?.7 (PB_CC2)
- net TCP1_VBUS: now also Q?.7 (S1), Q?.8 (S1), U?.13 (PB_VBUS), U?.14 (PB_VBUS), U?.15 (PB_VBUS), U?.16 (PB_VBUS)
- net TCP_LDO_3V3: now also C?.1, C?.1, R?.1, U?.10 (VPWR), U?.34 (LDO_3V3)
- new net: C?.1, U?.3 (VBIAS)
- new net: R?.2, U?.9 (~{FLT})
- new net ADCIN1: U?.33 (ADCIN1)
- new net ADCIN2: U?.35 (ADCIN2)
- new net PMEC_I2C_TCP_IRQ: U?.43 (I2C_EC_IRQ_N)
- new net PMEC_I2C_TCP_SCL: U?.42 (I2C_EC_SCL)
- new net PMEC_I2C_TCP_SDA: U?.40 (I2C_EC_SDA)
- new net TCP0_GATE_VBUS: Q?.1 (G1), U?.19 (PA_GATE_VBUS)
- new net TCP0_GATE_VSYS: Q?.4 (G2), U?.5 (PA_GATE_VSYS)
- new net TCP1_GATE_VBUS: Q?.1 (G1), U?.18 (PB_GATE_VBUS)
- new net TCP1_GATE_VSYS: Q?.4 (G2), U?.4 (PB_GATE_VSYS)
- new net TCP_5V: U?.11 (PP5V), U?.12 (PP5V), U?.17 (PP5V), U?.20 (PP5V), U?.25 (PP5V), U?.26 (PP5V)
- new net TCP_LDO_1V5: C?.1, U?.37 (LDO_1V5)
- new net TCP_VIN_3V3: C?.1, U?.32 (VIN_3V3)
- new net VBUS: Q?.5 (S2), Q?.5 (S2), Q?.6 (S2), Q?.6 (S2)
- new net VSYS: U?.3 (VSYS)
Other:
- moved on the sheet: C1, C10, C11, C12, C13, C14, C15, C16, C2, C3, C4, C5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

Commit message: Schematic updates July 25, 2024
Parts:
- removed U1: BQ25700A, symbol mediacow:BQ25700A
- added C?: 1uF, symbol Device:C_Small
- added C?: 4.7uF, symbol Device:C_Small
- added C?: 100nF, symbol Device:C_Small
- added C? (x2): 10uF, symbol Device:C_Small
- added C?: 150uF, symbol Device:C_Polarized_Small_US
- added C?: 22nF, symbol Device:C_Small
- added D?: CUS05S40, Diode_SMD:D_SOD-323, symbol Device:D_Schottky_Small_Filled
- added J?: Conn_01x16_Socket, symbol Connector:Conn_01x16_Socket
- added L?: 6.6uH, symbol Device:L_Small
- added Q? (x2): ISC019N03L5S, Package_TO_SOT_SMD:TDSON-8-1, symbol mediacow:ISC019N03L5S
- added R?: 63.4K, symbol Device:R_Small
- added R? (x2): 4.7K, symbol Device:R_Small
- added R?: 100k, symbol Device:R_Small
- added R? (x2): 10m, symbol Device:R_Small
- added U?: BTS6142D, Package_TO_SOT_SMD:TO-252-4, symbol Power_Management:BTS6142D
- added U?: LTC4162EUFD-LAD, 05-08-1712_ADI, symbol mediacow:LTC4162EUFD-LAD-TRPBF
Connections:
- net GND: now also C?.2, C?.2, C?.2, C?.2, C?.2, C?.2, R?.1, U?.16 (SYNC), U?.23 (PGND), U?.24 (PGND), U?.29 (AGND)
- net VBUS: now also Q?.1 (S), Q?.2 (S), Q?.3 (S), U?.7 (VIN)
- net VSYS renamed BC_CLN
- net BC_CLN: now also C?.1, C?.1, Q?.5 (D), Q?.6 (D), Q?.7 (D), Q?.8 (D), R?.2, U?.27 (VOUT), U?.28 (VOUT), U?.3 (VOUTA), U?.4 (CLN)
- new net: L?.2, Q?.1 (S), Q?.2 (S), Q?.3 (S), R?.1, U?.21 (CSP)
- new net: R?.2, U?.11 (RT)
- new net: L?.1, U?.25 (SW), U?.26 (SW)
- new net: U?.1 (OUT), U?.5 (OUT)
- new net: C?.1, D?.1 (K), U?.1 (BOOST)
- new net BC_BATFET: Q?.4 (G), U?.22 (BATFET)
- new net BC_CLP: Q?.5 (D), Q?.6 (D), Q?.7 (D), Q?.8 (D), R?.1, U?.5 (CLP)
- new net BC_DVCC: R?.2, R?.2, R?.2, U?.15 (DVCC)
- new net BC_INFET: Q?.4 (G), U?.6 (INFET)
- new net BC_INTVCC: C?.1, D?.2 (A), U?.17 (CELLS0), U?.2 (INTVCC)
- new net BC_NTC: U?.10 (NTC)
- new net BC_NTCBIAS: U?.9 (NTCBIAS)
- new net BC_SCL: R?.1, U?.13 (SCL)
- new net BC_SDA: R?.1, U?.14 (SDA)
- new net BC_SMBAL: R?.1, U?.12 (*SMBALERT)
- new net BC_SW: C?.2
- new net BC_VCC2P5: U?.18 (CELLS1)
- new net VBAT: C?.1, C?.1, R?.2, U?.19 (BATSENS+), U?.20 (CSN)
- new net VCC2P5: C?.1, U?.8 (VCC2P5)
Other:
- moved on the sheet: U?

Commit message: schem update 2 July 25, 2024
Parts:
- added U?: TPS51397A, symbol mediacow:TPS51397A
Changed lines of the file:
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@@
+	)
+	(symbol
+		(lib_id "mediacow:TPS51397A")
+		(at 374.65 372.11 0)
+		(unit 1)
+		(exclude_from_sim no)
+		(in_bom yes)
+		(on_board yes)
+		(dnp no)
+		(fields_autoplaced yes)
+		(property "Reference" "U?"
+			(at 374.65 353.06 0)
+			(effects
+				(font
+					(size 1.27 1.27)
+				)
+			)
+		)
+		(property "Value" "TPS51397A"
+			(at 374.65 355.6 0)
+			(effects
+				(font
+					(size 1.27 1.27)
+				)
+			)
+		)
+		(property "Footprint" ""
+			(at 374.65 373.38 0)
+			(effects
+				(font
+					(size 1.27 1.27)
+				)
+				(hide yes)
+			)
+		)
+		(property "Datasheet" ""
+			(at 374.65 373.38 0)
+			(effects
+				(font
+					(size 1.27 1.27)
+				)
+				(hide yes)
+			)
+		)
+		(property "Description" ""
+			(at 374.65 373.38 0)
+			(effects
+				(font
+					(size 1.27 1.27)
+				)
+				(hide yes)
+			)
+		)
+		(pin "14"
+		)
+		(pin "7"
+		)
+		(pin "13"
+		)
+		(pin "2"
+		)
+		(pin "3"
+		)
+		(pin "12"
+		)
+		(pin "11"
+		)
+		(pin "8"
+		)
+		(pin "16"
+		)
+		(pin "4"
+		)
+		(pin "20"
+		)
+		(pin "6"
+		)
+		(pin "19"
+		)
+		(pin "1"
+		)
+		(pin "17"
+		)
+		(pin "10"
+		)
+		(pin "9"
+		)
+		(pin "5"
+		)
+		(pin "15"
+		)
+		(pin "18"
+		)
+		(instances
+			(project "mct2"
+				(path "/0917e100-0497-47cd-9e32-3e43ad224d2b/a8bf6592-f5ae-4d8b-8322-3be7272b77f0"
+					(reference "U?")
+					(unit 1)
+				)
+			)
+		)
 	)
 	(symbol

Commit message: July 27, 2024
Parts:
- removed C?: 1uF, symbol Device:C_Small
- removed C?: 4.7uF, symbol Device:C_Small
- removed C?: 100nF, symbol Device:C_Small
- removed C?: 22nF, symbol Device:C_Small
- removed U?: BTS6142D, Package_TO_SOT_SMD:TO-252-4, symbol Power_Management:BTS6142D
- removed U?: LTC4162EUFD-LAD, 05-08-1712_ADI, symbol mediacow:LTC4162EUFD-LAD-TRPBF
- added C?: 220pF, symbol Device:C_Small
- added C?: 1uF, symbol Device:C_Small
- added C?: 10uF, symbol Device:C_Small
- added C? (x2): 100nF, symbol Device:C_Small
- added C?: 22nF, symbol Device:C_Small
- added R?: 1.2K, symbol Device:R_Small
- added R?: 10K, symbol Device:R_Small
- added U?: LTC4162EUFD-LAD, 05-08-1712_ADI, symbol mediacow:LTC4162EUFD-LAD
- added U?: BTS7006-1EPP, Package_SO:Infineon_PG-TSDSO-14-22, symbol mediacow:BTS7006-1EPP
Connections:
- net BC_INTVCC: now also U?.17 (CELLS0)
- net BC_NTC: now also R?.2, U?.10 (NTC)
- net BC_SCL: now also R?.2, U?.13 (SCL); no longer R?.1
- net BC_SDA: now also R?.2, U?.14 (SDA); no longer R?.1
- net BC_SMBAL: now also R?.2, U?.12 (SMBALERT#); no longer R?.1
- net BC_VCC2P5: now also U?.18 (CELLS1)
- net GND: now also U?.49 (GND), C?.2, C?.2, C?.2, C?.2, U?.1 (GND), U?.16 (SYNC), U?.23 (PGND1), U?.24 (PGND2), U?.29 (EPAD)
- net VBAT: now also U?.19 (BATSENS+), U?.20 (CSN)
- net VBUS: now also C?.1, U?.7 (VIN)
- net at L?.2, Q?.1 (S), Q?.2 (S)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: now also U?.21 (CSP)
- net at R?.2: now also U?.11 (RT)
- net at L?.1: now also C?.2, U?.25 (SW), U?.26 (SW)
- net at D?.1 (K): now also C?.1, U?.1 (BOOST)
- net BC_BATFET: no longer names the net of Q?.4 (G)
- net BC_BATFET: now also U?.22 (BATFET)
- net BC_CLN renamed VSYS
- net VSYS: now also C?.1, U?.27 (VOUT), U?.28 (VOUT), U?.3 (VOUTA), U?.4 (CLN)
- net BC_CLP: no longer names the net of Q?.5 (D), Q?.6 (D), Q?.7 (D), Q?.8 (D), R?.1
- net BC_CLP: now also U?.5 (CLP)
- removed net BC_DVCC: R?.2, R?.2, R?.2
- net BC_INFET: no longer names the net of Q?.4 (G)
- net BC_INFET: now also U?.6 (INFET)
- new net: C?.1, U?.8 (VCC2P5)
- new net: R?.1, R?.1, R?.1, U?.15 (DVCC)
- new net: R?.1, U?.4 (IS)
- new net: C?.1, U?.2 (INTVCC)
- new net: R?.1, U?.9 (NTCBIAS)
- new net: U?.10 (OUT), U?.12 (OUT), U?.13 (OUT), U?.14 (OUT), U?.8 (OUT), U?.9 (OUT)
Other:
- note added: "Battery Charger"
- note added: "CTCL 2021-2024"
- note added: "July 4, 2024 - July 26, 2024"
- note added: "MediaCow Touch 2 - Power Subsystem"
- note added: "System Power Control"
- note added: "USB Type-C"
- moved on the sheet: C1, C10, C11, C12, C13, C14, C15, C16, C2, C3, C4, C5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

Commit message: Aug 1, 2024
Parts:
- removed U?: STM32L4A6RGTx, Package_QFP:LQFP-64_10x10mm_P0.5mm, symbol MCU_ST_STM32L4:STM32L4A6RGTx
Other:
- note added: "July 4, 2024 - July 30, 2024"
- note removed: "July 4, 2024 - July 26, 2024"
- moved on the sheet: C?

Commit message: Aug 2, 2024
Connections:
- net GND: now also J?.1 (Pin_1), J?.14 (Pin_14), J?.15 (Pin_15), J?.16 (Pin_16), J?.2 (Pin_2), J?.3 (Pin_3)
- net VBAT: now also J?.10 (Pin_10), J?.11 (Pin_11), J?.6 (Pin_6), J?.7 (Pin_7), J?.8 (Pin_8), J?.9 (Pin_9)
- net BAT_SMB_C: now reaches J?.12 (Pin_12)
- net BAT_SMB_D: now reaches J?.13 (Pin_13)
- net BAT_THERM_N: now reaches J?.4 (Pin_4)
- net BAT_THERM_P: now reaches J?.5 (Pin_5)
Other:
- note added: "July 4, 2024 - August 2, 2024"
- note added: "WARNING: This pinout is a guess of what it could be. Ensure this pinout is correct before starting PCB design."
- note removed: "July 4, 2024 - July 30, 2024"
- moved on the sheet: J?

Commit message: Aug 3, 2024
Parts:
- added C? (x3): 10uF, symbol Device:C_Small
- added C?: 10nF, symbol Device:C_Small
- added C?: 1uF, symbol Device:C_Small
- added C? (x4): 22uF, symbol Device:C_Small
- added C? (x2): 100nF, symbol Device:C_Small
- added C?: 22pF, symbol Device:C_Small
- added D?: MMSZ5231BS-7-F, Diode_SMD:D_SOD-323, symbol Device:D_Zener_Small_Filled
- added L?: 2.2uH, symbol Device:L_Small
- added R?: 100K, symbol Device:R_Small
- added R? (x3): 20K, symbol Device:R_Small
- added R?: 150K, symbol Device:R_Small
- added R? (x2): 0, symbol Device:R_Small
- added U?: TPS51386RJNR, VQFN-HR12_RJN_TEX, symbol mediacow:TPS51386RJNR
Connections:
- net GND: now also C?.2, C?.2, C?.2, C?.2, C?.2, C?.2, C?.2, C?.2, C?.2, C?.2, D?.2 (A), R?.2, R?.2, U?.10 (AGND), U?.12 (MODE), U?.2 (PGND)
- net VSYS: now also C?.1, C?.1, C?.1, C?.1, R?.1, U?.1 (VIN)
- new net: R?.1, U?.3 (PG)
- new net: C?.1, R?.2, U?.9 (VCC)
- new net: C?.2, R?.1, R?.2, U?.4 (FB)
- new net: C?.2, L?.1, U?.7 (SW)
- new net: R?.1, U?.8 (VBST)
- new net: C?.1, D?.1 (K), R?.1, R?.2
- new net: C?.1, R?.2 (x2)
- new net REG_USB_5V_EN: U?.11 (EN)
- new net USB_5V: C?.1, C?.1, C?.1, C?.1, L?.2, R?.1, R?.1
- no-connect marks 0 -> 1
Other:
- note added: "July 4, 2024 - August 3, 2024"
- note removed: "July 4, 2024 - August 2, 2024"
