File: circuits/mct2/mct2_power.kicad_sch (KiCad schematic)
At the start: 87 parts, among them J3 USB_C_Receptacle, J4 USB_C_Receptacle, U4 TPD4EUSB30, U5 TPD4EUSB30, U6 TPD4EUSB30, U7 TPD4EUSB30, U9 TPD6S300A

Commit message: Aug 7, 2024 stuff in case I don't work on this before going to FMB
Parts:
- removed Q? (x2): SiSF00DN, symbol mediacow:SiSF00DN
- removed U?: TPS65994ADRSLR, RSL0048B-IPC_A, symbol mediacow:TPS65994ADRSLR
- added C? (x10): 100nF, symbol Device:C_Small
- added C? (x4): 22uF, symbol Device:C_Small
- added C? (x4): 10uF, symbol Device:C_Small
- added C?: 22nF, symbol Device:C_Small
- added C? (x2): 1uF, symbol Device:C_Small
- added D? (x2): PPS1045, Package_TO_SOT_SMD:TO-277B, symbol mediacow:PPS1045
- added L?: 4.7uF, symbol Device:L_Small
- added Q? (x2): NX3008NBKVL, symbol mediacow:NX3008NBKVL
- added Q? (x4): BSZ086P03NS3E, mediacow:Infineon_PG-TSDSON-8, symbol mediacow:BSZ086P03NS3E
- added Q? (x2): T2N7002BK, symbol mediacow:T2N7002BK
- added R? (x4): 60.4K, symbol Device:R_Small
- added R? (x10): 10K, symbol Device:R_Small
- added R? (x2): 100K, symbol Device:R_Small
- added R? (x2): 0, symbol Device:R_Small
- added R?: 21.5K, symbol Device:R_Small
- added R? (x2): DNP, symbol Device:R_Small
- added R? (x2): 590K, symbol Device:R_Small
- added R? (x2): 1K, symbol Device:R_Small
- added U?: TPS65988DKRSHR, mediacow:QFN_DKRSHR_TEX, symbol mediacow:TPS65988DKRSHR
- added U?: TLV1701A, symbol mediacow:TLV1701
- added U?: TLV1701, symbol mediacow:TLV1701
- added U?: MPS8859, symbol mediacow:MP8859GQ
Connections:
- net REG_USB_5V_EN is gone; now on an unnamed net: U?.11 (EN)
- net GND: now also J3.A1 (GND), J3.A12 (GND), J3.B1 (GND), J3.B12 (GND), J3.S1 (SHIELD), J4.A1 (GND), J4.A12 (GND), J4.B1 (GND), J4.B12 (GND), J4.S1 (SHIELD), C?.2, C?.2, C?.2, C?.2, C?.2, C?.2, C?.2, C?.2, C?.2, C?.2, C?.2, Q?.2 (S), Q?.2 (S), Q?.2 (S), Q?.2 (S), R?.1, R?.2, R?.2, R?.2, R?.2, R?.2, R?.2, R?.2, U?.2 (V-), U?.2 (V-), U?.20 (GND), U?.51 (GND), U?.59 (GND)
- net TCP0_CC1: now also U?.45 (C2_CC1)
- net TCP0_CC2: now also U?.47 (C2_CC2)
- net TCP0_VBUS: now also C?.1, Q?.1 (S), Q?.2 (S), Q?.3 (S)
- net TCP1_CC1: now also U?.24 (C1_CC1)
- net TCP1_CC2: now also U?.26 (C1_CC2)
- net TCP1_VBUS: now also C?.1, D?.3 (K), D?.3 (K), Q?.1 (S), Q?.2 (S), Q?.3 (S)
- net TCP_LDO_3V3: now also C?.1, C?.1, R?.1, R?.1, U?.5 (V+), U?.5 (V+)
- net VSYS: now also U?.1 (IN)
- new net: R?.1, R?.2, U?.3 (-) (x2)
- new net: C?.1, U?.13 (VBUS1), U?.14 (VBUS1)
- new net: C?.1, U?.3 (VBUS2), U?.4 (VBUS2)
- new net: C?.1, U?.35 (LDO_1V8)
- new net: C?.1, U?.9 (LDO_3V3)
- new net: C?.1, C?.1, C?.1, D?.1 (A), D?.2 (A), Q?.1 (S), Q?.2 (S), Q?.3 (S), R?.1 (x2)
- new net: C?.2, C?.2, C?.2, Q?.4 (G), Q?.4 (G), R?.1, R?.2 (x2)
- new net: Q?.3 (D), R?.2 (x2)
- new net: Q?.3 (D), Q?.G (1), R?.1, R?.2 (x2)
- new net: R?.1, R?.1, R?.2, U?.1 (+) (x2)
- new net: C?.1, L?.1, U?.15 (SW1)
- new net: C?.2, L?.2, U?.14 (SW2)
- new net: C?.1, Q?.5 (D), Q?.5 (D), Q?.6 (D), Q?.6 (D), Q?.7 (D), Q?.7 (D), Q?.8 (D), Q?.8 (D), R?.1, R?.1 (x2)
- new net: R?.1, U?.13 (BST2)
- new net: C?.1, R?.2
- new net: C?.1, R?.1, U?.7 (OC)
- new net: R?.1, R?.2, U?.4 (ADD)
- new net: R?.2, U?.9 (VCC)
- new net: Q?.G (1), R?.2, R?.2, U?.4 (x2)
- new net: R?.2, U?.16 (BST1)
- new net: C?.2, R?.1
- new net SMEC_SDA2: U?.6 (SDA)
- new net TCP_DRAIN1: U?.15 (DRAIN1), U?.19 (DRAIN1), U?.58 (DRAIN1), U?.8 (DRAIN1)
- new net TCP_DRAIN2: U?.52 (DRAIN2), U?.56 (DRAIN2), U?.57 (DRAIN2), U?.7 (DRAIN2)
- new net TCP_HPD1: U?.30 (HPD1(GPIO3))
- new net TCP_HPD2: U?.31 (HPD2_(GPIO4))
- new net TCP_PA_EXT_EN: R?.1
- new net TCP_PB_EXT_EN: R?.1
- new net TCP_PPHV1_EN: U?.3 (EN)
- new net TCP_PP_HV1: C?.1, U?.11 (PP_HV1), U?.12 (PP_HV1)
- new net TCP_PP_HV2: C?.1, U?.1 (PP_HV2), U?.2 (PP_HV2)
Other:
- note added: "DRAIN1 and DRAIN2 must be left floating"
- note added: "July 4, 2024 - August 6, 2024"
- note removed: "July 4, 2024 - August 3, 2024"
- moved on the sheet: C?, D?, J?, L?, Q?, R?, U?

Commit message: Aug 10, 2024
Parts:
- removed C? (x6): 10uF, symbol Device:C_Small
- removed C?: 220pF, symbol Device:C_Small
- removed C?: 10nF, symbol Device:C_Small
- removed C?: 1uF, symbol Device:C_Small
- removed C? (x4): 22uF, symbol Device:C_Small
- removed C? (x2): 100nF, symbol Device:C_Small
- removed C?: 22pF, symbol Device:C_Small
- removed D?: MMSZ5231BS-7-F, Diode_SMD:D_SOD-323, symbol Device:D_Zener_Small_Filled
- removed L?: 2.2uH, symbol Device:L_Small
- removed R?: 100K, symbol Device:R_Small
- removed R? (x3): 20K, symbol Device:R_Small
- removed R?: 150K, symbol Device:R_Small
- removed R? (x2): 0, symbol Device:R_Small
- removed U?: TPS51386RJNR, VQFN-HR12_RJN_TEX, symbol mediacow:TPS51386RJNR
- removed U?: TPS51397A, symbol mediacow:TPS51397A
- added C? (x4): 10uF, symbol Device:C_Small
- added C? (x2): 100nF, symbol Device:C_Small
- added C?: 22nF, symbol Device:C_Small
- added C? (x2): 100uF, symbol Device:C_Small
- added L?: 4.7uF, symbol Device:L_Small
- added R?: 301K, symbol Device:R_Small
- added R? (x2): 0, symbol Device:R_Small
- added R?: 21.5K, symbol Device:R_Small
- added R? (x2): 4.7K, symbol Device:R_Small
- added R?: 499K, symbol Device:R_Small
- added U?: MPS8859, symbol mediacow:MP8859GQ
Connections:
- net GND: now also C?.2, C?.2, R?.2, U?.10 (AGND), U?.11 (GND), U?.2 (GND), C?.2, C?.2, C?.2, C?.2, C?.2, C?.2, C?.2, R?.1, R?.2, U?.10 (AGND), U?.11 (GND), U?.2 (GND)
- net TCP1_VBUS: no longer D?.3 (K), D?.3 (K)
- net TCP_PPHV1_EN: now also U?.3 (EN)
- net TCP_PP_HV1: now also U?.12 (OUT), C?.1, C?.1, C?.1
- net TCP_PP_HV2: now also C?.1, C?.1, C?.1, U?.12 (OUT)
- net VBUS: now also D?.3 (K), D?.3 (K)
- net VSYS: now also U?.10 (OUT), U?.12 (OUT), U?.13 (OUT), U?.14 (OUT), U?.8 (OUT), U?.9 (OUT), U?.1 (IN); no longer C?.1, C?.1, Q?.5 (D), Q?.6 (D), Q?.7 (D), Q?.8 (D), R?.2, U?.27 (VOUT), U?.28 (VOUT), U?.3 (VOUTA), U?.4 (CLN)
- net SMB2_SCL: now reaches U?.5 (SCL)
- net SMB2_SCL: now also U?.5 (SCL)
- net SMB2_ALT: now reaches U?.8 (ALT)
- net SMB2_ALT: now also U?.8 (ALT)
- net VSB: now reaches U?.15 (VS)
- net VSB: now also C?.1, C?.1, Q?.5 (D), Q?.6 (D), Q?.7 (D), Q?.8 (D), R?.2, U?.27 (VOUT), U?.28 (VOUT), U?.3 (VOUTA), U?.4 (CLN)
- net at U?.2 (IN): now also R?.2
- net at U?.3 (DEN): now also R?.2
- net SMEC_SDA2 renamed SMB2_SDA
- net SMB2_SDA: now also U?.6 (SDA)
- new net: C?.1, L?.1, U?.15 (SW1)
- new net: C?.2, L?.2, U?.14 (SW2)
- new net: R?.1, R?.2, U?.4 (ADD)
- new net: C?.2, R?.1
- new net: R?.1, U?.13 (BST2)
- new net: C?.1, R?.2
- new net: C?.1, R?.1, U?.7 (OC)
- new net: R?.2, U?.16 (BST1)
- new net: R?.2, U?.9 (VCC)
- new net VSYS_SW_DEN: R?.1
- new net VSYS_SW_IN: R?.1
- no-connect marks 1 -> 0
Other:
- note added: "July 4, 2024 - August 10, 2024"
- note removed: "July 4, 2024 - August 6, 2024"
- moved on the sheet: C?, D?, J?, L?, Q?, R?, U?

Commit message: Aug 11, 2024 1
Parts:
- added R?: 540K, symbol Device:R_Small
Connections:
- net at R?.1, U?.4 (IS): now also R?.2
- new net VSYS_SW_IS: R?.1
Other:
- note added: "July 4, 2024 - August 11, 2024"
- note removed: "July 4, 2024 - August 10, 2024"
- moved on the sheet: R?, U?

Commit message: Aug 11, 2024 2
Connections:
- net GND: no longer U6.7 (NC)
- net SMB2_ALT: now also U?.34 (I2C2_IRQ)
- net SMB2_SCL: now also U?.32 (I2C2_SCL)
- net SMB2_SDA: now also U?.33 (I2C2_SDA)
- net TCP_LDO_3V3: now also C?.1, U?.9 (LDO_3V3)
- net TCP_LDO_1V8: now reaches C?.1, U?.35 (LDO_1V8)
- net TCP_PP_HV1 renamed TCP0_PPHV
- net TCP_PP_HV2 renamed TCP1_PPHV
Other:
- note added: "MediaCow Touch 2"
- note added: "MediaCow Touch 2 - System"
- note removed: "MediaCow Touch 2 - Power Subsystem"
- note removed: "System Power Control"
- moved on the sheet: C1, C10, C11, C12, C13, C14, C15, C16, C2, C3, C4, C5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

Commit message: Aug 13, 2024
Parts:
- added D?: MMSZ5227B, symbol Device:D_Zener_Small_Filled
- R?: value 540K -> 470K
Connections:
- net GND: now also D?.2 (A)
- net VSYS_SW_IS: now also D?.1 (K)
Other:
- note added: "July 4, 2024 - August 13, 2024"
- note added: "MediaCow Touch 2 - Power"
- note removed: "July 4, 2024 - August 11, 2024"
- note removed: "MediaCow Touch 2 - System"
- moved on the sheet: R?, U?

Commit message: Aug 17, 2024
Parts:
- added C? (x8): 22uF, symbol Device:C_Small
- added C? (x4): 100nF, symbol Device:C_Small
- added C? (x2): 10nF, symbol Device:C_Small
- added C? (x6): 10uF, symbol Device:C_Small
- added C? (x2): 1uF, symbol Device:C_Small
- added C? (x2): 22pF, symbol Device:C_Small
- added D? (x2): MMSZ5231BS-7-F, Diode_SMD:D_SOD-323, symbol Device:D_Zener_Small_Filled
- added L? (x2): 2.2uH, symbol Device:L_Small
- added R? (x6): 20K, symbol Device:R_Small
- added R? (x2): 100K, symbol Device:R_Small
- added R? (x2): 150K, symbol Device:R_Small
- added R? (x4): 0, symbol Device:R_Small
- added U? (x2): TPS51386RJNR, VQFN-HR12_RJN_TEX, symbol mediacow:TPS51386RJNR
- R? (x3): now not fitted
Connections:
- net GND: now also C?.2, C?.2, C?.2, C?.2, C?.2, C?.2, C?.2, C?.2, C?.2, C?.2, C?.2, C?.2, C?.2, C?.2, C?.2, C?.2, C?.2, C?.2, C?.2, C?.2, D?.2 (A), D?.2 (A), R?.2, R?.2, R?.2, R?.2, U?.10 (AGND), U?.10 (AGND), U?.12 (MODE), U?.12 (MODE), U?.2 (PGND), U?.2 (PGND)
- net VSYS: now also C?.1, C?.1, C?.1, C?.1, C?.1, C?.1, C?.1, C?.1, R?.1, R?.1, U?.1 (VIN), U?.1 (VIN)
- new net: C?.1, D?.1 (K), R?.1, R?.2, U?.11 (EN) (x2)
- new net: C?.1, R?.2, U?.9 (VCC) (x2)
- new net: C?.1, R?.2 (x4)
- new net: C?.2, L?.1, U?.7 (SW) (x2)
- new net: C?.2, R?.1, R?.2, U?.4 (FB) (x2)
- new net: R?.1, U?.8 (VBST) (x2)
- new net USB_5V: C?.1, C?.1, C?.1, C?.1, L?.2, R?.1, R?.1
- new net USB_5V_PG: R?.1, U?.3 (PG)
- new net VSYS_LV: C?.1, C?.1, C?.1, C?.1, L?.2, R?.1, R?.1
- new net VSYS_LV_PG: R?.1, U?.3 (PG)
- no-connect marks 0 -> 4
Other:
- note added: "Power Switch"
- note added: "USB_5V"
- note added: "VSYS_LV"
- moved on the sheet: D?, R?, U?

Commit message: Aug 19, 2024
Connections:
- net SMB2_ALT is gone; now on net SMB1_ALT: U?.34 (I2C2_IRQ), U?.8 (ALT), U?.8 (ALT)
- net SMB2_SCL is gone; now on net SMB1_SCL: U?.32 (I2C2_SCL), U?.5 (SCL), U?.5 (SCL)
- net SMB2_SDA is gone; now on net SMB1_SDA: U?.33 (I2C2_SDA), U?.6 (SDA), U?.6 (SDA)
- net BC_SCL renamed SMB1_SCL
- net BC_SDA renamed SMB1_SDA
- net BC_SMBAL renamed SMB1_ALT
Other:
- note added: "July 4, 2024 - August 19, 2024"
- note removed: "July 4, 2024 - August 13, 2024"
- moved on the sheet: C?, D?, J?, L?, Q?, R?, U?

Commit message: Aug 21, 2024 1
Parts:
- added C? (x3): 10uF, symbol Device:C_Small
- added C? (x4): 22uF, symbol Device:C_Small
- added C?: 1uF, symbol Device:C_Small
- added C? (x2): 100nF, symbol Device:C_Small
- added C?: 10nF, symbol Device:C_Small
- added C?: 22pF, symbol Device:C_Small
- added D?: MMSZ5231BS-7-F, Diode_SMD:D_SOD-323, symbol Device:D_Zener_Small_Filled
- added L?: 2.2uH, symbol Device:L_Small
- added R? (x3): 20K, symbol Device:R_Small
- added R?: 90K, symbol Device:R_Small
- added R? (x2): 0, symbol Device:R_Small
- added R?: 100K, symbol Device:R_Small
- added U?: TPS51386RJNR, VQFN-HR12_RJN_TEX, symbol mediacow:TPS51386RJNR
Connections:
- net GND: now also C?.2, C?.2, C?.2, C?.2, C?.2, C?.2, C?.2, C?.2, C?.2, C?.2, D?.2 (A), R?.2, R?.2, U?.10 (AGND), U?.12 (MODE), U?.2 (PGND)
- net VSYS: now also C?.1, C?.1, C?.1, C?.1, R?.1, U?.1 (VIN)
- net VSYS_LV_PG: now also R?.1, U?.3 (PG)
- new net: C?.1, D?.1 (K), R?.1, R?.2, U?.11 (EN)
- new net: C?.2, L?.1, U?.7 (SW)
- new net: C?.2, R?.1, R?.2, U?.4 (FB)
- new net: C?.1, R?.2, U?.9 (VCC)
- new net: C?.1, R?.2 (x2)
- new net: R?.1, U?.8 (VBST)
- new net M2_3V3: C?.1, C?.1, C?.1, C?.1, L?.2, R?.1, R?.1
- no-connect marks 4 -> 6
Other:
- note added: "M2_3V3"
