File: circuits/mct2/mct2_power.kicad_sch (KiCad schematic)
At the start: 204 parts, among them J3 USB_C_Receptacle, J4 USB_C_Receptacle, U4 TPD4EUSB30, U5 TPD4EUSB30, U6 TPD4EUSB30, U7 TPD4EUSB30, U9 TPD6S300A

Commit message: Aug 22, 2024 1
Parts:
- added C? (x9): 10nF, symbol Device:C_Small
- added C?: 100nF, symbol Device:C_Small
- added C?: 10uF, symbol Device:C_Small
- added C? (x2): 22uF, symbol Device:C_Small
- added C? (x2): 1uF, symbol Device:C_Small
- added R? (x4): 3.3K, symbol Device:R_Small
- added R?: 100K, symbol Device:R_Small
- added U?: W25X05CLSN, Package_SO:SOIC-8_3.9x4.9mm_P1.27mm, symbol mediacow:W25X05CLSN
- added U?: MIC5504-3.3YM5, Package_TO_SOT_SMD:SOT-23-5, symbol Regulator_Linear:MIC5504-3.3YM5
Connections:
- net GND: now also C?.2, C?.2, C?.2, C?.2, C?.2, C?.2, C?.2, C?.2, C?.2, C?.2, C?.2, C?.2, C?.2, C?.2, C?.2, R?.2, U?.2 (GND), U?.4 (GND)
- net TCP0_VBUS: now also C?.1, C?.1, C?.1, C?.1
- net TCP1_VBUS: now also C?.1, C?.1, C?.1, C?.1
- net TCP_LDO_3V3: now also C?.1, R?.1, R?.1, R?.1, R?.1, U?.8 (VCC)
- net TCP_PPHV1_EN: no longer U?.3 (EN)
- net VSYS_LV: now also U?.25 (PP1_CABLE), U?.46 (PP2_CABLE), C?.1, C?.1, C?.1, U?.1 (VIN), U?.3 (EN)
- net VSYS_LV_PG: no longer R?.1, U?.3 (PG)
- net at U?.44 (HRESET): now also C?.1, R?.1
- net at U?.5 (VIN_3V3): now also C?.1, C?.1, U?.5 (VOUT)
- net SMB1_ALT renamed SYS_SMB_ALT
- net SMB1_SCL renamed SYS_SMB_SCL
- net SMB1_SDA renamed SYS_SMB_SDA
- new net: R?.2, U?.3 (~{WP})
- new net: R?.2, U?.7 (~{HOLD})
- new net M2_3V3_PG: R?.1, U?.3 (PG)
- new net TCP_NVM_CLK: U?.6 (SCK)
- new net TCP_NVM_CS: R?.2, U?.1 (~{CS})
- new net TCP_NVM_MISO: R?.2, U?.2 (DO(IO1))
- new net TCP_NVM_MOSI: U?.5 (DI(IO0))
- new net TCP_PPHV2_EN: U?.3 (EN)
- no-connect marks 6 -> 9
Other:
- note added: "July 4, 2024 - August 21, 2024"
- note removed: "July 4, 2024 - August 19, 2024"
- moved on the sheet: C?

Commit message: Aug 28, 2024
Parts:
- added C? (x2): 1uF, symbol Device:C_Small
- added C?: 100nF, symbol Device:C_Small
- added D?: WP154A4SEJ3VBDZGC/CA, Connector_PinSocket_1.27mm:PinSocket_1x04_P1.27mm_Vertical, symbol Device:LED_RABG
- added U?: IS31FL3193, Package_DFN_QFN:DFN-10-1EP_3x3mm_P0.5mm_EP1.75x2.7mm, symbol mediacow:IS31FL3193
Connections:
- net GND: now also C?.2, C?.2, C?.2, U?.6 (GND), U?.7 (AD)
- new net: D?.1 (RK), U?.3 (OUT1)
- new net: D?.3 (BK), U?.5 (OUT3)
- new net: D?.4 (GK), U?.4 (OUT2)
- new net LED_3V3: C?.1, C?.1, C?.1, D?.2 (A), U?.2 (VDD)
Other:
- moved on the sheet: C1, C10, C11, C12, C13, C14, C15, C16, C2, C3, C4, C5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

Commit message: Aug 31, 2024
Parts:
- removed C? (x6): 10uF, symbol Device:C_Small
- removed C? (x4): 100nF, symbol Device:C_Small
- removed C? (x2): 10nF, symbol Device:C_Small
- removed C? (x3): 1uF, symbol Device:C_Small
- removed C? (x4): 22uF, symbol Device:C_Small
- removed C?: 22nF, symbol Device:C_Small
- removed C?: 100uF, symbol Device:C_Small
- removed C?: 22pF, symbol Device:C_Small
- removed D? (x2): MMSZ5231BS-7-F, Diode_SMD:D_SOD-323, symbol Device:D_Zener_Small_Filled
- removed L?: 4.7uF, symbol Device:L_Small
- removed L?: 2.2uH, symbol Device:L_Small
- removed R? (x5): 20K, symbol Device:R_Small
- removed R?: 100K, symbol Device:R_Small
- removed R? (x4): 0, symbol Device:R_Small
- removed R?: 21.5K, symbol Device:R_Small
- removed R?: 150K, symbol Device:R_Small
- removed R? (x2): DNP, symbol Device:R_Small
- removed U?: MIC5504-3.3YM5, Package_TO_SOT_SMD:SOT-23-5, symbol Regulator_Linear:MIC5504-3.3YM5
- removed U?: TPS51386RJNR, VQFN-HR12_RJN_TEX, symbol mediacow:TPS51386RJNR
- removed U?: MPS8859, symbol mediacow:MP8859GQ
- added C? (x2): 2.2uF, symbol Device:C_Small
- added C? (x13): 100nF, symbol Device:C_Small
- added C? (x9): 10uF, symbol Device:C_Small
- added C?: 100uF, symbol Device:C_Small
- added C? (x6): 1uF, symbol Device:C_Small
- added C? (x12): 22uF, symbol Device:C_Small
- added C? (x3): 4.7uF, symbol Device:C_Small
- added C?: 22nF, symbol Device:C_Small
- added D? (x2): SS15, Diode_SMD:D_SMA, symbol Device:D_Schottky_Small_Filled
- added D?: BAT201M3, Diode_SMD:D_SOD-323F, symbol Device:D_Schottky_Small_Filled
- added J?: Conn_01x04_Pin, Connector:FanPinHeader_1x04_P2.54mm_Vertical, symbol Connector:Conn_01x04_Pin
- added L?: 13uH, symbol Device:L_Small
- added L? (x4): 3.9uH, symbol Device:L_Small
- added L?: 15uH, symbol Device:L_Small
- added L?: 17uH, symbol Device:L_Small
- added L?: 4.7uF, symbol Device:L_Small
- added R? (x2): 1M, symbol Device:R_Small
- added R? (x3): 10K, symbol Device:R_Small
- added R?: 140K, symbol Device:R_Small
- added R?: 20.7K, symbol Device:R_Small
- added R? (x3): 100K, symbol Device:R_Small
- added R?: 5.23K, symbol Device:R_Small
- added R?: 499K, symbol Device:R_Small
- added R? (x3): 0, symbol Device:R_Small
- added R?: 21.5K, symbol Device:R_Small
- added R?: 301K, symbol Device:R_Small
- added U? (x2): TLV73333PDBV, Package_TO_SOT_SMD:SOT-23-5, symbol Regulator_Linear:TLV73333PDBV
- added U?: AP63205WU, Package_TO_SOT_SMD:TSOT-23-6, symbol mediacow:AP63205WU
- added U?: TPS563300, symbol mediacow:TPS563300
- added U? (x2): SY21019, Package_TO_SOT_SMD:SOT-23-6, symbol mediacow:SY21019
- added U? (x3): AP63203, Package_TO_SOT_SMD:TSOT-23-6, symbol mediacow:AP63203WU
- added U?: MIC5504-1.8YM5, Package_TO_SOT_SMD:SOT-23-5, symbol Regulator_Linear:MIC5504-1.8YM5
- added U?: MPS8859, symbol mediacow:MP8859GQ
Connections:
- net GND: now also C?.1, C?.1, C?.1, C?.1, C?.1, C?.2, C?.2, C?.2, C?.2, C?.2, C?.2, C?.2, C?.2, C?.2, C?.2, C?.2, C?.2, C?.2, C?.2, C?.2, C?.2, C?.2, C?.2, C?.2, C?.2, C?.2, C?.2, C?.2, C?.2, C?.2, C?.2, C?.2, C?.2, C?.2, D?.2 (A), D?.2 (A), J?.1 (Pin_1), R?.1, R?.2, R?.2, R?.2, R?.2, R?.2, R?.2, R?.2, U?.10 (AGND), U?.11 (GND), U?.2 (GND), U?.2 (GND), U?.2 (GND), U?.2 (GND), U?.2 (GND), U?.2 (GND), U?.4 (GND), U?.4 (GND), U?.4 (GND), U?.4 (GND)
- net SYS_SMB_ALT: no longer U?.8 (ALT)
- net SYS_SMB_SCL: no longer U?.5 (SCL)
- net SYS_SMB_SDA: no longer U?.6 (SDA)
- net TCP0_PPHV: now also C?.1, C?.1, C?.1, U?.12 (OUT)
- net TCP_LDO_3V3: now also D?.2 (A); no longer C?.1, R?.1, R?.1, R?.1, R?.1, U?.8 (VCC)
- net TCP_NVM_CLK: now also U?.38 (SPI_CLK_(GPIO10))
- net TCP_NVM_CS: now also U?.39 (SPI_SS_(GPIO11))
- net TCP_NVM_MISO: now also U?.36 (SPI_MISO_(GPIO8))
- net TCP_NVM_MOSI: now also U?.37 (SPI_MOSI_(GPIO9))
- net VSB: no longer U?.15 (VS)
- net VSYS: now also U?.15 (VS), C?.1, C?.1, C?.1, C?.1, C?.1, C?.1, C?.1, C?.1, C?.1, C?.1, C?.2, C?.2, R?.1, R?.1, U?.1 (IN), U?.2 (EN), U?.2 (EN), U?.3 (VIN), U?.3 (VIN), U?.3 (VIN), U?.3 (VIN), U?.3 (VIN), U?.5 (IN), U?.5 (IN); no longer U?.10 (OUT), U?.12 (OUT), U?.13 (OUT), U?.14 (OUT), U?.8 (OUT), U?.9 (OUT)
- net USB_5V_EN: now reaches U?.11 (EN)
- net TCP_VIN_3V3: now reaches U?.5 (VIN_3V3)
- net TCP_VIN_3V3: now also C?.1, C?.1, C?.1, C?.2, L?.2, U?.1 (FB)
- net LED_EN: now reaches U?.1 (SDB)
- net LED_EN: now also R?.1
- net LED_VBM: now reaches U?.10 (V_BM)
- net SYS_I2C_SCL: now reaches U?.8 (SCL)
- net SYS_I2C_SCL: now also U?.5 (SCL), U?.5 (SCL)
- net SYS_I2C_SDA: now reaches U?.9 (SDA)
- net SYS_I2C_SDA: now also U?.6 (SDA), U?.6 (SDA)
- net TCP_PPHV2_EN renamed TCP1_PPHV_EN
- net VSYS_SW_DEN renamed VSYS_SOM_DEN
- net VSYS_SW_IN renamed VSYS_SOM_IN
- net VSYS_SW_IS renamed VSYS_SOM_IS
- new net: C?.1, R?.2 (x2)
- new net: C?.2, L?.1, U?.5 (SW) (x5)
- new net: C?.1, C?.1, C?.1, C?.1, C?.2, L?.2, R?.1, U?.1 (IN), U?.1 (IN), U?.1 (VIN), U?.3 (EN), U?.3 (EN), U?.3 (EN)
- new net: C?.1, U?.6 (BST) (x4)
- new net: U?.1 (NC), U?.7 (NC)
- new net: C?.2, C?.2, C?.2, C?.2, U?.4 (GND)
- new net: R?.1, U?.6 (BST)
- new net: R?.1, R?.2, U?.8 (FB)
- new net: C?.1, D?.1 (K), L?.1, U?.6 (LX) (x2)
- new net: C?.1, D?.1 (K), R?.1, R?.1, R?.1, R?.1, U?.8 (VCC)
- new net: C?.1, C?.1, J?.2 (Pin_2), L?.2, R?.1
- new net: R?.1, R?.2, U?.3 (FB) (x2)
- new net: C?.2, U?.1 (BS) (x2)
- new net: C?.2, L?.2, U?.14 (SW2)
- new net: R?.1, R?.2, U?.4 (ADD)
- new net: R?.2, U?.9 (VCC)
- new net: R?.1, U?.13 (BST2)
- new net: R?.1, R?.2, U?.4 (EN)
- new net: C?.2, R?.1
- new net: R?.2, U?.16 (BST1)
- new net: C?.1, R?.1, U?.7 (OC)
- new net: C?.1, L?.1, U?.15 (SW1)
- new net FAN_12V_EN: U?.2 (EN)
- new net FAN_PWM: J?.4 (Pin_4)
- new net FAN_TAC: J?.3 (Pin_3)
- new net HDMI_5V: C?.1, C?.1, L?.2, U?.1 (FB)
- new net HDMI_5V_EN: U?.2 (EN)
- new net ICM_1V8: C?.1, U?.5 (VOUT)
- new net KP_VDD: C?.1, C?.1, L?.2, U?.1 (FB)
- new net OLED_VDD: C?.1, C?.1, L?.2, U?.1 (FB)
- new net OLED_VDD_EN: U?.2 (EN)
- new net OLED_VOLED: C?.1, C?.2, L?.2, R?.1
- new net OLED_VOLED_EN: R?.1, R?.2, U?.4 (EN)
- new net SMEC_VDD: C?.1, U?.5 (OUT)
- new net SMEC_VDDA: C?.1, U?.5 (OUT)
- new net SYS_I2C_ALT: U?.8 (ALT), U?.8 (ALT)
- new net TCP0_PPHV_EN: U?.3 (EN)
- new net VSYS_SOM: U?.10 (OUT), U?.12 (OUT), U?.13 (OUT), U?.14 (OUT), U?.8 (OUT), U?.9 (OUT)
- no-connect marks 9 -> 23
Other:
- note added: "0x62"
- note added: "FAN_12V"
- note added: "HDMI_5V"
- note added: "July 4, 2024 - August 31, 2024"
- note added: "KP_VDD"
- note added: "MP8859 Address Selection - From MP8859 Rev 1.0 VCC-ADD ADD-GND Address NC NC 0x60 499 301 0x62 301 499 0x64 100 NC 0x66"
- note added: "OLED_VDD"
- note added: "OLED_VOLED"
- note added: "SMEC_PREG, SMEC_VDD, SMEC_VDDA, ICM_1V8"
- note added: "SoM Power Switch"
- note added: "TCP0_PPHV"
- note added: "TCP1_PPHV"
- note added: "TCP_VIN_3V3"
- note added: "Type-C Controller Flash - Optional"
- note removed: "July 4, 2024 - August 21, 2024"
- note removed: "Power Switch"
- note removed: "VSYS_LV"
- moved on the sheet: C?, D?, L?, Q?, R?, U?

Commit message: Sep 4, 2024 2
Parts:
- D?: value BAT201M3 -> BAT201M3
Changed lines of the file:
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@@
 			)
 		)
-		(property "Value" " BAT201M3"
+		(property "Value" "BAT201M3"
 			(at 345.694 455.93 0)
 			(effects

Commit message: Sep 5, 2024 2
Parts:
- U4, U5, U6, U7: value TPD4EUSB30 -> TPD4USB_EXT30
Changed lines of the file:
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@@
 			)
 		)
-		(property "Value" "TPD4EUSB30"
+		(property "Value" "TPD4USB_EXT30"
 			(at 772.668 437.134 0)
 			(effects
@@
 			)
 		)
-		(property "Value" "TPD4EUSB30"
+		(property "Value" "TPD4USB_EXT30"
 			(at 749.808 437.134 0)
 			(effects
@@
 			)
 		)
-		(property "Value" "TPD4EUSB30"
+		(property "Value" "TPD4USB_EXT30"
 			(at 749.808 325.374 0)
 			(effects
@@
 			)
 		)
-		(property "Value" "TPD4EUSB30"
+		(property "Value" "TPD4USB_EXT30"
 			(at 772.668 325.374 0)
 			(effects

Commit message: Sep 12, 2024 2
Parts:
- removed C? (x2): 100nF, symbol Device:C_Small
- removed C?: 22uF, symbol Device:C_Small
- removed C?: 2.2uF, symbol Device:C_Small
- removed C? (x2): 1uF, symbol Device:C_Small
- removed C?: 4.7uF, symbol Device:C_Small
- removed D?: SS15, Diode_SMD:D_SMA, symbol Device:D_Schottky_Small_Filled
- removed L?: 13uH, symbol Device:L_Small
- removed R?: 20.7K, symbol Device:R_Small
- removed R?: 10K, symbol Device:R_Small
- removed R?: 1M, symbol Device:R_Small
- removed R?: 100K, symbol Device:R_Small
- removed U?: TLV73333PDBV, Package_TO_SOT_SMD:SOT-23-5, symbol Regulator_Linear:TLV73333PDBV
- removed U?: SY21019, Package_TO_SOT_SMD:SOT-23-6, symbol mediacow:SY21019
- added C? (x3): 10uF, symbol Device:C_Small
- added C? (x4): 22uF, symbol Device:C_Small
- added C? (x2): 100nF, symbol Device:C_Small
- added C?: 1uF, symbol Device:C_Small
- added C?: 22pF, symbol Device:C_Small
- added C?: 10nF, symbol Device:C_Small
- added D?: MMSZ5231BS-7-F, Diode_SMD:D_SOD-323, symbol Device:D_Zener_Small_Filled
- added L?: 2.2uH, symbol Device:L_Small
- added R?: 90K, symbol Device:R_Small
- added R? (x3): 20K, symbol Device:R_Small
- added R?: 100K, symbol Device:R_Small
- added R? (x2): 0, symbol Device:R_Small
- added U?: TPS51386RJNR, VQFN-HR12_RJN_TEX, symbol mediacow:TPS51386RJNR
Connections:
- net GND: now also C?.2, C?.2, C?.2, C?.2, C?.2, C?.2, C?.2, C?.2, C?.2, C?.2, D?.2 (A), R?.2, R?.2, U?.10 (AGND), U?.12 (MODE), U?.2 (PGND)
- net M2_3V3_PG: now also R?.1, U?.3 (PG)
- net SMEC_VDD: now also C?.1, C?.1, U?.1 (IN), U?.1 (VIN), U?.3 (EN), U?.3 (EN), C?.1, C?.1, C?.1, C?.1, L?.2, R?.1, R?.1
- net VSYS: now also C?.1, C?.1, C?.1, C?.1, R?.1, U?.1 (VIN)
- new net: C?.2, R?.1, R?.2, U?.4 (FB)
- new net: C?.1, R?.2, U?.9 (VCC)
- new net: R?.1, U?.8 (VBST)
- new net: C?.1, R?.2 (x2)
- new net: C?.2, L?.1, U?.7 (SW)
- new net: C?.1, D?.1 (K), R?.1, R?.2, U?.11 (EN)
- no-connect marks 23 -> 25
Other:
- note added: "SMEC_VDD, ICM_1V8"
- note removed: "SMEC_PREG, SMEC_VDD, SMEC_VDDA, ICM_1V8"
- moved on the sheet: C?, U?
