File: circuits/mct2/mct2_io.kicad_sch (KiCad schematic)
At the start: 16 parts, among them J4 USB3_A_Stacked, J5 USB3_A_Stacked, J6 USB_A_Stacked, U1 TUSB7340, U2 TPS25221, U6 TPS25221, U7 TPS25221, U8 TPD2EUSB30

Commit message: schem update July 19 2024
Parts:
- removed C1, C2: 100nF, symbol Device:C_Small
- removed J4: USB3_A_Stacked, Connector_USB:USB3_A_Molex_48406-0001_Horizontal_Stacked, symbol Connector:USB3_A_Stacked
- removed J5: USB3_A_Stacked, symbol Connector:USB3_A_Stacked
- removed J6: USB_A_Stacked, symbol Connector:USB_A_Stacked
- removed LF1, LF2: ECMF2-40A100N6, symbol mediacow:ECMF2-40A100N6
- removed R1: 9.09K 1%, symbol Device:R_Small
- removed R2, R6, R7: 80K, symbol Device:R_Small
- removed U1: TUSB7340, Package_DFN_QFN:Texas_S-PWQFN-N100_EP5.5x5.5mm_ThermalVias, symbol Interface_USB:TUSB7340
- removed U2, U6, U7: TPS25221, symbol mediacow:TPS25221
- removed U8: TPD2EUSB30, Package_TO_SOT_SMD:Texas_DRT-3, symbol Power_Protection:TPD2EUSB30

Commit message: July 21, 2024
Parts:
- added SW?: Camera, symbol Switch:SW_SPST
- added SW?: User 1, symbol Switch:SW_SPST
- added SW?: Radio, symbol Switch:SW_SPST
- added SW?: User 3, symbol Switch:SW_SPST
- added SW?: Reset, symbol Switch:SW_SPST
- added SW?: Vol -, symbol Switch:SW_SPST
- added SW?: Power, symbol Switch:SW_SPST
- added SW?: User 2, symbol Switch:SW_SPST
- added SW?: User 4, symbol Switch:SW_SPST
- added SW?: Vol +, symbol Switch:SW_SPST
- added U?: 92HD95, Package_DFN_QFN:QFN-40-1EP_5x5mm_P0.4mm_EP3.6x3.6mm_ThermalVias, symbol mediacow:92HD95

Commit message: July 23, 2024
Parts:
- removed SW?: Camera, symbol Switch:SW_SPST
- removed SW?: User 1, symbol Switch:SW_SPST
- removed SW?: Radio, symbol Switch:SW_SPST
- removed SW?: User 3, symbol Switch:SW_SPST
- removed SW?: Reset, symbol Switch:SW_SPST
- removed SW?: Vol -, symbol Switch:SW_SPST
- removed SW?: Power, symbol Switch:SW_SPST
- removed SW?: User 2, symbol Switch:SW_SPST
- removed SW?: User 4, symbol Switch:SW_SPST
- removed SW?: Vol +, symbol Switch:SW_SPST
- added C? (x2): 120uF, symbol Device:C_Small
- added C? (x10): 100nF, symbol Device:C_Small
- added J? (x2): USB3_A_Stacked, symbol Connector:USB3_A_Stacked
- added J? (x2): USB_A_Stacked, symbol Connector:USB_A_Stacked
- added R? (x8): 100K, symbol Device:R_Small
- added R? (x6): 56K, symbol Device:R_Small
- added R? (x6): 20K, symbol Device:R_Small
- added SW?: Radio, symbol Switch:SW_SPST
- added SW?: Vol -, symbol Switch:SW_Push
- added SW?: User 4, symbol Switch:SW_Push
- added SW?: User 1, symbol Switch:SW_Push
- added SW?: Camera, symbol Switch:SW_SPST
- added SW?: User 2, symbol Switch:SW_Push
- added SW?: User 3, symbol Switch:SW_Push
- added SW?: Vol +, symbol Switch:SW_Push
- added U? (x6): TPS25221, symbol mediacow:TPS25221
- added U?: TCA6408A, symbol mediacow:TCA6408A
- added U? (x2): TPD4EUSB30, Package_SON:USON-10_2.5x1.0mm_P0.5mm, symbol mediacow:TPD4EUSB30
- added U? (x2): TPD4EUSB30, Package_TO_SOT_SMD:Texas_DRT-3, symbol mediacow:TPD2EUSB30
Connections:
- new net: R?.1, U?.5 (ILIM) (x6)
- new net: R?.2, SW?.1 (A), U?.12 (P7)
- new net: R?.2, SW?.1 (A), U?.11 (P6)
- new net: R?.2, SW?.1, U?.10 (P5)
- new net: R?.2, SW?.1, U?.4 (P0)
- new net: R?.2, SW?.1, U?.5 (P1)
- new net: R?.2, SW?.1, U?.6 (P2)
- new net: R?.2, SW?.1, U?.7 (P3)
- new net: R?.2, SW?.1, U?.9 (P4)
- new net EUSB0_DN: J?.2 (D1-), U?.2 (D1-)
- new net EUSB0_DP: J?.3 (D1+), U?.1 (D1+)
- new net EUSB0_EN: R?.1, U?.3 (EN)
- new net EUSB0_FLT: U?.4 (FAULT)
- new net EUSB0_SSRX1N: J?.5 (SSRX1-), U?.2 (D1-)
- new net EUSB0_SSRX1P: J?.6 (SSRX1+), U?.1 (D1+)
- new net EUSB0_SSTX1N: J?.8 (SSTX1-), U?.4 (D2-)
- new net EUSB0_SSTX1P: J?.9 (SSTX1+), U?.3 (GND)
- new net EUSB0_VBUS: C?.1, J?.1 (VBUS1), U?.6 (OUT)
- new net EUSB1_DN: J?.11 (D2-), U?.2 (D1-)
- new net EUSB1_DP: J?.12 (D2+), U?.1 (D1+)
- new net EUSB1_EN: R?.1, U?.3 (EN)
- new net EUSB1_FLT: U?.4 (FAULT)
- new net EUSB1_SSRX1N: J?.14 (SSRX2-), U?.2 (D1-)
- new net EUSB1_SSRX1P: J?.15 (SSRX2+), U?.1 (D1+)
- new net EUSB1_SSTX1N: J?.17 (SSTX2-), U?.4 (D2-)
- new net EUSB1_SSTX1P: J?.18 (SSTX2+), U?.3 (GND)
- new net EUSB1_VBUS: C?.1, J?.10 (VBUS2), U?.6 (OUT)
- new net EUSB2_DN: J?.2 (D1-)
- new net EUSB2_DP: J?.3 (D1+)
- new net EUSB2_EN: R?.1, U?.3 (EN)
- new net EUSB2_FLT: U?.4 (FAULT)
- new net EUSB2_VBUS: C?.1, J?.1 (VBUS1), U?.6 (OUT)
- new net EUSB3_DN: J?.6 (D2-)
- new net EUSB3_DP: J?.7 (D2+)
- new net EUSB3_EN: R?.1, U?.3 (EN)
- new net EUSB3_FLT: U?.4 (FAULT)
- new net EUSB3_VBUS: C?.1, J?.5 (VBUS2), U?.6 (OUT)
- new net EUSB4_DN: J?.2 (D1-)
- new net EUSB4_DP: J?.3 (D1+)
- new net EUSB4_EN: R?.1, U?.3 (EN)
- new net EUSB4_FLT: U?.4 (FAULT)
- new net EUSB4_VBUS: C?.1, J?.1 (VBUS1), U?.6 (OUT)
- new net EUSB5_DN: J?.6 (D2-)
- new net EUSB5_DP: J?.7 (D2+)
- new net EUSB5_EN: R?.1, U?.3 (EN)
- new net EUSB5_FLT: U?.4 (FAULT)
- new net EUSB5_VBUS: C?.1, J?.5 (VBUS2), U?.6 (OUT)
- new net GND: C?.2, C?.2, C?.2, C?.2, C?.2, C?.2, C?.2, C?.2, C?.2, C?.2, C?.2, C?.2, R?.2, R?.2, R?.2, R?.2, R?.2, R?.2, R?.2, R?.2, R?.2, R?.2, R?.2, R?.2, SW?.2, SW?.2, SW?.2, SW?.2, SW?.2, SW?.2, SW?.2 (B), SW?.2 (B), U?.2 (GND), U?.2 (GND), U?.2 (GND), U?.2 (GND), U?.2 (GND), U?.2 (GND), U?.3 (GND), U?.3 (GND), U?.3 (GND), U?.3 (GND), U?.8 (GND), U?.8 (GND), U?.8 (GND)
- new net IOEX_BTN_INT: U?.13 (INT)
- new net IOEX_BTN_RST: U?.3 (RESET)
- new net IOEX_BTN_SCL: U?.14 (SCL)
- new net IOEX_BTN_SDA: U?.15 (SDA)
- new net SMEC_IO_3V3: R?.1, R?.1, R?.1, R?.1, R?.1, R?.1, R?.1, R?.1, U?.16 (VCCP)
- new net USB_5V: C?.1, C?.1, C?.1, C?.1, C?.1, C?.1, U?.1 (IN), U?.1 (IN), U?.1 (IN), U?.1 (IN), U?.1 (IN), U?.1 (IN)
Other:
- moved on the sheet: U?

Commit message: Schematic updates July 25, 2024
Parts:
- added C? (x4): 2.2nF, symbol Device:C_Small
- added C? (x3): 2.2uF, symbol Device:C_Small
- added C? (x2): 1uF, symbol Device:C_Small
- added C?: 10uF, symbol Device:C_Small
- added J?: Internal Speaker Header, Connector_JST:JST_PH_S4B-PH-K_1x04_P2.00mm_Horizontal, symbol Connector:Conn_01x04_Pin
- added R?: 22, symbol Device:R_Small
- added R? (x4): 3.3, symbol Device:R_Small
Connections:
- net GND: now also U?.2 (ADDR), U?.34 (PVSS), U?.35 (PVSS), C?.2, C?.2, C?.2, C?.2, C?.2, R?.2, R?.2, R?.2, R?.2
- net SMEC_IO_3V3: now also U?.1 (VCCI)
- net HDA_SYNC: now reaches U?.10 (SYNC)
- net HDA_RST: now reaches U?.11 (RESET#)
- net HDA_SENSE_A: now reaches U?.13 (SENSE_A)
- net at U?.20 (VrefFilt): now also C?.1
- net at U?.21 (CAP2): now also C?.1
- net HP_L: now reaches U?.23 (PORTA_L)
- net HP_R: now reaches U?.24 (PORTA_R)
- net at U?.25 (VPos): now also C?.1
- net at U?.26 (VNeg): now also C?.1
- net at U?.27 (FCap2): now also C?.2
- net at U?.28 (FCap1): now also C?.1
- net at U?.29 (CPVreg): now also C?.1
- net at U?.32 (PORTD_+L): now also C?.2, J?.1 (Pin_1)
- net at U?.33 (PORTD_-L): now also C?.2, J?.2 (Pin_2)
- net at U?.36 (PORTD_-R): now also C?.2, J?.3 (Pin_3)
- net at U?.37 (PORTD_+R): now also C?.2, J?.4 (Pin_4)
- net HDA_SDOUT: now reaches U?.5 (SDATA_OUT)
- net HDA_BCLK: now reaches U?.6 (BITCLK)
- net at U?.8 (SDATA_IN): now also R?.2
- new net: C?.1, R?.1 (x4)
- new net HDA_SDIN: R?.1
Other:
- note added: "See 92HD95 Reference Schematics document"
- moved on the sheet: C?, R?, SW?, U?

Commit message: July 27, 2024
Parts:
- added U? (x4): TPD4EUSB30, Package_TO_SOT_SMD:Texas_DRT-3, symbol mediacow:TPD2EUSB30
Connections:
- net EUSB2_DN: now also U?.2 (D1-), U?.2 (D1-)
- net EUSB2_DP: now also U?.1 (D1+), U?.1 (D1+)
- net EUSB4_DN: now also U?.2 (D1-), U?.2 (D1-)
- net EUSB4_DP: now also U?.1 (D1+), U?.1 (D1+)
- net GND: now also U?.3 (GND), U?.3 (GND), U?.3 (GND), U?.3 (GND)
Other:
- moved on the sheet: C?, J?, R?, SW?, U?

Commit message: Aug 3, 2024
Parts:
- removed R? (x8): 100K, symbol Device:R_Small
- removed SW?: Radio, symbol Switch:SW_SPST
- removed SW?: Vol -, symbol Switch:SW_Push
- removed SW?: User 4, symbol Switch:SW_Push
- removed SW?: User 1, symbol Switch:SW_Push
- removed SW?: Camera, symbol Switch:SW_SPST
- removed SW?: User 2, symbol Switch:SW_Push
- removed SW?: User 3, symbol Switch:SW_Push
- removed SW?: Vol +, symbol Switch:SW_Push
- removed U?: TCA6408A, symbol mediacow:TCA6408A
- added C? (x3): 4.7uF, symbol Device:C_Small
- added C? (x2): 100nF, symbol Device:C_Small
- added C?: 10nF, symbol Device:C_Small
- added C?: 1uF, symbol Device:C_Small
- added C?: 10uF, symbol Device:C_Small
- added D?: B250A, symbol Device:D_Schottky_Small_Filled
- added J?: Conn_01x24, symbol Connector_Generic:Conn_01x24
- added J?: Conn_01x08, symbol Connector_Generic:Conn_01x08
- added L?: 15uH, symbol Device:L_Small
- added R?: 910K, symbol Device:R_Small
- added R? (x2): 0, symbol Device:R_Small
- added R?: 220K, symbol Device:R_Small
- added R?: 16K, symbol Device:R_Small
- added R? (x2): DNP, symbol Device:R_Small
- added U?: RT6200, Package_TO_SOT_SMD:SOT-23-6, symbol mediacow:RT6200
Connections:
- net GND: now also C?.2, C?.2, C?.2, C?.2, C?.2, C?.2, C?.2, D?.2 (A), J?.1 (Pin_1), J?.2 (Pin_2), J?.24 (Pin_24), J?.3 (Pin_3), R?.1, R?.2, R?.2, R?.2, U?.2 (GND)
- new net: C?.1, C?.1, J?.5 (Pin_5)
- new net: J?.21 (Pin_21), R?.2
- new net: C?.1, C?.1, J?.22 (Pin_22)
- new net: J?.7 (Pin_7), R?.1, R?.2
- new net: C?.2, D?.1 (K), L?.1, U?.6 (PHASE)
- new net: C?.1, U?.1 (BOOT)
- new net: R?.1, R?.2, U?.3 (FB)
- new net: R?.1, R?.2
- new net OLED_CS: J?.8 (Pin_8)
- new net OLED_D0: J?.13 (Pin_13)
- new net OLED_D1: J?.14 (Pin_14)
- new net OLED_D2: J?.15 (Pin_15)
- new net OLED_D3: J?.16 (Pin_16)
- new net OLED_D4: J?.17 (Pin_17)
- new net OLED_D5: J?.18 (Pin_18)
- new net OLED_D6: J?.19 (Pin_19)
- new net OLED_D7: J?.20 (Pin_20)
- new net OLED_DC: J?.10 (Pin_10)
- new net OLED_RD: J?.12 (Pin_12)
- new net OLED_RES: J?.9 (Pin_9)
- new net OLED_VDD: J?.6 (Pin_6), R?.1, R?.1
- new net OLED_VOLED: C?.1, C?.1, J?.23 (Pin_23), L?.2, R?.1
- new net OLED_VOLED_EN: U?.4 (EN)
- new net OLED_WR: J?.11 (Pin_11)
- new net VSB: C?.1, U?.5 (VIN)
- no-connect marks 0 -> 1
Other:
- note added: "12v"
- note added: "CTCL 2021-2024"
- note added: "July 4, 2024 - August 3, 2024"
- note added: "MediaCow Touch 2 - IO Subsystem"

Commit message: Aug 7, 2024 stuff in case I don't work on this before going to FMB
Parts:
- added C?: 1nF, symbol Device:C_Small
- added J?: 8P8C_LED_Shielded, symbol Connector:8P8C_LED_Shielded
- added R? (x4): 75, symbol Device:R_Small
- added T?: ~, symbol mediacow:SM42002EL
- added U?: WGI210AT, Package_DFN_QFN:QFN-64-1EP_9x9mm_P0.5mm_EP3.4x3.4mm, symbol Interface_Ethernet:WGI210AT
Connections:
- net GND: now also C?.2, J?.SH
- new net: J?.1, T?.13 (MX4-)
- new net: J?.2, T?.14 (MX4+)
- new net: R?.1, T?.15 (CT)
- new net: J?.3, T?.16 (MX3-)
- new net: J?.4, T?.17 (MX3+)
- new net: R?.1, T?.18 (CT)
- new net: J?.5, T?.19 (MX2-)
- new net: J?.6, T?.20 (MX2+)
- new net: R?.1, T?.21 (CT)
- new net: J?.7, T?.22 (MX1-)
- new net: J?.8, T?.23 (MX1+)
- new net: R?.1, T?.24 (CT)
- new net: C?.1, R?.2, R?.2, R?.2, R?.2
- new net: U?.10 (VDD3p3), U?.27 (VDD3p3), U?.41 (VDD3p3), U?.64 (VDD3p3)
Other:
- note added: "July 4, 2024 - August 7, 2024"
- note removed: "July 4, 2024 - August 3, 2024"

Commit message: Aug 10, 2024
Parts:
- removed R? (x2): 0, symbol Device:R_Small
- removed R? (x2): DNP, symbol Device:R_Small
- added C?: 10nF, symbol Device:C_Small
- added C? (x4): 22uF, symbol Device:C_Small
- added C?: 39nF, symbol Device:C_Small
- added C? (x12): 100nF, symbol Device:C_Small
- added C? (x3): 10uF, symbol Device:C_Small
- added C?: 22pF, symbol Device:C_Small
- added C? (x3): 15uF, symbol Device:C_Small
- added C? (x2): 27pF, symbol Device:C_Small
- added C?: 1uF, symbol Device:C_Small
- added D?: MMSZ5231BS-7-F, Diode_SMD:D_SOD-323, symbol Device:D_Zener_Small_Filled
- added JP? (x2): ~, symbol Jumper:SolderJumper_3_Open
- added L?: 2.2uH, symbol Device:L_Small
- added R?: 100K, symbol Device:R_Small
- added R? (x2): 0, symbol Device:R_Small
- added R? (x3): 20K, symbol Device:R_Small
- added R?: 150K, symbol Device:R_Small
- added U?: W25Q16JVSS, Package_SO:SOIC-8_5.23x5.23mm_P1.27mm, symbol Memory_Flash:W25Q16JVSS
- added U?: TPS51386RJNR, VQFN-HR12_RJN_TEX, symbol mediacow:TPS51386RJNR
- added Y?: ECS-250-18-33-JGN-TR3, symbol Device:Crystal_GND24
Connections:
- net GND: now also J?.4 (GND1), J?.4 (GND1), J?.8 (GND2), J?.8 (GND2), J?.9 (Shield), J?.9 (Shield), U?.65 (GND), C?.2, C?.2, C?.2, C?.2, C?.2, C?.2, C?.2, C?.2, C?.2, C?.2, C?.2, C?.2, C?.2, C?.2, C?.2, C?.2, C?.2, C?.2, C?.2, C?.2, C?.2, C?.2, C?.2, C?.2, C?.2, D?.2 (A), JP?.1 (A), JP?.1 (A), R?.2, R?.2, U?.10 (AGND), U?.12 (MODE), U?.2 (PGND), U?.4 (GND), Y?.2, Y?.4
- net OLED_VDD: now also JP?.3 (B), JP?.3 (B); no longer J?.6 (Pin_6)
- net USB_5V: now also C?.1, C?.1, C?.1, C?.1, L?.2, R?.1, R?.1
- net at J?.7 (Pin_7): now also JP?.2 (C)
- net LAN_PG: now reaches U?.1 (LAN_PWR_GOOD)
- net LAN_FLSH_MOSI: now reaches U?.12 (NVM_SI)
- net LAN_FLSH_MOSI: now also U?.5 (DI(IO0))
- net LAN_FLSH_CLK: now reaches U?.13 (NVM_SK)
- net LAN_FLSH_CLK: now also U?.6 (CLK)
- net LAN_FLSH_MISO: now reaches U?.14 (NVM_SO)
- net LAN_FLSH_MISO: now also U?.2 (DO(IO1))
- net LAN_FLSH_CS: now reaches U?.15 (~{NVM_CS})
- net LAN_FLSH_CS: now also U?.1 (~{CS})
- net PCIE_LAN_TX_N: now reaches U?.20 (PE_Tn)
- net PCIE_LAN_TX_P: now reaches U?.21 (PE_Tp)
- net PCIE_LAN_RX_N: now reaches U?.23 (PE_Rn)
- net PCIE_LAN_RX_P: now reaches U?.24 (PE_Rp)
- net PCIE_LAN_CLK_N: now reaches U?.25 (PECLKn)
- net PCIE_LAN_CLK_P: now reaches U?.26 (PECLKp)
- net LAN_EN: now reaches U?.28 (~{DEV_OFF})
- net SMB2_SCL: now reaches U?.34 (SMB_CLK)
- net SMB2_ALT: now reaches U?.35 (~{SMB_ALRT})
- net SMB2_SDA: now reaches U?.36 (SMB_DATA)
- net at U?.37 (CBOT): now also C?.1
- net LAN_0V9: now reaches U?.38 (VDD0p9_OUT)
- net LAN_0V9: now also C?.1, C?.1, C?.1, C?.1, C?.1
- net LAN_1V5: now reaches U?.39 (VDD1p5_OUT)
- net LAN_1V5: now also C?.1, C?.1, C?.1
- net at U?.40 (CTOP): now also C?.2
- net at U?.45 (XTAL2): now also C?.1, Y?.1
- net at U?.46 (XTAL1): now also C?.1, Y?.3
- net HDA_PB: now reaches U?.12 (PC_Beep)
- net EUSB0_VBUS: no longer names the net of C?.1, J?.1 (VBUS1), U?.6 (OUT)
- net EUSB1_VBUS: no longer names the net of C?.1, J?.10 (VBUS2), U?.6 (OUT)
- net EUSB2_VBUS: no longer names the net of C?.1, J?.1 (VBUS1), U?.6 (OUT)
- net EUSB3_VBUS: no longer names the net of C?.1, J?.5 (VBUS2), U?.6 (OUT)
- net EUSB4_VBUS: no longer names the net of C?.1, J?.1 (VBUS1), U?.6 (OUT)
- net EUSB5_VBUS: no longer names the net of C?.1, J?.5 (VBUS2), U?.6 (OUT)
- new net: C?.1, D?.1 (K), R?.1, R?.2, U?.11 (EN)
- new net: R?.1, U?.3 (PG)
- new net: C?.1, R?.2, U?.9 (VCC)
- new net: R?.1, U?.8 (VBST)
- new net: C?.1, R?.2 (x2)
- new net: J?.6 (Pin_6), JP?.2 (C)
- new net: C?.2, R?.1, R?.2, U?.4 (FB)
- new net: C?.2, L?.1, U?.7 (SW)
- new net VSYS: C?.1, C?.1, C?.1, C?.1, R?.1, U?.1 (VIN)
- no-connect marks 1 -> 4
Other:
- note added: "July 4, 2024 - August 9, 2024"
- note removed: "July 4, 2024 - August 7, 2024"
- moved on the sheet: C?, D?, J?, J?A, J?B, L?, R?, T?, U?
