File: circuits/mct2/mct2_io.kicad_sch (KiCad schematic)
At the start: 198 parts

Commit message: Aug 26, 2024
Parts:
- removed C?: 2.2uF, symbol Device:C_Small
- removed C?: 22uF, symbol Device:C_Small
- removed C?: 100nF, symbol Device:C_Small
- removed D?: SS15, Diode_SMD:D_SMA, symbol Device:D_Schottky_Small_Filled
- removed L?: 15uH, symbol Device:L_Small
- removed R?: 100K, symbol Device:R_Small
- removed R?: 10K, symbol Device:R_Small
- removed R?: 1M, symbol Device:R_Small
- removed R?: 13.7K, symbol Device:R_Small
- removed U?: SY21019, Package_TO_SOT_SMD:SOT-23-6, symbol mediacow:SY21019
Connections:
- net HDMI_5V is gone; now on net VSYS_LV: C?.1, C?.2, U?.10 (VCC5V)
Other:
- note added: "July 4, 2024 - August 26, 2024"
- note removed: "July 4, 2024 - August 21, 2024"

Commit message: Aug 31, 2024
Parts:
- removed C? (x7): 100nF, symbol Device:C_Small
- removed C?: 330nF, symbol Device:C_Small
- removed C? (x3): 4.7uF, symbol Device:C_Small
- removed C? (x3): 2.2uF, symbol Device:C_Small
- removed C? (x3): 22uF, symbol Device:C_Small
- removed C? (x2): 10uF, symbol Device:C_Small
- removed C?: 22pF, symbol Device:C_Small
- removed D? (x3): SS15, Diode_SMD:D_SMA, symbol Device:D_Schottky_Small_Filled
- removed J?: Conn_01x08, symbol Connector_Generic:Conn_01x08
- removed L?: 2.2uF, symbol Device:L_Small
- removed L? (x3): 15uH, symbol Device:L_Small
- removed R?: 430k, symbol Device:R_Small
- removed R? (x3): 1M, symbol Device:R_Small
- removed R?: 5.23K, symbol Device:R_Small
- removed R? (x3): 10K, symbol Device:R_Small
- removed R? (x2): 22.1K, symbol Device:R_Small
- removed R? (x5): 100K, symbol Device:R_Small
- removed U?: L78L33_SO8, Package_SO:SOIC-8_3.9x4.9mm_P1.27mm, symbol Regulator_Linear:L78L33_SO8
- removed U? (x3): SY21019, Package_TO_SOT_SMD:SOT-23-6, symbol mediacow:SY21019
- removed U?: AP3401DN, mediacow:Diodes_U-DFN2020-6_Type_J, symbol mediacow:AP3401DN
- added C? (x2): 22uF, symbol Device:C_Small
- added C?: 100nF, symbol Device:C_Small
- added C?: 10uF, symbol Device:C_Small
- added L?: 3.9uH, symbol Device:L_Small
- added U?: AP63203, Package_TO_SOT_SMD:TSOT-23-6, symbol mediacow:AP63203WU
- D?: value D_Schottky_Small_Filled -> BAT201M3; footprint (none) -> Diode_SMD:D_SOD-323F
Connections:
- net GND: now also C?.2, C?.2, C?.2, U?.4 (GND)
- net LAN_3V3: now also C?.1, C?.1, L?.2, U?.1 (FB)
- net DDIB_CEC_CN: now reaches J?.13 (CEC)
- net DDIB_CEC_CN: now also U?.6 (CEC_B)
- net KP_VDD: now reaches J?.1 (Pin_1)
- net DDIB_CEC: now reaches U?.24 (CEC_A)
- net SMEC_3V3_IO renamed SMEC_VDD
- net VSYS_LV: no longer names the net of C?.1, C?.2, U?.10 (VCC5V)
- new net: C?.1, U?.6 (BST)
- new net: C?.2, L?.1, U?.5 (SW)
- new net LAN_3V3_EN: U?.2 (EN)
- new net VSYS: C?.1, U?.3 (VIN)
- no-connect marks 50 -> 47
Other:
- note added: "July 4, 2024 - August 31, 2024"
- note removed: "July 4, 2024 - August 26, 2024"
- moved on the sheet: C?, J?, JP?, L?, NT?, R?, U?

Commit message: Sep 4, 2024 2
Parts:
- D?: value BAT201M3 -> BAT201M3
Changed lines of the file:
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@@
 			)
 		)
-		(property "Value" " BAT201M3"
+		(property "Value" "BAT201M3"
 			(at 835.914 477.52 0)
 			(effects

Commit message: Sep 5, 2024 1
Other:
- note added: "MediaCow Touch 2 - IO"
- note removed: "MediaCow Touch 2 - System"
Changed lines of the file:
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@@
 		)
 	)
-	(text "MediaCow Touch 2 - System"
+	(text "MediaCow Touch 2 - IO"
 		(exclude_from_sim no)
 		(at 1098.042 820.674 0)

Commit message: Sep 5, 2024 2
Parts:
- U? (x7): value TPD4EUSB30 -> TPD4USB_EXT30
Connections:
- net EUSB0_DN renamed USB_EXT0_DN
- net EUSB0_DP renamed USB_EXT0_DP
- net EUSB0_EN renamed USB_EXT0_EN
- net EUSB0_FLT renamed USB_EXT0_FLT
- net EUSB0_SSRX1N renamed USB_EXT0_SSRX1N
- net EUSB0_SSRX1P renamed USB_EXT0_SSRX1P
- net EUSB0_SSTX1N renamed USB_EXT0_SSTX1N
- net EUSB0_SSTX1P renamed USB_EXT0_SSTX1P
- net EUSB1_DN renamed USB_EXT1_DN
- net EUSB1_DP renamed USB_EXT1_DP
- net EUSB1_EN renamed USB_EXT1_EN
- net EUSB1_FLT renamed USB_EXT1_FLT
- net EUSB1_SSRX1N renamed USB_EXT1_SSRX1N
- net EUSB1_SSRX1P renamed USB_EXT1_SSRX1P
- net EUSB1_SSTX1N renamed USB_EXT1_SSTX1N
- net EUSB1_SSTX1P renamed USB_EXT1_SSTX1P
- net EUSB2_DN renamed USB_EXT2_DN
- net EUSB2_DP renamed USB_EXT2_DP
- net EUSB2_EN renamed USB_EXT2_EN
- net EUSB2_FLT renamed USB_EXT2_FLT
- net EUSB3_DN renamed USB_EXT3_DN
- net EUSB3_DP renamed USB_EXT3_DP
- net EUSB3_EN renamed USB_EXT3_EN
- net EUSB3_FLT renamed USB_EXT3_FLT
Changed lines of the file:
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@@
 		)
 	)
-	(global_label "EUSB3_FLT"
+	(global_label "USB_EXT3_FLT"
 		(shape input)
 		(at 1057.91 189.23 0)
@@
 		)
 	)
-	(global_label "EUSB1_EN"
+	(global_label "USB_EXT1_EN"
 		(shape input)
 		(at 1021.08 116.84 180)
@@
 		)
 	)
-	(global_label "EUSB0_SSTX1P"
+	(global_label "USB_EXT0_SSTX1P"
 		(shape input)
 		(at 1078.23 68.58 180)
@@
 		)
 	)
-	(global_label "EUSB0_SSTX1N"
+	(global_label "USB_EXT0_SSTX1N"
 		(shape input)
 		(at 1078.23 66.04 180)
@@
 		)
 	)
-	(global_label "EUSB1_SSRX1P"
+	(global_label "USB_EXT1_SSRX1P"
 		(shape input)
 		(at 1080.77 127 180)
@@
 		)
 	)
-	(global_label "EUSB2_EN"
+	(global_label "USB_EXT2_EN"
 		(shape input)
 		(at 1021.08 166.37 180)
@@
 		)
 	)
-	(global_label "EUSB2_FLT"
+	(global_label "USB_EXT2_FLT"
 		(shape input)
 		(at 1057.91 166.37 0)
@@
 		)
 	)
-	(global_label "EUSB0_DP"
+	(global_label "USB_EXT0_DP"
 		(shape input)
 		(at 1109.98 53.34 180)
@@
 		)
 	)
-	(global_label "EUSB1_SSRX1N"
+	(global_label "USB_EXT1_SSRX1N"
 		(shape input)
 		(at 1080.77 124.46 180)
@@
 		)
 	)
-	(global_label "EUSB1_SSTX1P"
+	(global_label "USB_EXT1_SSTX1P"
 		(shape input)
 		(at 1080.77 134.62 180)
@@
 		)
 	)
-	(global_label "EUSB1_DN"
+	(global_label "USB_EXT1_DN"
 		(shape input)
 		(at 1112.52 116.84 180)
@@
 		)
 	)
-	(global_label "EUSB0_FLT"
+	(global_label "USB_EXT0_FLT"
 		(shape input)
 		(at 1057.91 50.8 0)
@@
 		)
 	)
-	(global_label "EUSB1_FLT"
+	(global_label "USB_EXT1_FLT"
 		(shape input)
 		(at 1057.91 116.84 0)
@@
 		)
 	)
-	(global_label "EUSB0_SSRX1P"
+	(global_label "USB_EXT0_SSRX1P"
 		(shape input)
 		(at 1078.23 60.96 180)
@@
 		)
 	)
-	(global_label "EUSB2_DN"
+	(global_label "USB_EXT2_DN"
 		(shape input)
 		(at 1096.01 181.61 180)
@@
 		)
 	)
-	(global_label "EUSB0_DN"
+	(global_label "USB_EXT0_DN"
 		(shape input)
 		(at 1109.98 50.8 180)
@@
 		)
 	)
-	(global_label "EUSB1_SSTX1N"
+	(global_label "USB_EXT1_SSTX1N"
 		(shape input)
 		(at 1080.77 132.08 180)
@@
 		)
 	)
-	(global_label "EUSB2_DP"
+	(global_label "USB_EXT2_DP"
 		(shape input)
 		(at 1096.01 179.07 180)
@@
 		)
 	)
-	(global_label "EUSB3_DN"
+	(global_label "USB_EXT3_DN"
 		(shape input)
 		(at 1096.01 186.69 180)
@@
 		)
 	)
-	(global_label "EUSB0_EN"
+	(global_label "USB_EXT0_EN"
 		(shape input)
 		(at 1021.08 50.8 180)
@@
 		)
 	)
-	(global_label "EUSB3_EN"
+	(global_label "USB_EXT3_EN"
 		(shape input)
 		(at 1021.08 189.23 180)
@@
 		)
 	)
-	(global_label "EUSB1_DP"
+	(global_label "USB_EXT1_DP"
 		(shape input)
 		(at 1112.52 119.38 180)
@@
 		)
 	)
-	(global_label "EUSB3_DP"
+	(global_label "USB_EXT3_DP"
 		(shape input)
 		(at 1096.01 184.15 180)
@@
 		)
 	)
-	(global_label "EUSB0_SSRX1N"
+	(global_label "USB_EXT0_SSRX1N"
 		(shape input)
 		(at 1078.23 58.42 180)
@@
 			)
 		)
-		(property "Value" "TPD4EUSB30"
+		(property "Value" "TPD4USB_EXT30"
 			(at 960.12 284.48 0)
 			(effects
@@
 			)
 		)
-		(property "Value" "TPD4EUSB30"
+		(property "Value" "TPD4USB_EXT30"
 			(at 1131.316 139.954 0)
 			(effects
@@
 			)
 		)
-		(property "Value" "TPD4EUSB30"
+		(property "Value" "TPD4USB_EXT30"
 			(at 1127.76 190.5 0)
 			(effects
@@
 			)
 		)
-		(property "Value" "TPD4EUSB30"
+		(property "Value" "TPD4USB_EXT30"
 			(at 1131.824 96.774 0)
 			(effects
@@
 			)
 		)
-		(property "Value" "TPD4EUSB30"
+		(property "Value" "TPD4USB_EXT30"
 			(at 1131.316 73.914 0)
 			(effects
@@
 			)
 		)
-		(property "Value" "TPD4EUSB30"
+		(property "Value" "TPD4USB_EXT30"
 			(at 1129.284 30.734 0)
 			(effects
@@
 			)
 		)
-		(property "Value" "TPD4EUSB30"
+		(property "Value" "TPD4USB_EXT30"
 			(at 1109.98 190.5 0)
 			(effects

Commit message: Sep 12, 2024 2
Parts:
- removed C? (x2): 4.7uF, symbol Device:C_Small
- removed C? (x2): 100nF, symbol Device:C_Small
- removed C?: 1uF, symbol Device:C_Small
- removed J?: Conn_01x24, symbol Connector_Generic:Conn_01x24
- removed J?: Conn_01x08, symbol Connector_Generic:Conn_01x08
- removed JP?: ~, symbol Jumper:SolderJumper_3_Open
- removed R?: 910K, symbol Device:R_Small
Connections:
- no-connect marks 47 -> 46
Other:
- note added: "July 4, 2024 - September 12, 2024"
- note removed: "July 4, 2024 - August 31, 2024"
- note removed: "OLED_VDD: 80XX GND: 68XX"
- moved on the sheet: C?, J?, L?, R?, U?
