File: circuits/mct2/mct2.kicad_sch (KiCad schematic)
At the start: 16 parts

Commit message: Aug 17, 2024
Parts:
- removed D?: D_Schottky_Small_Filled, symbol Device:D_Schottky_Small_Filled
Connections:
- net SOM_IO_3V3: now also C?.1, C?.1, R?.2, U?. (VCC)
- net PCIE_NVME_REF_N renamed PCIE_M2M_REF_N
- net PCIE_NVME_REF_P renamed PCIE_M2M_REF_P
- net PCIE_NVME_RX0_N renamed PCIE_M2M_RX0_N
- net PCIE_NVME_RX0_P renamed PCIE_M2M_RX0_P
- net PCIE_NVME_RX1_N renamed PCIE_M2M_RX1_N
- net PCIE_NVME_RX1_P renamed PCIE_M2M_RX1_P
- net PCIE_NVME_RX2_N renamed PCIE_M2M_RX2_N
- net PCIE_NVME_RX2_P renamed PCIE_M2M_RX2_P
- net PCIE_NVME_RX3_N renamed PCIE_M2M_RX3_N
- net PCIE_NVME_RX3_P renamed PCIE_M2M_RX3_P
- net PCIE_NVME_TX0_N renamed PCIE_M2M_TX0_N
- net PCIE_NVME_TX0_P renamed PCIE_M2M_TX0_P
- net PCIE_NVME_TX1_N renamed PCIE_M2M_TX1_N
- net PCIE_NVME_TX1_P renamed PCIE_M2M_TX1_P
- net PCIE_NVME_TX2_N renamed PCIE_M2M_TX2_N
- net PCIE_NVME_TX2_P renamed PCIE_M2M_TX2_P
- net PCIE_NVME_TX3_N renamed PCIE_M2M_TX3_N
- net PCIE_NVME_TX3_P renamed PCIE_M2M_TX3_P
- net SMB3_ALT renamed SML_ALT
- net SMB3_SCL renamed SML_SCL
- net SMB3_SDA renamed SML_SDA
- net USB_EXT3_N: no longer names the net of A1.79 (USB2_P3-)
- net USB_EXT3_P: no longer names the net of A1.81 (USB2_P3+)
- net USB_EXT4_N: no longer names the net of A1.72 (USB2_P4-)
- net USB_EXT4_P: no longer names the net of A1.70 (USB2_P4+)
- no-connect marks 8 -> 12

Commit message: Aug 17, 2024 2
Changed lines of the file:
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@@
 		(at 501.65 537.21)
 	)
+	(bus_entry
+		(at 659.13 516.89)
+		(size 2.54 2.54)
+		(stroke
+			(width 0)
+			(type default)
+		)
+	)
 	(wire
 		(pts
@@
 	(wire
 		(pts
-			(xy 499.11 381) (xy 501.65 381)
+			(xy 477.52 381) (xy 501.65 381)
 		)
 		(stroke
@@
 	(wire
 		(pts
-			(xy 499.11 388.62) (xy 501.65 388.62)
+			(xy 477.52 388.62) (xy 501.65 388.62)
 		)
 		(stroke
@@
 	(wire
 		(pts
-			(xy 499.11 393.7) (xy 501.65 393.7)
+			(xy 477.52 393.7) (xy 501.65 393.7)
 		)
 		(stroke
@@
 	(wire
 		(pts
-			(xy 499.11 403.86) (xy 501.65 403.86)
+			(xy 477.52 403.86) (xy 501.65 403.86)
 		)
 		(stroke
@@
 	(wire
 		(pts
-			(xy 499.11 365.76) (xy 501.65 365.76)
+			(xy 477.52 365.76) (xy 501.65 365.76)
 		)
 		(stroke
@@
 	(wire
 		(pts
-			(xy 499.11 398.78) (xy 501.65 398.78)
+			(xy 477.52 398.78) (xy 501.65 398.78)
 		)
 		(stroke
@@
 	(wire
 		(pts
-			(xy 499.11 401.32) (xy 501.65 401.32)
+			(xy 477.52 401.32) (xy 501.65 401.32)
 		)
 		(stroke
@@
 	(wire
 		(pts
-			(xy 499.11 368.3) (xy 501.65 368.3)
+			(xy 477.52 368.3) (xy 501.65 368.3)
 		)
 		(stroke
@@
 	(wire
 		(pts
-			(xy 499.11 375.92) (xy 501.65 375.92)
+			(xy 477.52 375.92) (xy 501.65 375.92)
 		)
 		(stroke
@@
 	(wire
 		(pts
-			(xy 499.11 370.84) (xy 501.65 370.84)
+			(xy 477.52 370.84) (xy 501.65 370.84)
 		)
 		(stroke
@@
 	(wire
 		(pts
-			(xy 499.11 386.08) (xy 501.65 386.08)
+			(xy 477.52 386.08) (xy 501.65 386.08)
 		)
 		(stroke
@@
 	(wire
 		(pts
-			(xy 499.11 391.16) (xy 501.65 391.16)
+			(xy 477.52 391.16) (xy 501.65 391.16)
 		)
 		(stroke
@@
 	(wire
 		(pts
-			(xy 499.11 373.38) (xy 501.65 373.38)
+			(xy 477.52 373.38) (xy 501.65 373.38)
 		)
 		(stroke
@@
 	(wire
 		(pts
-			(xy 499.11 378.46) (xy 501.65 378.46)
+			(xy 477.52 378.46) (xy 501.65 378.46)
 		)
 		(stroke
@@
 	(wire
 		(pts
-			(xy 499.11 383.54) (xy 501.65 383.54)
+			(xy 477.52 383.54) (xy 501.65 383.54)
 		)
 		(stroke
@@
 	(wire
 		(pts
-			(xy 499.11 396.24) (xy 501.65 396.24)
+			(xy 477.52 396.24) (xy 501.65 396.24)
 		)
 		(stroke
@@
 	(global_label "SSUSB1_RXN"
 		(shape input)
-		(at 499.11 383.54 180)
+		(at 477.52 383.54 180)
 		(fields_autoplaced yes)
 		(effects
@@
 		)
 		(property "Intersheetrefs" "${INTERSHEET_REFS}"
-			(at 483.9087 383.54 0)
+			(at 462.3187 383.54 0)
 			(effects
 				(font
@@
 	(global_label "PCIE_M2E_TX0_P"
 		(shape input)
-		(at 499.11 386.08 180)
+		(at 477.52 386.08 180)
 		(fields_autoplaced yes)
 		(effects
@@
 		)
 		(property "Intersheetrefs" "${INTERSHEET_REFS}"
-			(at 483.1226 386.08 0)
+			(at 461.5326 386.08 0)
 			(effects
 				(font
@@
 	(global_label "PCIE_M2E_RX0_P"
 		(shape input)
-		(at 499.11 391.16 180)
+		(at 477.52 391.16 180)
 		(fields_autoplaced yes)
 		(effects
@@
 		)
 		(property "Intersheetrefs" "${INTERSHEET_REFS}"
-			(at 482.8202 391.16 0)
+			(at 461.2302 391.16 0)
 			(effects
 				(font
@@
 	(global_label "PCIE_M2E_TX0_N"
 		(shape input)
-		(at 499.11 388.62 180)
+		(at 477.52 388.62 180)
 		(fields_autoplaced yes)
 		(effects
@@
 		)
 		(property "Intersheetrefs" "${INTERSHEET_REFS}"
-			(at 483.0621 388.62 0)
+			(at 461.4721 388.62 0)
 			(effects
 				(font
@@
 	(global_label "SSUSB1_TXP"
 		(shape input)
-		(at 499.11 375.92 180)
+		(at 477.52 375.92 180)
 		(fields_autoplaced yes)
 		(effects
@@
 		)
 		(property "Intersheetrefs" "${INTERSHEET_REFS}"
-			(at 484.2716 375.92 0)
+			(at 462.6816 375.92 0)
 			(effects
 				(font
@@
 	(global_label "SSUSB1_RXP"
 		(shape input)
-		(at 499.11 381 180)
+		(at 477.52 381 180)
 		(fields_autoplaced yes)
 		(effects
@@
 		)
 		(property "Intersheetrefs" "${INTERSHEET_REFS}"
-			(at 484.2716 381 0)
+			(at 462.6816 381 0)
 			(effects
 				(font
@@
 	(global_label "PCIE_LAN_RX0_P"
 		(shape input)
-		(at 499.11 401.32 180)
+		(at 477.52 401.32 180)
 		(fields_autoplaced yes)
 		(effects
@@
 		)
 		(property "Intersheetrefs" "${INTERSHEET_REFS}"
-			(at 482.8202 401.32 0)
+			(at 461.2302 401.32 0)
 			(effects
 				(font
@@
 	(global_label "SSUSB0_TXP"
 		(shape input)
-		(at 499.11 368.3 180)
+		(at 477.52 368.3 180)
 		(fields_autoplaced yes)
 		(effects
@@
 		)
 		(property "Intersheetrefs" "${INTERSHEET_REFS}"
-			(at 484.2716 368.3 0)
+			(at 462.6816 368.3 0)
 			(effects
 				(font
@@
 	(global_label "SSUSB0_RXN"
 		(shape input)
-		(at 499.11 373.38 180)
+		(at 477.52 373.38 180)
 		(fields_autoplaced yes)
 		(effects
@@
 		)
 		(property "Intersheetrefs" "${INTERSHEET_REFS}"
-			(at 483.9087 373.38 0)
+			(at 462.3187 373.38 0)
 			(effects
 				(font
@@
 	(global_label "PCIE_LAN_TX0_P"
 		(shape input)
-		(at 499.11 396.24 180)
+		(at 477.52 396.24 180)
 		(fields_autoplaced yes)
 		(effects
@@
 		)
 		(property "Intersheetrefs" "${INTERSHEET_REFS}"
-			(at 483.1226 396.24 0)
+			(at 461.5326 396.24 0)
 			(effects
 				(font
@@
 	(global_label "SSUSB0_TXP"
 		(shape input)
-		(at 499.11 365.76 180)
+		(at 477.52 365.76 180)
 		(fields_autoplaced yes)
 		(effects
@@
 		)
 		(property "Intersheetrefs" "${INTERSHEET_REFS}"
-			(at 484.2716 365.76 0)
+			(at 462.6816 365.76 0)
 			(effects
 				(font
@@
 	(global_label "PCIE_M2E_RX0_N"
 		(shape input)
-		(at 499.11 393.7 180)
+		(at 477.52 393.7 180)
 		(fields_autoplaced yes)
 		(effects
@@
 		)
 		(property "Intersheetrefs" "${INTERSHEET_REFS}"
-			(at 482.7597 393.7 0)
+			(at 461.1697 393.7 0)
 			(effects
 				(font
@@
 	(global_label "PCIE_LAN_RX0_N"
 		(shape input)
-		(at 499.11 403.86 180)
+		(at 477.52 403.86 180)
 		(fields_autoplaced yes)
 		(effects
@@
 		)
 		(property "Intersheetrefs" "${INTERSHEET_REFS}"
-			(at 482.7597 403.86 0)
+			(at 461.1697 403.86 0)
 			(effects
 				(font
@@
 	(global_label "SSUSB0_RXP"
 		(shape input)
-		(at 499.11 370.84 180)
+		(at 477.52 370.84 180)
 		(fields_autoplaced yes)
 		(effects
@@
 		)
 		(property "Intersheetrefs" "${INTERSHEET_REFS}"
-			(at 484.2716 370.84 0)
+			(at 462.6816 370.84 0)
 			(effects
 				(font
@@
 	(global_label "SSUSB1_TXN"
 		(shape input)
-		(at 499.11 378.46 180)
+		(at 477.52 378.46 180)
 		(fields_autoplaced yes)
 		(effects
@@
 		)
 		(property "Intersheetrefs" "${INTERSHEET_REFS}"
-			(at 484.2111 378.46 0)
+			(at 462.6211 378.46 0)
 			(effects
 				(font
@@
 	(global_label "PCIE_LAN_TX0_N"
 		(shape input)
-		(at 499.11 398.78 180)
+		(at 477.52 398.78 180)
 		(fields_autoplaced yes)
 		(effects
@@
 		)
 		(property "Intersheetrefs" "${INTERSHEET_REFS}"
-			(at 483.0621 398.78 0)
+			(at 461.4721 398.78 0)
 			(effects
 				(font

Commit message: Aug 19, 2024
Changed lines of the file:
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@@
 		(at 501.65 537.21)
 	)
-	(bus_entry
-		(at 659.13 516.89)
-		(size 2.54 2.54)
-		(stroke
-			(width 0)
-			(type default)
-		)
-	)
 	(wire
 		(pts
@@
 	(wire
 		(pts
-			(xy 499.11 414.02) (xy 501.65 414.02)
+			(xy 477.52 414.02) (xy 501.65 414.02)
 		)
 		(stroke
@@
 	(wire
 		(pts
-			(xy 499.11 411.48) (xy 501.65 411.48)
+			(xy 477.52 411.48) (xy 501.65 411.48)
 		)
 		(stroke
@@
 	(wire
 		(pts
-			(xy 499.11 408.94) (xy 501.65 408.94)
+			(xy 477.52 408.94) (xy 501.65 408.94)
 		)
 		(stroke
@@
 	(wire
 		(pts
-			(xy 499.11 419.1) (xy 501.65 419.1)
+			(xy 477.52 419.1) (xy 501.65 419.1)
 		)
 		(stroke
@@
 	(wire
 		(pts
-			(xy 499.11 431.8) (xy 501.65 431.8)
+			(xy 477.52 431.8) (xy 501.65 431.8)
 		)
 		(stroke
@@
 	(wire
 		(pts
-			(xy 499.11 416.56) (xy 501.65 416.56)
+			(xy 477.52 416.56) (xy 501.65 416.56)
 		)
 		(stroke
@@
 	(wire
 		(pts
-			(xy 499.11 424.18) (xy 501.65 424.18)
+			(xy 477.52 424.18) (xy 501.65 424.18)
 		)
 		(stroke
@@
 	(wire
 		(pts
-			(xy 499.11 439.42) (xy 501.65 439.42)
+			(xy 477.52 439.42) (xy 501.65 439.42)
 		)
 		(stroke
@@
 	(wire
 		(pts
-			(xy 499.11 444.5) (xy 501.65 444.5)
+			(xy 477.52 444.5) (xy 501.65 444.5)
 		)
 		(stroke
@@
 	(wire
 		(pts
-			(xy 499.11 421.64) (xy 501.65 421.64)
+			(xy 477.52 421.64) (xy 501.65 421.64)
 		)
 		(stroke
@@
 	(wire
 		(pts
-			(xy 499.11 447.04) (xy 501.65 447.04)
+			(xy 477.52 447.04) (xy 501.65 447.04)
 		)
 		(stroke
@@
 	(wire
 		(pts
-			(xy 499.11 426.72) (xy 501.65 426.72)
+			(xy 477.52 426.72) (xy 501.65 426.72)
 		)
 		(stroke
@@
 	(wire
 		(pts
-			(xy 499.11 441.96) (xy 501.65 441.96)
+			(xy 477.52 441.96) (xy 501.65 441.96)
 		)
 		(stroke
@@
 	(wire
 		(pts
-			(xy 499.11 434.34) (xy 501.65 434.34)
+			(xy 477.52 434.34) (xy 501.65 434.34)
 		)
 		(stroke
@@
 	(wire
 		(pts
-			(xy 499.11 429.26) (xy 501.65 429.26)
+			(xy 477.52 429.26) (xy 501.65 429.26)
 		)
 		(stroke
@@
 	(wire
 		(pts
-			(xy 499.11 436.88) (xy 501.65 436.88)
+			(xy 477.52 436.88) (xy 501.65 436.88)
 		)
 		(stroke
@@
 	(global_label "PCIE_M2M_TX0_P"
 		(shape input)
-		(at 499.11 408.94 180)
+		(at 477.52 408.94 180)
 		(fields_autoplaced yes)
 		(effects
@@
 		)
 		(property "Intersheetrefs" "${INTERSHEET_REFS}"
-			(at 479.2521 408.94 0)
+			(at 457.6621 408.94 0)
 			(effects
 				(font
@@
 	(global_label "PCIE_M2M_RX1_N"
 		(shape input)
-		(at 499.11 426.72 180)
+		(at 477.52 426.72 180)
 		(fields_autoplaced yes)
 		(effects
@@
 		)
 		(property "Intersheetrefs" "${INTERSHEET_REFS}"
-			(at 478.8892 426.72 0)
+			(at 457.2992 426.72 0)
 			(effects
 				(font
@@
 	(global_label "PCIE_M2M_TX0_N"
 		(shape input)
-		(at 499.11 411.48 180)
+		(at 477.52 411.48 180)
 		(fields_autoplaced yes)
 		(effects
@@
 		)
 		(property "Intersheetrefs" "${INTERSHEET_REFS}"
-			(at 479.1916 411.48 0)
+			(at 457.6016 411.48 0)
 			(effects
 				(font
@@
 	(global_label "PCIE_M2M_RX3_N"
 		(shape input)
-		(at 499.11 447.04 180)
+		(at 477.52 447.04 180)
 		(fields_autoplaced yes)
 		(effects
@@
 		)
 		(property "Intersheetrefs" "${INTERSHEET_REFS}"
-			(at 478.8892 447.04 0)
+			(at 457.2992 447.04 0)
 			(effects
 				(font
@@
 	(global_label "PCIE_M2M_RX2_N"
 		(shape input)
-		(at 499.11 436.88 180)
+		(at 477.52 436.88 180)
 		(fields_autoplaced yes)
 		(effects
@@
 		)
 		(property "Intersheetrefs" "${INTERSHEET_REFS}"
-			(at 478.8892 436.88 0)
+			(at 457.2992 436.88 0)
 			(effects
 				(font
@@
 	(global_label "PCIE_M2M_TX3_N"
 		(shape input)
-		(at 499.11 441.96 180)
+		(at 477.52 441.96 180)
 		(fields_autoplaced yes)
 		(effects
@@
 		)
 		(property "Intersheetrefs" "${INTERSHEET_REFS}"
-			(at 479.1916 441.96 0)
+			(at 457.6016 441.96 0)
 			(effects
 				(font
@@
 	(global_label "PCIE_M2M_TX1_N"
 		(shape input)
-		(at 499.11 421.64 180)
+		(at 477.52 421.64 180)
 		(fields_autoplaced yes)
 		(effects
@@
 		)
 		(property "Intersheetrefs" "${INTERSHEET_REFS}"
-			(at 479.1916 421.64 0)
+			(at 457.6016 421.64 0)
 			(effects
 				(font
@@
 	(global_label "PCIE_M2M_TX2_N"
 		(shape input)
-		(at 499.11 431.8 180)
+		(at 477.52 431.8 180)
 		(fields_autoplaced yes)
 		(effects
@@
 		)
 		(property "Intersheetrefs" "${INTERSHEET_REFS}"
-			(at 479.1916 431.8 0)
+			(at 457.6016 431.8 0)
 			(effects
 				(font
@@
 	(global_label "PCIE_M2M_RX0_P"
 		(shape input)
-		(at 499.11 414.02 180)
+		(at 477.52 414.02 180)
 		(fields_autoplaced yes)
 		(effects
@@
 		)
 		(property "Intersheetrefs" "${INTERSHEET_REFS}"
-			(at 478.9497 414.02 0)
+			(at 457.3597 414.02 0)
 			(effects
 				(font
@@
 	(global_label "PCIE_M2M_RX2_P"
 		(shape input)
-		(at 499.11 434.34 180)
+		(at 477.52 434.34 180)
 		(fields_autoplaced yes)
 		(effects
@@
 		)
 		(property "Intersheetrefs" "${INTERSHEET_REFS}"
-			(at 478.9497 434.34 0)
+			(at 457.3597 434.34 0)
 			(effects
 				(font
@@
 	(global_label "PCIE_M2M_RX3_P"
 		(shape input)
-		(at 499.11 444.5 180)
+		(at 477.52 444.5 180)
 		(fields_autoplaced yes)
 		(effects
@@
 		)
 		(property "Intersheetrefs" "${INTERSHEET_REFS}"
-			(at 478.9497 444.5 0)
+			(at 457.3597 444.5 0)
 			(effects
 				(font
@@
 	(global_label "PCIE_M2M_TX3_P"
 		(shape input)
-		(at 499.11 439.42 180)
+		(at 477.52 439.42 180)
 		(fields_autoplaced yes)
 		(effects
@@
 		)
 		(property "Intersheetrefs" "${INTERSHEET_REFS}"
-			(at 479.2521 439.42 0)
+			(at 457.6621 439.42 0)
 			(effects
 				(font
@@
 	(global_label "PCIE_M2M_RX0_N"
 		(shape input)
-		(at 499.11 416.56 180)
+		(at 477.52 416.56 180)
 		(fields_autoplaced yes)
 		(effects
@@
 		)
 		(property "Intersheetrefs" "${INTERSHEET_REFS}"
-			(at 478.8892 416.56 0)
+			(at 457.2992 416.56 0)
 			(effects
 				(font
@@
 	(global_label "PCIE_M2M_TX2_P"
 		(shape input)
-		(at 499.11 429.26 180)
+		(at 477.52 429.26 180)
 		(fields_autoplaced yes)
 		(effects
@@
 		)
 		(property "Intersheetrefs" "${INTERSHEET_REFS}"
-			(at 479.2521 429.26 0)
+			(at 457.6621 429.26 0)
 			(effects
 				(font
@@
 	(global_label "PCIE_M2M_RX1_P"
 		(shape input)
-		(at 499.11 424.18 180)
+		(at 477.52 424.18 180)
 		(fields_autoplaced yes)
 		(effects
@@
 		)
 		(property "Intersheetrefs" "${INTERSHEET_REFS}"
-			(at 478.9497 424.18 0)
+			(at 457.3597 424.18 0)
 			(effects
 				(font
@@
 	(global_label "PCIE_M2M_TX1_P"
 		(shape input)
-		(at 499.11 419.1 180)
+		(at 477.52 419.1 180)
 		(fields_autoplaced yes)
 		(effects
@@
 		)
 		(property "Intersheetrefs" "${INTERSHEET_REFS}"
-			(at 479.2521 419.1 0)
+			(at 457.6621 419.1 0)
 			(effects
 				(font

Commit message: Aug 21, 2024 1
Parts:
- added R? (x2): 10K, symbol Device:R_Small
Connections:
- net SOM_IO_3V3: now also R?.1, R?.1
- net RTC_VBAT: now reaches A1.115 (VBAT), BT?.1 (+)
- net at A1.100 (~{CLKREQ3}): now also R?.2
- net at A1.102 (~{CLKREQ4}): now also R?.2
- net USB_SMEC_P: now reaches A1.76 (USB2_P7+)
- net USB_SMEC_N: now reaches A1.78 (USB2_P7-)
Other:
- moved on the sheet: BT?

Commit message: Aug 31, 2024
Parts:
- J?: footprint (none) -> Connector_PinHeader_2.54mm:PinHeader_1x02_P2.54mm_Vertical
Connections:
- net USB_CAM_N: now also A1.84 (USB2_P8-); no longer A1.114 (USB2_P6-)
- net USB_CAM_P: now also A1.82 (USB2_P8+); no longer A1.112 (USB2_P6+)
- net USB_M2E_N: now also A1.78 (USB2_P7-); no longer A1.109 (USB2_P5-)
- net USB_M2E_P: now also A1.76 (USB2_P7+); no longer A1.111 (USB2_P5+)
- net USB_SMEC_N: now also A1.109 (USB2_P5-); no longer A1.78 (USB2_P7-)
- net USB_SMEC_P: now also A1.111 (USB2_P5+); no longer A1.76 (USB2_P7+)
Other:
- note added: "July 4, 2024 - August 31, 2024"
- note removed: "July 4, 2024 - August 11, 2024"
- moved on the sheet: A1, BT?, C?, J?, R?, SW?, U?

Commit message: Sep 4, 2024 1
Parts:
- added R? (x16): 0, Resistor_SMD:R_0402_1005Metric, symbol Device:R_Small
- added R?: 100K, symbol Device:R_Small
- added R? (x2): 4.7K, symbol Device:R_Small
- J?: value Conn_01x02 -> Debug UART
Connections:
- net PCIE_LAN_RX0_N: now also R?.1; no longer A1.36 (HSIO3_RX-)
- net PCIE_LAN_RX0_P: now also R?.1; no longer A1.34 (HSIO3_RX+)
- net PCIE_M2E_RX0_N: now also R?.1; no longer A1.30 (HSIO2_RX-)
- net PCIE_M2E_RX0_P: now also R?.1; no longer A1.28 (HSIO2_RX+)
- net PCIE_M2M_RX0_N: now also R?.1; no longer A1.42 (HSIO8_RX-)
- net PCIE_M2M_RX0_P: now also R?.1; no longer A1.40 (HSIO8_RX+)
- net PCIE_M2M_RX1_N: now also R?.1; no longer A1.48 (HSIO9_RX-)
- net PCIE_M2M_RX1_P: now also R?.1; no longer A1.46 (HSIO9_RX+)
- net PCIE_M2M_RX2_N: now also R?.1; no longer A1.54 (HSIO10_RX-)
- net PCIE_M2M_RX2_P: now also R?.1; no longer A1.52 (HSIO10_RX+)
- net PCIE_M2M_RX3_N: now also R?.1; no longer A1.60 (HSIO11_RX-)
- net PCIE_M2M_RX3_P: now also R?.1; no longer A1.58 (HSIO11_RX+)
- net SOM_IO_3V3: now also R?.2, R?.2, R?.2
- net SOM_SMB_ALT: now also R?.1
- net SOM_SMB_SCL: now also R?.1
- net SOM_SMB_SDA: now also R?.1
- net SSUSB0_RXN: now also R?.1; no longer A1.18 (HSIO0_RX-)
- net SSUSB0_RXP: now also R?.1; no longer A1.16 (HSIO0_RX+)
- net SSUSB1_RXN: now also R?.1; no longer A1.24 (HSIO1_RX-)
- net SSUSB1_RXP: now also R?.1; no longer A1.22 (HSIO1_RX+)
- net USB_EXT1_N: now also A1.109 (USB2_P5-); no longer A1.67 (USB2_P1-)
- net USB_EXT1_P: now also A1.111 (USB2_P5+); no longer A1.69 (USB2_P1+)
- net USB_EXT2_N: now also A1.114 (USB2_P6-); no longer A1.73 (USB2_P2-)
- net USB_EXT2_P: now also A1.112 (USB2_P6+); no longer A1.75 (USB2_P2+)
- net USB_SMEC_N: now also A1.72 (USB2_P4-); no longer A1.109 (USB2_P5-)
- net USB_SMEC_P: now also A1.70 (USB2_P4+); no longer A1.111 (USB2_P5+)
- net SOM_USB_OC: now reaches A1.129 (~{USB_OC})
- net SIO_FAN1_PWM: now reaches A1.2 (FAN1_PWM)
- net SIO_FAN1_TAC: now reaches A1.4 (FAN1_TAC)
- net SIO_FAN2_PWM: now reaches A1.6 (FAN2_PWM)
- net SIO_FAN2_TAC: now reaches A1.8 (FAN2_TAC)
- net SIO_TSENSE: now reaches A1.9 (TSENSE)
- new net: A1.58 (HSIO11_RX+), R?.2
- new net: A1.16 (HSIO0_RX+), R?.2
- new net: A1.30 (HSIO2_RX-), R?.2
- new net: A1.34 (HSIO3_RX+), R?.2
- new net: A1.42 (HSIO8_RX-), R?.2
- new net: A1.28 (HSIO2_RX+), R?.2
- new net: A1.46 (HSIO9_RX+), R?.2
- new net: A1.52 (HSIO10_RX+), R?.2
- new net: A1.48 (HSIO9_RX-), R?.2
- new net: A1.36 (HSIO3_RX-), R?.2
- new net: A1.22 (HSIO1_RX+), R?.2
- new net: A1.24 (HSIO1_RX-), R?.2
- new net: A1.18 (HSIO0_RX-), R?.2
- new net: A1.40 (HSIO8_RX+), R?.2
- new net: A1.54 (HSIO10_RX-), R?.2
- new net: A1.60 (HSIO11_RX-), R?.2
- new net TCP0_DN: A1.67 (USB2_P1-)
- new net TCP0_DP: A1.69 (USB2_P1+)
- new net TCP1_DN: A1.73 (USB2_P2-)
- new net TCP1_DP: A1.75 (USB2_P2+)
Other:
- note added: "July 4, 2024 - September 4, 2024"
- note removed: "July 4, 2024 - August 31, 2024"
- moved on the sheet: J?

Commit message: Sep 4, 2024 2
Connections:
- no-connect marks 12 -> 29
Other:
- note added: "Note: SIO fan and pin connections may be unused"
- note added: "To-Do: find out if AUX is needed for HDMI"
Changed lines of the file:
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@@
+	)
+	(no_connect
+		(at 306.07 347.98)
+	)
+	(no_connect
+		(at 306.07 328.93)
+	)
+	(no_connect
+		(at 306.07 323.85)
+	)
+	(no_connect
+		(at 306.07 294.64)
+	)
+	(no_connect
+		(at 306.07 292.1)
+	)
+	(no_connect
+		(at 306.07 345.44)
+	)
+	(no_connect
+		(at 306.07 289.56)
 	)
 	(no_connect
@@
 	)
 	(no_connect
+		(at 306.07 335.28)
+	)
+	(no_connect
 		(at 224.79 280.67)
 	)
 	(no_connect
+		(at 306.07 331.47)
+	)
+	(no_connect
 		(at 224.79 195.58)
 	)
@@
 	)
 	(no_connect
+		(at 306.07 318.77)
+	)
+	(no_connect
+		(at 306.07 342.9)
+	)
+	(no_connect
 		(at 306.07 110.49)
 	)
 	(no_connect
+		(at 306.07 337.82)
+	)
+	(no_connect
+		(at 306.07 297.18)
+	)
+	(no_connect
+		(at 306.07 299.72)
+	)
+	(no_connect
 		(at 224.79 316.23)
 	)
 	(no_connect
 		(at 224.79 318.77)
+	)
+	(no_connect
+		(at 306.07 340.36)
+	)
+	(no_connect
+		(at 306.07 326.39)
+	)
+	(no_connect
+		(at 306.07 321.31)
 	)
 	(no_connect
@@
 				(size 1.27 1.27)
 			)
+		)
+	)
+	(text "Note: SIO fan and pin \nconnections may be unused"
+		(exclude_from_sim no)
+		(at 323.342 94.996 0)
+		(effects
+			(font
+				(size 1.27 1.27)
+			)
+			(justify left)
 		)
 	)
@@
 		)
 	)
+	(text "To-Do: find out if AUX \nis needed for HDMI\n"
+		(exclude_from_sim no)
+		(at 199.898 247.904 0)
+		(effects
+			(font
+				(size 1.27 1.27)
+			)
+			(justify left)
+		)
+	)

Commit message: Sep 5, 2024 2
Parts:
- added J? (x2): ~, Connector_PinHeader_2.54mm:PinHeader_1x02_P2.54mm_Vertical, symbol Connector_Generic:Conn_01x02
Connections:
- net SOM_TPM_IRQ: now reaches A1.127 (TPM_IRQ)
- net at A1.138 (UART2_TXD): now also J?.2 (Pin_2)
- net at A1.140 (UART2_RXD): now also J?.1 (Pin_1)
- net at A1.141 (UART1_RXD): now also J?.1 (Pin_1)
- net at A1.143 (UART1_TXD): now also J?.2 (Pin_2)
- net USB2_EXT2_N: now reaches A1.79 (USB2_P3-)
- net USB2_EXT2_P: now reaches A1.81 (USB2_P3+)
- net TCP0_DN renamed USB2_EXT0_N
- net TCP0_DP renamed USB2_EXT0_P
- net TCP1_DN renamed USB2_EXT1_N
- net TCP1_DP renamed USB2_EXT1_P
- net USB_EXT1_N renamed USB2_TCP0_DN
- net USB_EXT1_P renamed USB2_TCP0_DP
- net USB_EXT2_N renamed USB2_TCP1_DN
- net USB_EXT2_P renamed USB2_TCP1_DP
- net USB_SMEC_N renamed USB2_EXT3_N
- net USB_SMEC_P renamed USB2_EXT3_P
