File: circuits/mct2/mct2_ec.kicad_sch (KiCad schematic)
At the start: 1 part

Commit message: Aug 2, 2024
Parts:
- removed U?: STM32U5A5ZJTx, Package_QFP:LQFP-144_20x20mm_P0.5mm, symbol MCU_ST_STM32U5:STM32U5A5ZJTx
- added U?: STM32L4P5ZGTx, Package_QFP:LQFP-144_20x20mm_P0.5mm, symbol MCU_ST_STM32L4:STM32L4P5ZGTx
Connections:
- net GND: now also U?.107 (VSS), U?.120 (VSS), U?.130 (VSS), U?.143 (VSS), U?.16 (VSS), U?.30 (VSSA), U?.38 (VSS), U?.51 (VSS), U?.61 (VSS), U?.71 (VSS), U?.83 (VSS), U?.94 (VSS)

Commit message: Aug 3, 2024
Parts:
- added C? (x2): 100nF, symbol Device:C_Small
- added U?: SiT1533AI-H4-DCC-32.768, symbol mediacow:SiT1533AI-H4-DCC-32.768
- added U?: SiT1602BI-13-XXN-48.000000, symbol mediacow:SiT1602BI-13-XXN-48.000000
Connections:
- net GND: now also C?.2, C?.2, U?.2 (GND), U?.2 (GND)
- net at U?.23 (PH0): now also U?.3 (OUT)
- net at U?.8 (PC14): now also U?.3 (OUT)
- new net SMEC_VDD: C?.1, C?.1, U?.4 (VDD), U?.4 (VDD)
- no-connect marks 0 -> 1

Commit message: Aug 10, 2024
Parts:
- added J?: Conn_01x04_Pin, Connector:FanPinHeader_1x04_P2.54mm_Vertical, symbol Connector:Conn_01x04_Pin
Connections:
- net GND: now also J?.1 (Pin_1)
- new net FAN_12V: J?.2 (Pin_2)
- new net FAN_PWM: J?.4 (Pin_4)
- new net FAN_TAC: J?.3 (Pin_3)
- no-connect marks 1 -> 2
Other:
- note added: "CTCL 2021-2024"
- note added: "July 4, 2024 - August 9, 2024"
- note added: "MediaCow Touch 2 - System Management Embedded Controller"
Changed lines of the file:
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@@
+	)
+	(no_connect
+		(at 453.39 417.83)
 	)
 	(no_connect
@@
 			(width 0)
 			(type default)
+		)
+	)
+	(text "CTCL 2021-2024"
+		(exclude_from_sim no)
+		(at 820.674 564.388 0)
+		(effects
+			(font
+				(size 1.27 1.27)
+			)
+		)
+	)
+	(text "July 4, 2024 - August 9, 2024"
+		(exclude_from_sim no)
+		(at 766.064 577.596 0)
+		(effects
+			(font
+				(size 1.27 1.27)
+			)
+		)
+	)
+	(text "MediaCow Touch 2 - System Management Embedded Controller"
+		(exclude_from_sim no)
+		(at 760.984 574.04 0)
+		(effects
+			(font
+				(size 1.27 1.27)
+			)
 		)
 	)
@@
 		)
 	)
+	(global_label "FAN_TAC"
+		(shape input)
+		(at 577.85 459.74 180)
+		(fields_autoplaced yes)
+		(effects
+			(font
+				(size 1.27 1.27)
+			)
+			(justify right)
+		)
+		(property "Intersheetrefs" "${INTERSHEET_REFS}"
+			(at 567.0633 459.74 0)
+			(effects
+				(font
+					(size 1.27 1.27)
+				)
+				(justify right)
+				(hide yes)
+			)
+		)
+	)
 	(global_label "SMEC_VDD"
 		(shape input)
@@
 		)
 	)
+	(global_label "FAN_12V"
+		(shape input)
+		(at 577.85 462.28 180)
+		(fields_autoplaced yes)
+		(effects
+			(font
+				(size 1.27 1.27)
+			)
+			(justify right)
+		)
+		(property "Intersheetrefs" "${INTERSHEET_REFS}"
+			(at 566.8819 462.28 0)
+			(effects
+				(font
+					(size 1.27 1.27)
+				)
+				(justify right)
+				(hide yes)
+			)
+		)
+	)
+	(global_label "FAN_PWM"
+		(shape input)
+		(at 577.85 457.2 180)
+		(fields_autoplaced yes)
+		(effects
+			(font
+				(size 1.27 1.27)
+			)
+			(justify right)
+		)
+		(property "Intersheetrefs" "${INTERSHEET_REFS}"
+			(at 566.2167 457.2 0)
+			(effects
+				(font
+					(size 1.27 1.27)
+				)
+				(justify right)
+				(hide yes)
+			)
+		)
+	)
 	(symbol
 		(lib_id "power:GND")
@@
 	(symbol
 		(lib_id "power:GND")
+		(at 577.85 464.82 0)
+		(unit 1)
+		(exclude_from_sim no)
+		(in_bom yes)
+		(on_board yes)
+		(dnp no)
+		(fields_autoplaced yes)
+		(property "Reference" "#PWR021"
+			(at 577.85 471.17 0)
+			(effects
+				(font
+					(size 1.27 1.27)
+				)
+				(hide yes)
+			)
+		)
+		(property "Value" "GND"
+			(at 577.85 469.9 0)
+			(effects
+				(font
+					(size 1.27 1.27)
+				)
+			)
+		)
+		(property "Footprint" ""
+			(at 577.85 464.82 0)
+			(effects
+				(font
+					(size 1.27 1.27)
+				)
+				(hide yes)
+			)
+		)
+		(property "Datasheet" ""
+			(at 577.85 464.82 0)
+			(effects
+				(font
+					(size 1.27 1.27)
+				)
+				(hide yes)
+			)
+		)
+		(property "Description" "Power symbol creates a global label with name \"GND\" , ground"
+			(at 577.85 464.82 0)
+			(effects
+				(font
+					(size 1.27 1.27)
+				)
+				(hide yes)
+			)
+		)
+		(pin "1"
+		)
+		(instances
+			(project ""
+				(path "/0917e100-0497-47cd-9e32-3e43ad224d2b/f1c7c14b-ceb5-428a-9125-91c37b884576"
+					(reference "#PWR021")
+					(unit 1)
+				)
+			)
+		)
+	)
+	(symbol
+		(lib_id "power:GND")
 		(at 331.47 311.15 0)
 		(unit 1)
@@
 					(unit 1)
 				)
+			)
+		)
+	)
+	(symbol
+		(lib_id "Connector:Conn_01x04_Pin")
+		(at 582.93 462.28 180)
+		(unit 1)
+		(exclude_from_sim no)
+		(in_bom yes)
+		(on_board yes)
+		(dnp no)
+		(fields_autoplaced yes)
+		(property "Reference" "J?"
+			(at 584.2 459.7399 0)
+			(effects
+				(font
+					(size 1.27 1.27)
+				)
+				(justify right)
+			)
+		)
+		(property "Value" "Conn_01x04_Pin"
+			(at 584.2 462.2799 0)
+			(effects
+				(font
+					(size 1.27 1.27)
+				)
+				(justify right)
+			)
+		)
+		(property "Footprint" "Connector:FanPinHeader_1x04_P2.54mm_Vertical"
+			(at 582.93 462.28 0)
+			(effects
+				(font
+					(size 1.27 1.27)
+				)
+				(hide yes)
+			)
+		)
+		(property "Datasheet" "~"
+			(at 582.93 462.28 0)
+			(effects
+				(font
+					(size 1.27 1.27)
+				)
+				(hide yes)
+			)
+		)
+		(property "Description" "Generic connector, single row, 01x04, script generated"
+			(at 582.93 462.28 0)
+			(effects
+				(font
+					(size 1.27 1.27)
+				)
+				(hide yes)
+			)
+		)
+		(pin "4"
+		)
+		(pin "3"
+		)
+		(pin "2"
+		)
+		(pin "1"
+		)
+		(instances
+			(project ""
+				(path "/0917e100-0497-47cd-9e32-3e43ad224d2b/f1c7c14b-ceb5-428a-9125-91c37b884576"
+					(reference "J?")
+					(unit 1)
+				)

Commit message: Aug 11, 2024 1
Parts:
- added C? (x8): 100nF, symbol Device:C_Small
- added C?: 22uF, symbol Device:C_Small
- added C?: 4.7uF, symbol Device:C_Small
- added D?: CMMSH1-60G, symbol Device:D_Schottky_Small_Filled
- added L?: 15uH, symbol Device:L_Small
- added R?: 1M, symbol Device:R_Small
- added U?: RAA211403, Package_TO_SOT_SMD:TSOT-23-5, symbol mediacow:RAA211403
Connections:
- net GND: now also C?.2, C?.2, C?.2, C?.2, C?.2, C?.2, C?.2, C?.2, C?.2, C?.2, D?.2 (A), U?.2 (GND)
- net SMEC_VDD: now also U?.108 (VDD), U?.121 (VDD), U?.144 (VDD), U?.17 (VDD), U?.39 (VDD), U?.52 (VDD), U?.62 (VDD), U?.72 (VDD), U?.84 (VDD), C?.1, C?.1, C?.1, C?.1, C?.1, C?.1, C?.1, C?.1, C?.1, L?.2, U?.1 (VOUT)
- new net: R?.2, U?.3 (EN)
- new net: D?.1 (K), L?.1, U?.5 (SW)
- new net VSB: C?.1, R?.1, U?.4 (VIN)

Commit message: Aug 11, 2024 2
Parts:
- added C? (x2): 100nF, symbol Device:C_Small
- added JP?: SolderJumper_2_Open, symbol Jumper:SolderJumper_2_Open
Connections:
- net GND: now also C?.2, C?.2, JP?.1 (A)
- net SMEC_VDD: now also U?.106 (VDDUSB), C?.1
- net at U?.8 (PC14): no longer U?.3 (OUT)
- net at U?.23 (PH0): no longer U?.3 (OUT)
- net at U?.25 (NRST): now also C?.1, JP?.2 (B)
- new net SMEC_HSE: U?.3 (OUT)
- new net SMEC_LSE: U?.3 (OUT)
Other:
- note added: "July 4, 2024 - August 11, 2024"
- note added: "MediaCow Touch 2"
- note added: "MediaCow Touch 2 - System"
- note added: "Reference STMCube32MX file smec.io for pin assignments"
- note removed: "July 4, 2024 - August 9, 2024"
- note removed: "MediaCow Touch 2 - System Management Embedded Controller"
- moved on the sheet: C?, J?, R?, U?

Commit message: Aug 13, 2024
Parts:
- removed C?: 22uF, symbol Device:C_Small
- removed C?: 4.7uF, symbol Device:C_Small
- removed D?: CMMSH1-60G, symbol Device:D_Schottky_Small_Filled
- removed L?: 15uH, symbol Device:L_Small
- removed R?: 1M, symbol Device:R_Small
- removed U?: RAA211403, Package_TO_SOT_SMD:TSOT-23-5, symbol mediacow:RAA211403
Connections:
- net SMEC_HSE: now also U?.23 (PH0)
- net SMEC_LSE: now also U?.8 (PC14)
Other:
- note added: "July 4, 2024 - August 13, 2024"
- note removed: "July 4, 2024 - August 11, 2024"

Commit message: Aug 19, 2024
Connections:
- net OLED_D2: now reaches U?.114 (PD0)
- net OLED_D3: now reaches U?.115 (PD1)
- net OLED_RD: now reaches U?.118 (PD4)
- net OLED_WR: now reaches U?.119 (PD5)
- net OLED_CS: now reaches U?.123 (PD7)
- net SMB1_SCL: now reaches U?.136 (PB6)
- net SMB1_SDA: now reaches U?.137 (PB7)
- net SMB1_ALT: now reaches U?.35 (PA1)
- net OLED_D4: now reaches U?.58 (PE7)
- net OLED_D5: now reaches U?.59 (PE8)
- net OLED_D6: now reaches U?.60 (PE9)
- net OLED_D7: now reaches U?.63 (PE10)
- net OLED_DC: now reaches U?.80 (PD11)
- net OLED_D0: now reaches U?.85 (PD14)
- net OLED_D1: now reaches U?.86 (PD15)

Commit message: Aug 21, 2024 1
Parts:
- removed C? (x3): 100nF, symbol Device:C_Small
- removed U?: STM32L4P5ZGTx, Package_QFP:LQFP-144_20x20mm_P0.5mm, symbol MCU_ST_STM32L4:STM32L4P5ZGTx
- added J?: Conn_01x02, Connector_PinHeader_1.00mm:PinHeader_1x02_P1.00mm_Vertical, symbol Connector_Generic:Conn_01x02
- added R? (x8): ?, symbol Device:R_Small
- added U?: ICM-20948, Sensor_Motion:InvenSense_QFN-24_3x3mm_P0.4mm, symbol Sensor_Motion:ICM-20948
- added U?: STM32L496VGTx, Package_QFP:LQFP-100_14x14mm_P0.5mm, symbol MCU_ST_STM32L4:STM32L496VGTx
- added U?: BMP384, symbol mediacow:BMP384
Connections:
- net GND: now also U?.10 (VSS), U?.19 (VSSA), U?.27 (VSS), U?.49 (VSS), U?.74 (VSS), U?.99 (VSS)
- net OLED_CS: now also U?.88 (PD7)
- net OLED_D0: now also U?.61 (PD14)
- net OLED_D1: now also U?.62 (PD15)
- net OLED_D2: now also U?.81 (PD0)
- net OLED_D3: now also U?.82 (PD1)
- net OLED_D4: now also U?.38 (PE7)
- net OLED_D5: now also U?.39 (PE8)
- net OLED_D6: now also U?.40 (PE9)
- net OLED_D7: now also U?.41 (PE10)
- net OLED_DC: now also U?.58 (PD11)
- net OLED_RD: now also U?.85 (PD4)
- net OLED_WR: now also U?.86 (PD5)
- net SMB1_ALT: now also U?.24 (PA1)
- net SMB1_SCL: now also R?.2, U?.92 (PB6)
- net SMB1_SDA: now also R?.2, U?.93 (PB7)
- net SMEC_HSE: now also U?.12 (PH0)
- net SMEC_LSE: now also U?.8 (PC14)
- net SMEC_VDD: now also R?.1, R?.1, R?.1, R?.1, R?.1, R?.1, R?.1, R?.1, U?.100 (VDD), U?.11 (VDD), U?.28 (VDD), U?.50 (VDD), U?.73 (VDDUSB), U?.75 (VDD)
- net SML_ALT: now also R?.2, U?.51 (PB12)
- net SML_SCL: now also R?.2, U?.47 (PB10)
- net SML_SDA: now also R?.2, U?.48 (PB11)
- net at C?.1, JP?.2 (B): now also U?.14 (NRST)
- new net: U?.18 (GND), U?.20 (GND)
- new net OLED_RST: U?.87 (PD6)
- new net RTC_VBAT: U?.6 (VBAT)
- new net SMEC_SW_CLK: J?.2 (Pin_2), U?.76 (PA14)
- new net SMEC_SW_DIO: J?.1 (Pin_1), U?.72 (PA13)
- new net SMEC_VDDA: U?.22 (VDDA)
- new net SOM_SMB_ALT: R?.2, U?.37 (PB2)
- new net SOM_SMB_SCL: R?.2, U?.15 (PC0)
- new net SOM_SMB_SDA: R?.2, U?.16 (PC1)
- new net USB_SMEC_N: U?.70 (PA11)
- new net USB_SMEC_P: U?.71 (PA12)
Other:
- note added: "July 4, 2024 - August 21, 2024"
- note removed: "July 4, 2024 - August 13, 2024"
- moved on the sheet: C?, JP?
