File: circuits/mct2/mct2_ec.kicad_sch (KiCad schematic)
At the start: 25 parts

Commit message: Aug 22, 2024 1
Parts:
- added C?: C_Small, symbol Device:C_Small
- added U?: MIC5504-1.8YM5, Package_TO_SOT_SMD:SOT-23-5, symbol Regulator_Linear:MIC5504-1.8YM5
- added U?: ~, symbol mediacow:TXS0104E
Connections:
- net GND: now also U?.18 (GND), U?.20 (GND), U?.3 (VSS), U?.8 (VSS), U?.9 (VSS), C?.2, U?.2 (GND), U?.7 (GND)
- net SMEC_VDD: now also U?.1 (VCCA)
- net at U?.10 (REGOUT): now also C?.1
- net at U?.22 (~{CS}): now also U?.10 (B4)
- net at U?.23 (SCL/SCLK): now also U?.11 (B3)
- net at U?.24 (SDA/SDI): now also U?.12 (B2)
- net at U?.8 (VDDIO): now also U?.14 (VCCB), U?.5 (VOUT)
- net at U?.9 (SDO/AD0): now also U?.13 (B1)
- net SMB1_ALT renamed SYS_SMB_ALT
- net SMB1_SCL renamed SYS_SMB_SCL
- net SMB1_SDA renamed SYS_SMB_SDA
- no-connect marks 2 -> 4
Other:
- moved on the sheet: R?, U?

Commit message: Aug 31, 2024
Parts:
- removed U?: MIC5504-1.8YM5, Package_TO_SOT_SMD:SOT-23-5, symbol Regulator_Linear:MIC5504-1.8YM5
- added C? (x2): 100nF, symbol Device:C_Small
- C?: value C_Small -> 100nF
Connections:
- net GND: now also U?.11 (FSYNC), C?.2, C?.2
- net at U?.12 (INT1): now also U?.10 (B4)
- net ICM_1V8: now reaches U?.13 (VDD)
- net ICM_1V8: now also U?.14 (VCCB), U?.22 (~{CS}), U?.8 (VDDIO), U?.9 (SDO/AD0), C?.1, C?.1
- net at U?.13 (B1): no longer U?.9 (SDO/AD0)
- net SYS_I2C_SCL: now reaches U?.59 (PD12)
- net SYS_I2C_SCL: now also U?.3 (A2)
- net SYS_I2C_SDA: now reaches U?.60 (PD13)
- net SYS_I2C_SDA: now also U?.4 (A3)
Other:
- note added: "1.8v logic"
- note added: "3.3v logic"
- note added: "July 4, 2024 - August 31, 2024"
- note removed: "July 4, 2024 - August 21, 2024"
- moved on the sheet: C?, U?

Commit message: Sep 4, 2024 1
Parts:
- removed R? (x3): ?, symbol Device:R_Small

Commit message: Sep 5, 2024 1
Parts:
- U?: value ~ -> TXS0104E
Connections:
- net SYS_I2C_SCL: now also U?.2 (SCL)
- net SYS_I2C_SDA: now also U?.4 (SDI)
Other:
- note added: "July 4, 2024 - September 5, 2024"
- note added: "MediaCow Touch 2 - SMEC"
- note removed: "July 4, 2024 - August 31, 2024"
- note removed: "MediaCow Touch 2 - System"
- moved on the sheet: U?
Changed lines of the file:
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@@
 	)
 	(junction
-		(at 467.36 233.68)
+		(at 406.4 182.88)
 		(diameter 0)
 		(color 0 0 0 0)
@@
 	(wire
 		(pts
-			(xy 467.36 233.68) (xy 464.82 233.68)
+			(xy 406.4 182.88) (xy 403.86 182.88)
 		)
 		(stroke
@@
 	(wire
 		(pts
-			(xy 469.9 233.68) (xy 467.36 233.68)
+			(xy 408.94 182.88) (xy 406.4 182.88)
 		)
 		(stroke
@@
 	(wire
 		(pts
+			(xy 388.62 170.18) (xy 396.24 170.18)
+		)
+		(stroke
+			(width 0)
+			(type default)
+		)
+	)
+	(wire
+		(pts
 			(xy 363.22 370.84) (xy 365.76 370.84)
 		)
@@
 	(wire
 		(pts
+			(xy 388.62 167.64) (xy 396.24 167.64)
+		)
+		(stroke
+			(width 0)
+			(type default)
+		)
+	)
+	(wire
+		(pts
 			(xy 485.14 391.16) (xy 485.14 396.24)
 		)
@@
 		)
 	)
-	(text "July 4, 2024 - August 31, 2024"
+	(text "July 4, 2024 - September 5, 2024"
 		(exclude_from_sim no)
 		(at 766.318 577.342 0)
@@
 		)
 	)
-	(text "MediaCow Touch 2 - System"
+	(text "MediaCow Touch 2 - SMEC"
 		(exclude_from_sim no)
 		(at 750.062 573.532 0)
@@
 		)
 	)
+	(global_label "SYS_I2C_SCL"
+		(shape input)
+		(at 388.62 167.64 180)
+		(fields_autoplaced yes)
+		(effects
+			(font
+				(size 1.27 1.27)
+			)
+			(justify right)
+		)
+		(property "Intersheetrefs" "${INTERSHEET_REFS}"
+			(at 373.6001 167.64 0)
+			(effects
+				(font
+					(size 1.27 1.27)
+				)
+				(justify right)
+				(hide yes)
+			)
+		)
+	)
 	(global_label "SMEC_LSE"
 		(shape input)
@@
 		)
 	)
+	(global_label "SYS_I2C_SDA"
+		(shape input)
+		(at 388.62 170.18 180)
+		(fields_autoplaced yes)
+		(effects
+			(font
+				(size 1.27 1.27)
+			)
+			(justify right)
+		)
+		(property "Intersheetrefs" "${INTERSHEET_REFS}"
+			(at 373.5396 170.18 0)
+			(effects
+				(font
+					(size 1.27 1.27)
+				)
+				(justify right)
+				(hide yes)
+			)
+		)
+	)
 	(global_label "SML_ALT"
 		(shape input)
@@
 	(symbol
 		(lib_id "power:GND")
-		(at 467.36 233.68 0)
+		(at 406.4 182.88 0)
 		(mirror y)
 		(unit 1)
@@
 		(fields_autoplaced yes)
 		(property "Reference" "#PWR0257"
-			(at 467.36 240.03 0)
+			(at 406.4 189.23 0)
 			(effects
 				(font
@@
 		)
 		(property "Value" "GND"
-			(at 467.36 238.76 0)
+			(at 406.4 187.96 0)
 			(effects
 				(font
@@
 		)
 		(property "Footprint" ""
-			(at 467.36 233.68 0)
+			(at 406.4 182.88 0)
 			(effects
 				(font
@@
 		)
 		(property "Datasheet" ""
-			(at 467.36 233.68 0)
+			(at 406.4 182.88 0)
 			(effects
 				(font
@@
 		)
 		(property "Description" "Power symbol creates a global label with name \"GND\" , ground"
-			(at 467.36 233.68 0)
+			(at 406.4 182.88 0)
 			(effects
 				(font
@@
 	(symbol
 		(lib_id "mediacow:BMP384")
-		(at 467.36 223.52 0)
+		(at 406.4 172.72 0)
 		(mirror y)
 		(unit 1)
@@
 		(fields_autoplaced yes)
 		(property "Reference" "U?"
-			(at 467.36 212.09 0)
+			(at 406.4 161.29 0)
 			(effects
 				(font
@@
 		)
 		(property "Value" "BMP384"
-			(at 467.36 214.63 0)
+			(at 406.4 163.83 0)
 			(effects
 				(font
@@
 		)
 		(property "Footprint" ""
-			(at 434.34 227.33 0)
+			(at 373.38 176.53 0)
 			(effects
 				(font
@@
 		)
 		(property "Datasheet" ""
-			(at 434.34 227.33 0)
+			(at 373.38 176.53 0)
 			(effects
 				(font
@@
 		)
 		(property "Description" ""
-			(at 434.34 227.33 0)
+			(at 373.38 176.53 0)
 			(effects
 				(font
@@
 		(on_board yes)
 		(dnp no)
-		(fields_autoplaced yes)
 		(property "Reference" "U?"
-			(at 367.9541 232.41 0)
+			(at 358.14 231.14 0)
 			(effects
 				(font
@@
 			)
 		)
-		(property "Value" "~"
-			(at 367.9541 233.68 0)
+		(property "Value" "TXS0104E"
+			(at 366.522 231.14 0)
 			(effects
 				(font

Commit message: Sep 5, 2024 2
Connections:
- net USB_SMEC_N: no longer names the net of U?.70 (PA11)
- net USB_SMEC_P: no longer names the net of U?.71 (PA12)
Changed lines of the file:
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@@
-	(wire
-		(pts
-			(xy 411.48 353.06) (xy 457.2 353.06)
-		)
-		(stroke
-			(width 0)
-			(type default)
-		)
-	)
 	(wire
 		(pts
@@
 		(pts
 			(xy 480.06 383.54) (xy 485.14 383.54)
-		)
-		(stroke
-			(width 0)
-			(type default)
-		)
-	)
-	(wire
-		(pts
-			(xy 411.48 355.6) (xy 457.2 355.6)
 		)
 		(stroke
@@
 		)
 	)
-	(global_label "USB_SMEC_N"
-		(shape input)
-		(at 457.2 353.06 0)
+	(global_label "SML_SCL"
+		(shape input)
+		(at 497.84 393.7 0)
 		(fields_autoplaced yes)
 		(effects
@@
 		)
 		(property "Intersheetrefs" "${INTERSHEET_REFS}"
-			(at 472.3408 353.06 0)
+			(at 510.4408 393.7 0)
 			(effects
 				(font
@@
 		)
 	)
-	(global_label "SML_SCL"
-		(shape input)
-		(at 497.84 393.7 0)
+	(global_label "FAN_TAC"
+		(shape input)
+		(at 452.12 270.51 180)
+		(fields_autoplaced yes)
+		(effects
+			(font
+				(size 1.27 1.27)
+			)
+			(justify right)
+		)
+		(property "Intersheetrefs" "${INTERSHEET_REFS}"
+			(at 441.3333 270.51 0)
+			(effects
+				(font
+					(size 1.27 1.27)
+				)
+				(justify right)
+				(hide yes)
+			)
+		)
+	)
+	(global_label "SMEC_VDD"
+		(shape input)
+		(at 497.84 383.54 0)
 		(fields_autoplaced yes)
 		(effects
@@
 		)
 		(property "Intersheetrefs" "${INTERSHEET_REFS}"
-			(at 510.4408 393.7 0)
+			(at 510.5013 383.54 0)
 			(effects
 				(font
@@
 		)
 	)
-	(global_label "FAN_TAC"
-		(shape input)
-		(at 452.12 270.51 180)
+	(global_label "SOM_SMB_SDA"
+		(shape input)
+		(at 414.02 414.02 0)
+		(fields_autoplaced yes)
+		(effects
+			(font
+				(size 1.27 1.27)
+			)
+			(justify left)
+		)
+		(property "Intersheetrefs" "${INTERSHEET_REFS}"
+			(at 426.6813 414.02 0)
+			(effects
+				(font
+					(size 1.27 1.27)
+				)
+				(justify left)
+				(hide yes)
+			)
+		)
+	)
+	(global_label "SYS_I2C_SDA"
+		(shape input)
+		(at 363.22 424.18 180)
 		(fields_autoplaced yes)
 		(effects
@@
 		)
 		(property "Intersheetrefs" "${INTERSHEET_REFS}"
-			(at 441.3333 270.51 0)
+			(at 348.1396 424.18 0)
 			(effects
 				(font
@@
 				(hide yes)
 			)
-		)
-	)
-	(global_label "SMEC_VDD"
-		(shape input)
-		(at 497.84 383.54 0)
-		(fields_autoplaced yes)
-		(effects
-			(font
-				(size 1.27 1.27)
-			)
-			(justify left)
-		)
-		(property "Intersheetrefs" "${INTERSHEET_REFS}"
-			(at 510.5013 383.54 0)
-			(effects
-				(font
-					(size 1.27 1.27)
-				)
-				(justify left)
-				(hide yes)
-			)
-		)
-	)
-	(global_label "SOM_SMB_SDA"
-		(shape input)
-		(at 414.02 414.02 0)
-		(fields_autoplaced yes)
-		(effects
-			(font
-				(size 1.27 1.27)
-			)
-			(justify left)
-		)
-		(property "Intersheetrefs" "${INTERSHEET_REFS}"
-			(at 426.6813 414.02 0)
-			(effects
-				(font
-					(size 1.27 1.27)
-				)
-				(justify left)
-				(hide yes)
-			)
-		)
-	)
-	(global_label "SYS_I2C_SDA"
-		(shape input)
-		(at 363.22 424.18 180)
-		(fields_autoplaced yes)
-		(effects
-			(font
-				(size 1.27 1.27)
-			)
-			(justify right)
-		)
-		(property "Intersheetrefs" "${INTERSHEET_REFS}"
-			(at 348.1396 424.18 0)
-			(effects
-				(font
-					(size 1.27 1.27)
-				)
-				(justify right)
-				(hide yes)
-			)
-		)
-	)
-	(global_label "USB_SMEC_P"
-		(shape input)
-		(at 457.2 355.6 0)
-		(fields_autoplaced yes)
-		(effects
-			(font
-				(size 1.27 1.27)
-			)
-			(justify left)
-		)
-		(property "Intersheetrefs" "${INTERSHEET_REFS}"
-			(at 472.2803 355.6 0)
-			(effects
-				(font
-					(size 1.27 1.27)
-				)
-				(justify left)
-				(hide yes)
-			)

Commit message: Sep 12, 2024 2
Parts:
- removed U?: STM32L496VGTx, Package_QFP:LQFP-100_14x14mm_P0.5mm, symbol MCU_ST_STM32L4:STM32L496VGTx
- removed U?: SiT1602BI-13-XXN-48.000000, symbol mediacow:SiT1602BI-13-XXN-48.000000
- added J?: Conn_ARM_JTAG_SWD_20, symbol Connector:Conn_ARM_JTAG_SWD_20
- added J?: Conn_01x08, symbol Connector_Generic:Conn_01x08
- added J?: Conn_01x40_Shielded, symbol Connector_Generic_Shielded:Conn_01x40_Shielded
- added Q?: NSS40201L, Package_TO_SOT_SMD:SOT-23, symbol Simulation_SPICE:NPN
- added R? (x2): 4.7K, symbol Device:R_Small
- added U? (x12): SP7021, symbol SP7021:SP7021
- added U?: SiT8008BI-11-33E-27.000000G, symbol mediacow:SiT8008BI-11-33E-27.000000G
- added U?: NSV45020AT1G, Diode_SMD:D_SOD-123, symbol mediacow:NSV45020AT1G
- added U?: NXS0108BQX, symbol mediacow:NXS0108BQX
Connections:
- net GND: now also J?.10 (GND), J?.12 (GND), J?.14 (GND), J?.16 (GND), J?.18 (GND), J?.20 (GND), J?.34 (Pin_34), J?.4 (GND), J?.4 (Pin_4), J?.40 (Pin_40), J?.6 (GND), J?.6 (Pin_6), J?.8 (GND), J?.SH (Shield), Q?.3 (E), R?.2, U?.10 (GND), U?.2 (GND)
- net SMEC_LSE: no longer U?.3 (OUT)
- net SMEC_VDD: now also U?.1 (OE), U?.4 (VDD)
- net SYS_SMB_ALT: now also J?.2 (Pin_2)
- net SYS_SMB_SCL: now also J?.3 (Pin_3)
- net SYS_SMB_SDA: now also J?.4 (Pin_4)
- new net: Q?.1 (C), U?.2 (K)
- new net: J?.1 (VTREF), U?.19 (VCCB)
- new net: J?.11 (RTCK), U?.17 (B3)
- new net: J?.13 (TDO/SWO), U?.14 (B6)
- new net: J?.15 (~{SRST}), U?.18 (B2)
- new net: J?.3 (~{TRST}), U?.20 (B1)
- new net: J?.5 (TDI), U?.13 (B7)
- new net: J?.7 (TMS/SWDIO), U?.15 (B5)
- new net: J?.9 (TCK/SWCLK), U?.16 (B4)
- new net: Q?.2 (B), R?.1, R?.2
- new net KP_RST: J?.5 (Pin_5)
- new net KP_SW_CAM: J?.8 (Pin_8)
- new net KP_SW_RAD: J?.7 (Pin_7)
- new net KP_VDD: J?.1 (Pin_1)
- new net SMEC_A926_JTAG_RTCK: U?.105 (JTAG_RTCK_A926_8051), U?.4 (A3)
- new net SMEC_A926_JTAG_TCLK: U?.106 (JTAG_TCLK_A926_8051), U?.5 (A4)
- new net SMEC_A926_JTAG_TDI: U?.112 (JTAG_TDI_A926_8051), U?.8 (A7)
- new net SMEC_A926_JTAG_TDO: U?.104 (JTAG_TDO_A926_8051), U?.7 (A6)
- new net SMEC_A926_JTAG_TMS: U?.107 (JTAG_TMS_A926_8051), U?.6 (A5)
- new net SMEC_A926_JTAG_TRST: U?.1 (A1), U?.113 (JTAG_TRST_A926_8051)
- new net SMEC_CA7_SWD_CLK: U?.102 (SWD_DATA_CA7)
- new net SMEC_CA7_SWD_DATA: U?.102 (SWD_DATA_CA7)
- new net SMEC_CLK_RTC: U?.123 (XTAL32K_IN), U?.3 (OUT)
- new net SMEC_CLK_SYS: U?.110 (XTAL_IN), U?.3 (OUT)
- new net SMEC_LCD_CS: J?.11 (Pin_11)
- new net SMEC_LCD_DB0: J?.28 (Pin_28)
- new net SMEC_LCD_DB1: J?.29 (Pin_29)
- new net SMEC_LCD_DB2: J?.30 (Pin_30)
- new net SMEC_LCD_DB3: J?.31 (Pin_31)
- new net SMEC_LCD_DB4: J?.32 (Pin_32)
- new net SMEC_LCD_DB5: J?.33 (Pin_33)
- new net SMEC_LCD_DE: J?.13 (Pin_13)
- new net SMEC_LCD_DG0: J?.22 (Pin_22)
- new net SMEC_LCD_DG1: J?.23 (Pin_23)
- new net SMEC_LCD_DG2: J?.24 (Pin_24)
- new net SMEC_LCD_DG3: J?.25 (Pin_25)
- new net SMEC_LCD_DG4: J?.26 (Pin_26)
- new net SMEC_LCD_DG5: J?.27 (Pin_27)
- new net SMEC_LCD_DR0: J?.16 (Pin_16)
- new net SMEC_LCD_DR1: J?.17 (Pin_17)
- new net SMEC_LCD_DR2: J?.18 (Pin_18)
- new net SMEC_LCD_DR3: J?.19 (Pin_19)
- new net SMEC_LCD_DR4: J?.20 (Pin_20)
- new net SMEC_LCD_DR5: J?.21 (Pin_21)
- new net SMEC_LCD_HSYNC: J?.15 (Pin_15)
- new net SMEC_LCD_LEDK: J?.2 (Pin_2), J?.3 (Pin_3), U?.1 (A)
- new net SMEC_LCD_LED_PWM: R?.1
- new net SMEC_LCD_PCLK: J?.12 (Pin_12)
- new net SMEC_LCD_PWM: J?.8 (Pin_8)
- new net SMEC_LCD_RST: J?.6 (Pin_6)
- new net SMEC_LCD_SCL: J?.10 (Pin_10)
- new net SMEC_LCD_SDA: J?.9 (Pin_9)
- new net SMEC_LCD_TE: J?.7 (Pin_7)
- new net SMEC_LCD_VCI: J?.5 (Pin_5)
- new net SMEC_LCD_VSYNC: J?.14 (Pin_14)
- new net SMEC_UART0_RX: U?.99 (UA0_RX)
- new net SMEC_UART0_TX: U?.98 (UA0_TX)
- new net VSYS: J?.1 (Pin_1)
- no-connect marks 4 -> 10
Other:
- note added: "July 4, 2024 - September 12, 2024"
- note added: "VSYS goes into LED Anode"
- note removed: "July 4, 2024 - September 5, 2024"
- moved on the sheet: C?, J?, JP?, R?, U?

Commit message: Sep 17, 2024 1
Connections:
- net SMEC_LCD_DB0 is gone; now on net SMEC_LCD_B0: J?.28 (Pin_28)
- net SMEC_LCD_DB1 is gone; now on net SMEC_LCD_B1: J?.29 (Pin_29)
- net SMEC_LCD_DB2 is gone; now on net SMEC_LCD_B2: J?.30 (Pin_30)
- net SMEC_LCD_DB3 is gone; now on net SMEC_LCD_B3: J?.31 (Pin_31)
- net SMEC_LCD_DB4 is gone; now on net SMEC_LCD_B4: J?.32 (Pin_32)
- net SMEC_LCD_DB5 is gone; now on net SMEC_LCD_B5: J?.33 (Pin_33)
- net SMEC_LCD_DG0 is gone; now on net SMEC_LCD_G0: J?.22 (Pin_22)
- net SMEC_LCD_DG1 is gone; now on net SMEC_LCD_G1: J?.23 (Pin_23)
- net SMEC_LCD_DG2 is gone; now on net SMEC_LCD_G2: J?.24 (Pin_24)
- net SMEC_LCD_DG3 is gone; now on net SMEC_LCD_G3: J?.25 (Pin_25)
- net SMEC_LCD_DG4 is gone; now on net SMEC_LCD_G4: J?.26 (Pin_26)
- net SMEC_LCD_DG5 is gone; now on net SMEC_LCD_G5: J?.27 (Pin_27)
- net SMEC_LCD_DR0 is gone; now on net SMEC_LCD_R0: J?.16 (Pin_16)
- net SMEC_LCD_DR1 is gone; now on net SMEC_LCD_R1: J?.17 (Pin_17)
- net SMEC_LCD_DR2 is gone; now on net SMEC_LCD_R2: J?.18 (Pin_18)
- net SMEC_LCD_DR3 is gone; now on net SMEC_LCD_R3: J?.19 (Pin_19)
- net SMEC_LCD_DR4 is gone; now on net SMEC_LCD_R4: J?.20 (Pin_20)
- net SMEC_LCD_DR5 is gone; now on net SMEC_LCD_R5: J?.21 (Pin_21)
- net SMEC_LCD_DE: now also U?.44 (GPIO_P4_07)
- net SMEC_LCD_HSYNC: now also U?.41 (GPIO_P4_04)
- net SMEC_LCD_PCLK: now also U?.43 (GPIO_P4_06)
- net SMEC_LCD_VSYNC: now also U?.42 (GPIO_P4_05)
- net SMEC_LCD_B0: now reaches U?.11 (GPIO_P1_04)
- net SMEC_LCD_B1: now reaches U?.12 (GPIO_P1_05)
- net SMEC_LCD_B2: now reaches U?.13 (GPIO_P1_06)
- net SMEC_LCD_B3: now reaches U?.14 (GPIO_P1_07)
- net SMEC_LCD_B4: now reaches U?.15 (GPIO_P2_00)
- net SMEC_LCD_B5: now reaches U?.16 (GPIO_P2_01)
- net SMEC_LCD_G0: now reaches U?.19 (GPIO_P2_04)
- net SMEC_LCD_G1: now reaches U?.20 (GPIO_P2_05)
- net SMEC_LCD_G2: now reaches U?.21 (GPIO_P2_06)
- net SMEC_LCD_G3: now reaches U?.22 (GPIO_P2_07)
- net SMEC_LCD_R4: now reaches U?.37 (GPIO_P4_00)
- net SMEC_LCD_R5: now reaches U?.38 (GPIO_P4_01)
- net SMEC_LCD_G4: now reaches U?.25 (GPIO_P3_00)
- net SMEC_LCD_G5: now reaches U?.26 (GPIO_P3_01)
- net SMEC_LCD_R0: now reaches U?.29 (GPIO_P3_04)
- net SMEC_LCD_R1: now reaches U?.30 (GPIO_P3_05)
- net SMEC_LCD_R2: now reaches U?.31 (GPIO_P3_06)
- net SMEC_LCD_R3: now reaches U?.32 (GPIO_P3_07)
Other:
- note added: "MediaCow Touch 2 "Paris" - CTCL 2021-2024"
- note removed: "CTCL 2021-2024"
- note removed: "Reference STMCube32MX file smec.io for pin assignments"
- moved on the sheet: C?, J?, U?, U?A, U?B, U?C, U?D, U?E, U?F, U?I, U?J, U?L
