File: circuits/mct2_buttons/mct2_buttons.kicad_sch (KiCad schematic)
At the start: 35 parts, among them J1 Conn_01x08, SW1 B3F-1052, SW10 B3F-1052, SW11 B3F-1052, SW12 B3F-1052, SW13 OS102011MS2QN1C, SW14 OS102011MS2QN1C, SW2 B3F-1052, SW3 B3F-1052, SW4 B3F-1052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

Commit message: Aug 3, 2024
Connections:
- net COL2: now reaches D1.1 (K), D10.1 (K), D4.1 (K), D7.1 (K)
- net COL2: now also U1.11 (COL2); no longer U1.9 (COL0)
- net COL1: now reaches D11.1 (K), D2.1 (K), D5.1 (K), D8.1 (K), U1.10 (COL1)
- net COL0: now reaches D12.1 (K), D3.1 (K), D6.1 (K), D9.1 (K)
- net COL0: now also U1.9 (COL0); no longer U1.11 (COL2)
Other:
- moved on the sheet: D1, D10, D11, D12, D2, D3, D4, D5, D6, D7, D8, D9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

Commit message: Aug 19, 2024
Parts:
- R1, R2: now not fitted
Other:
- note added: "July 31, 2024 - August 19, 2024"
- note removed: "July 31, 2024 - August 1, 2024"
- note removed: "To STM32U5A5ZJ"
Changed lines of the file:
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@@
 		)
 	)
-	(text "July 31, 2024 - August 1, 2024"
+	(text "July 31, 2024 - August 19, 2024"
 		(exclude_from_sim no)
 		(at 222.504 193.548 0)
@@
 		(exclude_from_sim no)
 		(at 251.714 196.342 0)
-		(effects
-			(font
-				(size 1.27 1.27)
-			)
-		)
-	)
-	(text "To STM32U5A5ZJ"
-		(exclude_from_sim no)
-		(at 273.558 61.468 0)
 		(effects
 			(font
@@
 		(in_bom yes)
 		(on_board yes)
-		(dnp no)
+		(dnp yes)
 		(property "Reference" "R1"
 			(at 239.776 38.354 0)
@@
 		(in_bom yes)
 		(on_board yes)
-		(dnp no)
+		(dnp yes)
 		(property "Reference" "R2"
 			(at 246.126 38.354 0)
@@
 		)
 		(property "Value" "GND"
-			(at 254.762 58.42 0)
-			(effects
-				(font
+			(at 252.984 58.42 90)
+			(effects
+				(font
