File: circuits/mct2_disp/mct2_disp.kicad_pcb (KiCad board)
At the start: 4 copper layers, 50 x 30 mm, 14 parts, among them J1 20455-040E-76, J2 20455-040E-76, J3 Touch Data - I2C, J4 Touch Data - USB, J5 External Backlight Control

Commit message: 20250224-2
Parts:
- moved J4 95.1 mm to (124.7, 84.8), turned to 180 degrees
- moved J3 76.9 mm to (135.0, 84.8), turned to 180 degrees
- moved J5 60.1 mm to (145.3, 84.8), turned to 180 degrees
- moved JP2 54.3 mm to (141.9, 91.3), turned to 90 degrees
- moved JP3 53.0 mm to (148.7, 91.3), turned to 90 degrees
- moved JP1 35.2 mm to (137.6, 92.0)
- moved C1 10.2 mm to (183.6, 93.3)
Connections:
- J5 pad 1: BL_EN_EXT -> BL_PWM_EXT
- J5 pad 2: BL_PWM_EXT -> BL_EN_EXT
Routing:
- net EDP_TX1_N: track 0.00 -> 38.6 mm
- net EDP_TX0_N: track 0.00 -> 38.6 mm
- net EDP_TX1_P: track 0.00 -> 38.6 mm
- net EDP_TX0_P: track 0.00 -> 38.6 mm
- net EDP_AUX_P: track 0.00 -> 38.6 mm
- net EDP_AUX_N: track 0.00 -> 38.6 mm
- net BL_PWM_MU: track 0.00 -> 34.2 mm, vias 0 -> 2
- net BL_EN_MU: track 0.00 -> 26.9 mm, vias 0 -> 2
- net BL_EN: track 0.00 -> 13.0 mm
- net BL_PWM: track 0.00 -> 5.97 mm
- net BL_EN_EXT: track 4.10 -> 7.40 mm
- net BL_PWM_EXT: track 7.68 -> 5.39 mm
Other:
- board text added: "Display"
- board text added: "MediaCow Touch 2 Touchscreen Adapter Board 20250224 - CTCL 2021-2025"
- board text added: "Source"
- board text removed: "MediaCow Touch 2 40p to 40p eDP Touchscreen Adapter Board 20250223 - CTCL 2021-2025"

Commit message: 20250311-1
Parts:
- J1: value 20455-040E-76 -> 20455-030E-76; footprint MediaCow:IPEX_20455-040E-76 -> MediaCow:IPEX_20455-030E-76
- moved R5 62.1 mm to (131.6, 116.7), turned to -90 degrees
- moved J5 50.3 mm to (115.0, 125.0), turned to 0 degrees
- moved JP3 45.7 mm to (112.5, 119.2), turned to -90 degrees
- moved J4 41.4 mm to (135.0, 125.0), turned to 0 degrees
- moved J3 41.4 mm to (125.0, 125.0), turned to 0 degrees
- moved JP2 36.6 mm to (118.4, 119.3), turned to -90 degrees
- moved JP1 28.9 mm to (131.6, 120.2)
- moved J2 21.9 mm to (146.7, 115.0)
- moved J1 20.2 mm to (104.4, 112.5)
Connections:
- J1 pad 10: BL_GND -> EDP_AUX_N
- J1 pad 11: BL_GND -> HS_GND
- J1 pad 12: BL_GND -> LCD_VCC
- J1 pad 13: BL_GND -> LCD_VCC
- J1 pad 14: EDP_HPD -> LCD_BIST
- J1 pad 17: LCD_GND -> EDP_HPD
- J1 pad 18: LCD_GND -> BL_GND
- J1 pad 19: LCD_BIST -> BL_GND
- J1 pad 2: BL_PWR -> HS_GND
- J1 pad 20: LCD_VCC -> BL_GND
- J1 pad 21: LCD_VCC -> BL_GND
- J1 pad 22: LCD_VCC -> BL_EN_MU
- J1 pad 23: LCD_VCC -> BL_PWM_MU
- J1 pad 24: HS_GND -> unconnected-(J1-Pad24)
- J1 pad 25: EDP_AUX_N -> unconnected-(J1-Pad25)
- J1 pad 26: EDP_AUX_P -> BL_PWR
- J1 pad 27: HS_GND -> BL_PWR
- J1 pad 28: EDP_TX0_P -> BL_PWR
- J1 pad 29: EDP_TX0_N -> BL_PWR
- J1 pad 3: BL_PWR -> EDP_TX1_N
- J1 pad 30: HS_GND -> unconnected-(J1-Pad30)
- J1 pad 4: BL_PWR -> EDP_TX1_P
- J1 pad 5: BL_PWR -> HS_GND
- J1 pad 6: unconnected-(J1-Pad6) -> EDP_TX0_N
- J1 pad 7: unconnected-(J1-Pad7) -> EDP_TX0_P
- J1 pad 8: BL_PWM_MU -> HS_GND
- J1 pad 9: BL_EN_MU -> EDP_AUX_P
- J1 pad S1: GND -> Net-(J1-SHIELD-PadS1)
- J1 pad S2: GND -> Net-(J1-SHIELD-PadS1)
- J1 pad S3: GND -> Net-(J1-SHIELD-PadS1)
- J1 pad S4: GND -> Net-(J1-SHIELD-PadS1)
- J2 pad 1: unconnected-(J2-Pad1) -> TP_VCC
- J2 pad 10: EDP_AUX_N -> TP_RST
- J2 pad 11: HS_GND -> unconnected-(J2-Pad11)
- J2 pad 12: LCD_VCC -> BL_PWR
- J2 pad 13: LCD_VCC -> BL_PWR
- J2 pad 14: LCD_BIST -> BL_PWR
- J2 pad 15: LCD_GND -> BL_PWR
- J2 pad 16: LCD_GND -> unconnected-(J2-Pad16)
- J2 pad 17: EDP_HPD -> unconnected-(J2-Pad17)
- J2 pad 18: BL_GND -> BL_PWM
- J2 pad 19: BL_GND -> BL_EN
- J2 pad 2: HS_GND -> TP_RS
- J2 pad 22: BL_EN -> BL_GND
- J2 pad 23: BL_PWM -> BL_GND
- J2 pad 24: unconnected-(J2-Pad24) -> EDP_HPD
- J2 pad 25: unconnected-(J2-Pad25) -> LCD_GND
- J2 pad 26: BL_PWR -> LCD_GND
- J2 pad 27: BL_PWR -> LCD_BIST
- J2 pad 28: BL_PWR -> LCD_VCC
- J2 pad 29: BL_PWR -> LCD_VCC
- J2 pad 3: EDP_TX1_N -> TP_VSS
- J2 pad 30: unconnected-(J2-Pad30) -> HS_GND
- J2 pad 31: TP_RST -> EDP_AUX_N
- J2 pad 32: TP_I2C_SCL -> EDP_AUX_P
- J2 pad 33: TP_I2C_SDA -> HS_GND
- J2 pad 34: TP_INT -> EDP_TX0_P
- J2 pad 35: TP_VSS -> EDP_TX0_N
- J2 pad 36: TP_USB_P -> HS_GND
- J2 pad 37: TP_USB_N -> EDP_TX1_P
- J2 pad 38: TP_VSS -> EDP_TX1_N
- J2 pad 39: TP_RS -> HS_GND
- J2 pad 4: EDP_TX1_P -> TP_USB_N
- J2 pad 40: TP_VCC -> unconnected-(J2-Pad40)
- J2 pad 5: HS_GND -> TP_USB_P
- J2 pad 6: EDP_TX0_N -> TP_VSS
- J2 pad 7: EDP_TX0_P -> TP_INT
- J2 pad 8: HS_GND -> TP_I2C_SDA
- J2 pad 9: EDP_AUX_P -> TP_I2C_SCL
Routing:
- net EDP_TX1_N: track 38.6 -> 0.00 mm
- net EDP_TX0_N: track 38.6 -> 0.00 mm
- net EDP_TX1_P: track 38.6 -> 0.00 mm
- net EDP_TX0_P: track 38.6 -> 0.00 mm
- net EDP_AUX_P: track 38.6 -> 0.00 mm
- net EDP_AUX_N: track 38.6 -> 0.00 mm
- net BL_PWM_MU: track 34.2 -> 6.93 mm, vias 2 -> 0
- net TP_USB_P: track 0.00 -> 17.2 mm
- net TP_USB_N: track 0.00 -> 16.4 mm
- net BL_EN_MU: track 26.9 -> 13.0 mm, vias 2 -> 0
- net BL_EN: track 13.0 -> 0.00 mm
- net BL_PWM: track 5.97 -> 0.00 mm
- net BL_PWM_EXT: track 5.39 -> 3.60 mm
- net BL_EN_EXT: track 7.40 -> 6.64 mm
- net (no net): vias 0 -> 1
