File: circuits/mct2_smec_smd/mct2_smec_smd.kicad_pcb (KiCad board)
At the start: 2 copper layers, 4 parts, among them J1 Input 1x40 FPC, J2 Conn_01x07, J3 Conn_02x15_Odd_Even, U1 GW1N-UV2QN48C7/I6

Commit message: 20250311-1
Parts:
- moved J1 32.1 mm to (147.2, 140.2)
- moved U1 30.2 mm to (161.2, 138.7), turned to 90 degrees
- moved J2 27.0 mm to (160.9, 111.4), turned to 90 degrees
- moved J3 12.4 mm to (217.5, 101.4)
Connections:
- U1 pad 10: RGB_G7 -> RGB_B7
- U1 pad 28: RGB_B0 -> RGB_R0
- U1 pad 29: RGB_B1 -> RGB_R1
- U1 pad 3: RGB_G0 -> RGB_B0
- U1 pad 30: RGB_B2 -> RGB_R2
- U1 pad 31: RGB_B3 -> RGB_R3
- U1 pad 32: RGB_B4 -> RGB_R4
- U1 pad 33: RGB_B5 -> RGB_R5
- U1 pad 34: RGB_B6 -> RGB_R6
- U1 pad 35: RGB_B7 -> RGB_R7
- U1 pad 38: RGB_R0 -> RGB_G0
- U1 pad 39: RGB_R1 -> RGB_G1
- U1 pad 4: RGB_G1 -> RGB_B1
- U1 pad 40: RGB_R2 -> RGB_G2
- U1 pad 41: RGB_R3 -> RGB_G3
- U1 pad 42: RGB_R4 -> RGB_G4
- U1 pad 43: RGB_R5 -> RGB_G5
- U1 pad 44: RGB_R6 -> RGB_G6
- U1 pad 45: RGB_R7 -> RGB_G7
- U1 pad 5: RGB_G2 -> RGB_B2
- U1 pad 6: RGB_G3 -> RGB_B3
- U1 pad 7: RGB_G4 -> RGB_B4
- U1 pad 8: RGB_G5 -> RGB_B5
- U1 pad 9: RGB_G6 -> RGB_B6
Routing:
- net RGB_B7: track 0.00 -> 17.9 mm
- net RGB_B6: track 0.00 -> 17.3 mm
- net RGB_B5: track 0.00 -> 16.7 mm
- net RGB_B4: track 0.00 -> 16.0 mm
- net RGB_B3: track 0.00 -> 15.3 mm
- net RGB_B2: track 0.00 -> 14.7 mm
- net RGB_B1: track 0.00 -> 14.1 mm
- net RGB_B0: track 0.00 -> 13.4 mm
- net RGB_G7: track 20.3 -> 9.75 mm
- net RGB_G6: track 20.0 -> 9.71 mm
- net RGB_G5: track 19.7 -> 9.67 mm
- net RGB_G4: track 19.4 -> 9.67 mm
- net RGB_G3: track 19.1 -> 9.71 mm
- net RGB_G2: track 18.9 -> 9.75 mm
- net RGB_G1: track 18.6 -> 9.79 mm
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Other:
- board outline added: 92 x 30 mm

Commit message: 20250313-1
Parts:
- added U2: ~, Package_TO_SOT_SMD:SOT-23-8, F.Cu at (195.1, 99.9)
- J2: footprint Connector_PinHeader_2.54mm:PinHeader_1x07_P2.54mm_Vertical -> Connector_PinHeader_2.54mm:PinHeader_1x07_P2.54mm_Vertical_SMD_Pin1Left
- moved J3 44.5 mm to (191.0, 137.2)
- moved J2 40.2 mm to (161.8, 151.6), turned to -90 degrees
Connections:
- U1 pad 15: RGB_HSYNC -> RGB_EN
- U1 pad 16: RGB_VSYNC -> RGB_HSYNC
- U1 pad 17: RGB_DE -> RGB_VSYNC
- U1 pad 18: RGB_EN -> RGB_DE
- U1 pad 20: unconnected-(U1F-IOL11A-Pad20) -> MIPI_D0_P
- U1 pad 21: MIPI_TE -> MIPI_D0_N
- U1 pad 22: MIPI_CLK_N -> MIPI_CLK_P
- U1 pad 23: MIPI_CLK_P -> MIPI_CLK_N
- U1 pad 24: MIPI_D0_N -> MIPI_TE
- U1 pad 27: MIPI_D0_P -> unconnected-(U1E-IOL17A-Pad27)
Routing:
- net RGB_DE: track 0.00 -> 30.3 mm
- net RGB_VSYNC: track 0.00 -> 29.1 mm
- net RGB_HSYNC: track 0.00 -> 27.8 mm
- net RGB_EN: track 0.00 -> 26.5 mm
- net RGB_PCLK: track 0.00 -> 25.2 mm
- net (no net): vias 0 -> 1
Other:
- copper layers 2 -> 4
- board text added: "JLC04161H-7628"

Commit message: 20250316-1
Parts:
- removed J2: Conn_01x07, Connector_PinHeader_2.54mm:PinHeader_1x07_P2.54mm_Vertical_SMD_Pin1Left
- U1: value GW1N-UV2QN48C7/I6 -> LIFCL-17-7SG72C; footprint Package_DFN_QFN:QFN-48-1EP_6x6mm_P0.4mm_EP4.2x4.2mm_ThermalVias -> Package_DFN_QFN:QFN-72-1EP_10x10mm_P0.5mm_EP6x6mm_ThermalVias
- moved U1 4.92 mm to (165.2, 141.5), turned to -90 degrees
Connections:
- U1 pad 10: RGB_B7 -> RGB_R2
- U1 pad 11: JTAG_TDO -> RGB_R3
- U1 pad 13: JTAG_MODE0 -> RGB_R4
- U1 pad 14: RGB_PCLK -> RGB_R5
- U1 pad 15: RGB_EN -> RGB_R6
- U1 pad 16: RGB_HSYNC -> RGB_R7
- U1 pad 17: RGB_VSYNC -> unconnected-(U1D-VCCAUXH5-Pad17)
- U1 pad 18: RGB_DE -> unconnected-(U1D-VCCIO5-Pad18)
- U1 pad 19: unconnected-(U1G-IOL6B/GCLKC_7-Pad19) -> RGB_G0
- U1 pad 2: GND -> unconnected-(U1E-DPHY0_DN2-Pad2)
- U1 pad 20: MIPI_D0_P -> RGB_G1
- U1 pad 21: MIPI_D0_N -> unconnected-(U1F-VCC-Pad21)
- U1 pad 22: MIPI_CLK_P -> unconnected-(U1C-PB56A-Pad22)
- U1 pad 23: MIPI_CLK_N -> unconnected-(U1C-PB56B-Pad23)
- U1 pad 24: MIPI_TE -> unconnected-(U1C-PB60A-Pad24)
- U1 pad 26: GND -> unconnected-(U1C-VCCIO3-Pad26)
- U1 pad 28: RGB_R0 -> unconnected-(U1C-PB64B-Pad28)
- U1 pad 29: RGB_R1 -> unconnected-(U1C-VCCAUXH3-Pad29)
- U1 pad 3: RGB_B0 -> MIPI_CLK_N
- U1 pad 30: RGB_R2 -> RGB_B0
- U1 pad 31: RGB_R3 -> RGB_B1
- U1 pad 32: RGB_R4 -> unconnected-(U1C-VCCIO3-Pad32)
- U1 pad 33: RGB_R5 -> RGB_B2
- U1 pad 34: RGB_R6 -> RGB_B3
- U1 pad 35: RGB_R7 -> unconnected-(U1F-VCC-Pad35)
- U1 pad 36: unconnected-(U1A-VCCIO2/VCCX-Pad36) -> RGB_B4
- U1 pad 37: unconnected-(U1A-VCCIO1-Pad37) -> RGB_B5
- U1 pad 38: RGB_G0 -> unconnected-(U1F-VCC-Pad38)
- U1 pad 39: RGB_G1 -> unconnected-(U1F-VCCADC18-Pad39)
- U1 pad 4: RGB_B1 -> MIPI_CLK_P
- U1 pad 40: RGB_G2 -> unconnected-(U1F-VCC-Pad40)
- U1 pad 41: RGB_G3 -> RGB_B6
- U1 pad 42: RGB_G4 -> RGB_B7
- U1 pad 43: RGB_G5 -> RGB_PCLK
- U1 pad 44: RGB_G6 -> RGB_EN
- U1 pad 45: RGB_G7 -> RGB_HSYNC
- U1 pad 46: unconnected-(U1C-IOR1B-Pad46) -> RGB_VSYNC
- U1 pad 48: JTAG_RECONFIG_N -> RGB_DE
- U1 pad 49: (no net) -> unconnected-(U1B-VCCIO1-Pad49)
- U1 pad 5: RGB_B2 -> unconnected-(U1F-VCC-Pad5)
- U1 pad 6: RGB_B3 -> unconnected-(U1F-VCC-Pad6)
- U1 pad 7: RGB_B4 -> unconnected-(U1F-VCCAUX-Pad7)
- U1 pad 8: RGB_B5 -> RGB_R0
- U1 pad 9: RGB_B6 -> RGB_R1
Routing:
- net RGB_G7: track 9.75 -> 0.00 mm
- net RGB_G2: track 9.75 -> 0.00 mm
- net RGB_G3: track 9.71 -> 0.00 mm
- net RGB_G6: track 9.71 -> 0.00 mm
- net RGB_G4: track 9.67 -> 0.00 mm
- net RGB_G5: track 9.67 -> 0.00 mm
- net RGB_DE: track 30.3 -> 22.6 mm
- net RGB_VSYNC: track 29.1 -> 21.7 mm
- net RGB_HSYNC: track 27.8 -> 21.0 mm
- net RGB_EN: track 26.5 -> 20.4 mm
- net RGB_PCLK: track 25.2 -> 19.6 mm
- net RGB_R0: track 17.0 -> 20.9 mm
- net RGB_R1: track 16.4 -> 20.3 mm
- net RGB_R2: track 15.7 -> 19.6 mm
- net RGB_R3: track 15.1 -> 18.8 mm
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