File: mct2_disp/mct2_disp.kicad_pcb (KiCad board)
At the start: 4 copper layers, 50 x 30 mm, 14 parts, among them J1 20455-030E-76, J2 20455-040E-76, J3 Touch Data - I2C, J4 Touch Data - USB, J5 External Backlight Control

Commit message: 20250410-1
Parts:
- added H1: MountingHole, MountingHole:MountingHole_2.7mm_M2.5, F.Cu at (125.5, 101.9)
- added H2: MountingHole, MountingHole:MountingHole_2.7mm_M2.5, F.Cu at (101.5, 128.9)
- added R6: 0R, Resistor_SMD:R_0603_1608Metric, F.Cu at (105.5, 125.9)
- JP2, JP3: footprint Jumper:SolderJumper-3_P1.3mm_Open_Pad1.0x1.5mm -> Jumper:SolderJumper-3_P1.3mm_Open_Pad0.3x0.7mm
- moved JP3 6.69 mm to (117.5, 119.3), turned to -90 degrees
- moved R5 5.64 mm to (137.5, 128.8), turned to 180 degrees
- moved JP1 4.18 mm to (136.7, 127.1), turned to 90 degrees
- moved JP2 3.57 mm to (119.2, 119.2), turned to -90 degrees
- moved J3 2.79 mm to (121.3, 127.1)
- moved J5 2.79 mm to (111.3, 127.1)
- moved J4 2.79 mm to (131.3, 127.1)
- moved R1 0.89 mm to (121.5, 120.2)
- moved R2 0.24 mm to (123.0, 120.1)
Connections:
- C1 pad 2: TP_VSS -> GND
- J1 pad 11: HS_GND -> GND
- J1 pad 15: LCD_GND -> GND
- J1 pad 16: LCD_GND -> GND
- J1 pad 18: BL_GND -> GND
- J1 pad 19: BL_GND -> GND
- J1 pad 2: HS_GND -> GND
- J1 pad 20: BL_GND -> GND
- J1 pad 21: BL_GND -> GND
- J1 pad 5: HS_GND -> GND
- J1 pad 8: HS_GND -> GND
- J2 pad 20: BL_GND -> GND
- J2 pad 21: BL_GND -> GND
- J2 pad 22: BL_GND -> GND
- J2 pad 23: BL_GND -> GND
- J2 pad 25: LCD_GND -> GND
- J2 pad 26: LCD_GND -> GND
- J2 pad 3: TP_VSS -> GND
- J2 pad 30: HS_GND -> GND
- J2 pad 33: HS_GND -> GND
- J2 pad 36: HS_GND -> GND
- J2 pad 39: HS_GND -> GND
- J2 pad 6: TP_VSS -> GND
- J3 pad 3: TP_VSS -> GND
- J3 pad MP: (no net) -> GND
- J4 pad 1: TP_VSS -> GND
- J4 pad 4: TP_VSS -> GND
- J4 pad MP: (no net) -> GND
- J5 pad 3: unconnected-(J5-Pin_3-Pad3) -> GND
- J5 pad 4: unconnected-(J5-Pin_4-Pad4) -> LCD_VCC
- J5 pad 6: unconnected-(J5-Pin_6-Pad6) -> Net-(J5-Pin_6)
- J5 pad MP: (no net) -> GND
- JP1 pad 2: TP_VSS -> GND
Routing:
- net GND: track 0.00 -> 162.8 mm, vias 0 -> 80
- net HS_GND: track 155.4 -> 0.00 mm, vias 72 -> 0
- net TP_VSS: track 34.5 -> 0.00 mm, vias 3 -> 0
- net LCD_VCC: track 0.00 -> 25.1 mm, vias 0 -> 2
- net Net-(J5-Pin_6): track 0.00 -> 7.92 mm, vias 0 -> 2
- net BL_PWM: track 37.7 -> 29.8 mm
- net BL_PWR: track 36.4 -> 44.2 mm, vias 0 -> 2
- net BL_PWM_EXT: track 2.95 -> 10.6 mm
- net TP_VCC: track 14.2 -> 6.77 mm
- net BL_EN_EXT: track 4.50 -> 11.6 mm
- net TP_I2C_SDA: track 28.5 -> 34.2 mm
- net TP_RS: track 6.24 -> 10.8 mm
- net BL_EN: track 32.3 -> 28.1 mm
- net BL_PWM_MU: track 8.63 -> 12.6 mm
- net TP_I2C_SCL: track 30.9 -> 33.7 mm
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- added copper zone on B.Cu, net GND
- added copper zone on F.Cu, net GND
- added copper zone on In1.Cu, net GND
- added copper zone on In2.Cu, net GND
- removed copper zone on In1.Cu, net HS_GND
- removed copper zone on In1.Cu, net TP_VSS
Other:
- outline, holes or cut-outs redrawn
- board text added: "External Backlight Control"
- board text added: "MediaCow Touch 2 Touchscreen Adapter Board 20250402 - CTCL 2021-2025"
- board text added: "Touch Data I2C"
- board text added: "Touch Data USB"
- board text removed: "MediaCow Touch 2 Touchscreen Adapter Board 20250324 - CTCL 2021-2025"
