File: mct2_disp/old/mct2_disp.kicad_sch (KiCad schematic)
At the start: 17 parts, among them J1 20455-030E-76, J2 20455-040E-76, J3 Touch Data - I2C, J4 Touch Data - USB, J5 External Backlight Control

Commit message: 20250410-1
Parts:
- removed H1, H2: MountingHole, MountingHole:MountingHole_2.7mm_M2.5, symbol Mechanical:MountingHole
- removed R6: 0R, Resistor_SMD:R_0603_1608Metric, symbol Device:R_Small
- added H1, H2, H3, H4: MountingHole_Pad, MountingHole:MountingHole_2.2mm_M2_Pad, symbol Mechanical:MountingHole_Pad
- J3, J4, J5: symbol Connector_Generic_MountingPin:Conn_01x06_MountingPin -> Connector:Conn_01x06_Socket
Connections:
- net BL_PWR: now also J5.6 (Pin_6)
- net GND: now also H1.1, H2.1, H3.1, H4.1; no longer C1.2, J1.11, J1.15, J1.16, J1.18, J1.19, J1.2, J1.20, J1.21, J1.5, J1.8, J2.20, J2.21, J2.22, J2.23, J2.25, J2.26, J2.3, J2.30, J2.33, J2.36, J2.39, J2.6, J3.3 (Pin_3), J3.MP (MountPin), J4.1 (Pin_1), J4.4 (Pin_4), J4.MP (MountPin), J5.MP (MountPin), JP1.2 (B)
- new net BL_GND: J1.18, J1.19, J1.20, J1.21, J2.20, J2.21, J2.22, J2.23
- new net HS_GND: J1.11, J1.2, J1.5, J1.8, J2.30, J2.33, J2.36, J2.39
- new net LCD_GND: J1.15, J1.16, J2.25, J2.26
- new net TP_VSS: C1.2, J2.3, J2.6, J3.3 (Pin_3), J4.1 (Pin_1), J4.4 (Pin_4), JP1.2 (B)
Other:
- note added: "February 15, 2025 - April 1, 2025"
- note removed: "February 15, 2025 - April 2, 2025"
- moved on the sheet: J3, J4, J5, R1, R2
