File: lite/circuits/mct2_lite/mct2_lite_power.kicad_sch (KiCad schematic)
At the start: 0 parts

Commit message: 20250410-1
Parts:
- added C? (x16): 220nF, Capacitor_SMD:C_0603_1608Metric, symbol Device:C_Small
- added C?: C_Small, symbol Device:C_Small
- added C? (x5): 1uF, symbol Device:C_Small
- added C? (x4): 22uF, symbol Device:C_Small
- added C? (x4): 220pF, symbol Device:C_Small
- added C? (x4): 10uF, symbol Device:C_Small
- added C? (x16): 100nF, symbol Device:C_Small
- added C? (x8): 10nF, symbol Device:C_Small
- added C? (x2): 100uF, symbol Device:C_Small
- added C? (x2): 22nF, symbol Device:C_Small
- added D? (x2): PPS1045, Package_TO_SOT_SMD:TO-277B, symbol mediacow:PPS1045
- added D?: TBD, symbol Device:D_Zener_Small
- added D?: WP154A4SEJ3VBDZGC/CA, Connector_PinSocket_1.27mm:PinSocket_1x04_P1.27mm_Vertical, symbol Device:LED_RABG
- added J? (x2): USB_C_Receptacle, symbol Connector:USB_C_Receptacle
- added L? (x2): 4.7uF, symbol Device:L_Small
- added Q? (x4): BSZ086P03NS3E, mediacow:Infineon_PG-TSDSON-8, symbol mediacow:BSZ086P03NS3E
- added Q? (x2): T2N7002BK, symbol mediacow:T2N7002BK
- added Q? (x2): NX3008NBKVL, symbol mediacow:NX3008NBKVL
- added R? (x4): 60.4K, symbol Device:R_Small
- added R?: 560K, symbol Device:R_Small
- added R? (x10): 10K, symbol Device:R_Small
- added R? (x3): 4.7K, symbol Device:R_Small
- added R? (x2): 590K, symbol Device:R_Small
- added R? (x5): 3.3K, symbol Device:R_Small
- added R? (x5): 100K, symbol Device:R_Small
- added R? (x4): 0, symbol Device:R_Small
- added R? (x2): 301K, symbol Device:R_Small
- added R? (x2): 499K, symbol Device:R_Small
- added R? (x2): 1K, symbol Device:R_Small
- added R? (x2): 21.5K, symbol Device:R_Small
- added R?: 1.2K, symbol Device:R_Small
- added U? (x4): TPD4USB_EXT30, Package_SON:USON-10_2.5x1.0mm_P0.5mm, symbol mediacow:TPD4EUSB30
- added U?: BTS7006-1EPP, Package_SO:Infineon_PG-TSDSO-14-22, symbol mediacow:BTS7006-1EPP
- added U?: TLV1701, Package_TO_SOT_SMD:SOT-353_SC-70-5, symbol mediacow:TLV1701
- added U? (x2): TPD6S300A, Package_DFN_QFN:WQFN-20-1EP_3x3mm_P0.4mm_EP1.7x1.7mm_ThermalVias, symbol Power_Protection:TPD6S300A
- added U? (x2): MPS8859, mediacow:QFN-16_MP8859, symbol mediacow:MP8859GQ
- added U?: IS31FL3193, Package_DFN_QFN:DFN-10-1EP_3x3mm_P0.5mm_EP1.75x2.7mm, symbol mediacow:IS31FL3193
- added U?: W25Q16JVSS, Package_SO:SOIC-8_5.23x5.23mm_P1.27mm, symbol Memory_Flash:W25Q16JVSS
- added U?: TPS65988DHRSHR, mediacow:QFN_DKRSHR_TEX, symbol MediaCow:TPS65988DHRSHR
- added U?: TLV1701A, Package_TO_SOT_SMD:SOT-353_SC-70-5, symbol mediacow:TLV1701
Connections:
- new net: R?.1, R?.1, R?.2, U?.1 (+) (x2)
- new net: D?.1 (K), R?.1, R?.2
- new net: C?.1, R?.2 (x3)
- new net: C?.2, J?.B3 (TX2-) (x2)
- new net: C?.1, C?.1, C?.1, D?.1 (A), D?.2 (A), Q?.1 (S), Q?.2 (S), Q?.3 (S), R?.1 (x2)
- new net: C?.2, J?.A2 (TX1+) (x2)
- new net: R?.1, U?.2 (IN)
- new net: R?.1, U?.3 (DEN)
- new net: R?.1, R?.1, U?.4 (IS)
- new net: R?.1, R?.2, U?.3 (-) (x2)
- new net: Q?.G (1), R?.2, R?.2, U?.4 (x2)
- new net: C?.2, C?.2, C?.2, Q?.4 (G), Q?.4 (G), R?.1, R?.2 (x2)
- new net: Q?.3 (D), R?.2 (x2)
- new net: C?.1, Q?.5 (D), Q?.5 (D), Q?.6 (D), Q?.6 (D), Q?.7 (D), Q?.7 (D), Q?.8 (D), Q?.8 (D), R?.1, R?.1 (x2)
- new net: C?.2, J?.B10 (RX1-) (x2)
- new net: C?.2, J?.B11 (RX1+) (x2)
- new net: C?.2, J?.A10 (RX2-) (x2)
- new net: C?.2, J?.A11 (RX2+) (x2)
- new net: C?.2, J?.A3 (TX1-) (x2)
- new net: C?.2, J?.B2 (TX2+) (x2)
- new net: C?.1, U?.3 (VBIAS) (x2)
- new net: R?.2, U?.9 (~{FLT}) (x2)
- new net: C?.2, R?.1 (x2)
- new net: R?.2, U?.16 (BST1) (x2)
- new net: Q?.3 (D), Q?.G (1), R?.1, R?.2 (x2)
- new net: R?.1, R?.2, U?.4 (ADD) (x2)
- new net: R?.2, U?.9 (VCC) (x2)
- new net: R?.1, U?.13 (BST2) (x2)
- new net: C?.2, L?.2, U?.14 (SW2) (x2)
- new net: C?.1, L?.1, U?.15 (SW1) (x2)
- new net: C?.1, R?.1, U?.7 (OC) (x2)
- new net: D?.1 (RK), U?.3 (OUT1)
- new net: D?.4 (GK), U?.4 (OUT2)
- new net: D?.3 (BK), U?.5 (OUT3)
- new net GND: C?.2, C?.2, C?.2, C?.2, C?.2, C?.2, C?.2, C?.2, C?.2, C?.2, C?.2, C?.2, C?.2, C?.2, C?.2, C?.2, C?.2, C?.2, C?.2, C?.2, C?.2, C?.2, C?.2, C?.2, C?.2, C?.2, C?.2, C?.2, C?.2, C?.2, C?.2, C?.2, C?.2, C?.2, C?.2, C?.2, D?.2 (A), J?.A1 (GND), J?.A1 (GND), J?.A12 (GND), J?.A12 (GND), J?.B1 (GND), J?.B1 (GND), J?.B12 (GND), J?.B12 (GND), J?.S1 (SHIELD), J?.S1 (SHIELD), Q?.2 (S), Q?.2 (S), Q?.2 (S), Q?.2 (S), R?.1, R?.1, R?.2, R?.2, R?.2, R?.2, R?.2, R?.2, R?.2, R?.2, R?.2, R?.2, U?.1 (GND), U?.10 (AGND), U?.10 (AGND), U?.11 (GND), U?.11 (GND), U?.13 (GND), U?.13 (GND), U?.16 (GND), U?.16 (GND), U?.17 (GND), U?.17 (GND), U?.18 (GND), U?.18 (GND), U?.2 (GND), U?.2 (GND), U?.2 (V-), U?.2 (V-), U?.20 (GND), U?.21 (GND), U?.21 (GND), U?.3 (GND), U?.3 (GND), U?.3 (GND), U?.3 (GND), U?.4 (GND), U?.51 (GND), U?.59 (GND), U?.6 (GND), U?.7 (AD), U?.8 (GND), U?.8 (GND), U?.8 (GND), U?.8 (GND), U?.8 (GND), U?.8 (GND)
- new net LED_3V3: C?.1, C?.1, C?.1, D?.2 (A), U?.2 (VDD)
- new net LED_EN: R?.1, U?.1 (SDB)
- new net LED_VBM: U?.10 (V_BM)
- new net SOM_VSYS: U?.10 (OUT), U?.12 (OUT), U?.13 (OUT), U?.14 (OUT), U?.8 (OUT), U?.9 (OUT)
- new net SYS_I2C_ALT: U?.8 (ALT), U?.8 (ALT)
- new net SYS_I2C_SCL: U?.5 (SCL), U?.5 (SCL), U?.8 (SCL)
- new net SYS_I2C_SDA: U?.6 (SDA), U?.6 (SDA), U?.9 (SDA)
- new net TCP0_CC1: C?.1, U?.4 (C_CC1)
- new net TCP0_CC1_CN: J?.A5 (CC1), U?.12 (CC1), U?.7 (RPD_G1)
- new net TCP0_CC2: C?.1, U?.5 (C_CC2)
- new net TCP0_CC2_CN: J?.B5 (CC2), U?.11 (CC2), U?.6 (RPD_G2)
- new net TCP0_DN: J?.A7 (D-), J?.B7 (D-), U?.19 (D2)
- new net TCP0_DP: J?.A6 (D+), J?.B6 (D+), U?.20 (D1)
- new net TCP0_PPHV: C?.1, C?.1, C?.1, U?.11 (PP_HV1), U?.12 (OUT), U?.12 (PP_HV1)
- new net TCP0_PPHV_EN: U?.3 (EN)
- new net TCP0_SBU1: U?.1 (C_SBU1)
- new net TCP0_SBU1_CN: J?.A8 (SBU1), U?.15 (SBU1), U?.24 (C1_CC1)
- new net TCP0_SBU2: U?.2 (C_SBU2)
- new net TCP0_SBU2_CN: J?.B8 (SBU2), U?.14 (SBU2), U?.26 (C1_CC2)
- new net TCP0_TX0_N: C?.1, U?.2 (D1-)
- new net TCP0_TX0_P: C?.1, U?.1 (D1+)
- new net TCP0_TX1_N: C?.1, U?.2 (D1-)
- new net TCP0_TX1_P: C?.1, U?.1 (D1+)
- new net TCP0_TXRX0_N: C?.1, U?.4 (D2-)
- new net TCP0_TXRX0_P: C?.1, U?.3 (GND)
- new net TCP0_TXRX1_N: C?.1, U?.4 (D2-)
- new net TCP0_TXRX1_P: C?.1, U?.3 (GND)
- new net TCP0_VBUS: C?.1, C?.1, C?.1, C?.1, C?.1, J?.A4 (VBUS), J?.A9 (VBUS), J?.B4 (VBUS), J?.B9 (VBUS), Q?.1 (S), Q?.2 (S), Q?.3 (S)
- new net TCP1_CC1: C?.1, U?.4 (C_CC1)
- new net TCP1_CC1_CN: J?.A5 (CC1), U?.12 (CC1), U?.45 (C2_CC1), U?.7 (RPD_G1)
- new net TCP1_CC2: C?.1, U?.5 (C_CC2)
- new net TCP1_CC2_CN: J?.B5 (CC2), U?.11 (CC2), U?.47 (C2_CC2), U?.6 (RPD_G2)
- new net TCP1_DN: J?.A7 (D-), J?.B7 (D-), U?.19 (D2)
- new net TCP1_DP: J?.A6 (D+), J?.B6 (D+), U?.20 (D1)
- new net TCP1_PPHV: C?.1, C?.1, C?.1, U?.1 (PP_HV2), U?.12 (OUT), U?.2 (PP_HV2)
- new net TCP1_PPHV_EN: U?.3 (EN)
- new net TCP1_SBU1: U?.1 (C_SBU1)
- new net TCP1_SBU1_CN: J?.B8 (SBU2), U?.15 (SBU1)
- new net TCP1_SBU2: U?.2 (C_SBU2)
- new net TCP1_SBU2_CN: J?.A8 (SBU1), U?.14 (SBU2)
- new net TCP1_TX0_N: C?.1, U?.2 (D1-)
- new net TCP1_TX0_P: C?.1, U?.1 (D1+)
- new net TCP1_TX1_N: C?.1, U?.2 (D1-)
- new net TCP1_TX1_P: C?.1, U?.1 (D1+)
- new net TCP1_TXRX0_N: C?.1, U?.4 (D2-)
- new net TCP1_TXRX0_P: C?.1, U?.3 (GND)
- new net TCP1_TXRX1_N: C?.1, U?.4 (D2-)
- new net TCP1_TXRX1_P: C?.1, U?.3 (GND)
- new net TCP1_VBUS: C?.1, C?.1, C?.1, C?.1, C?.1, J?.A4 (VBUS), J?.A9 (VBUS), J?.B4 (VBUS), J?.B9 (VBUS), Q?.1 (S), Q?.2 (S), Q?.3 (S)
- new net TCP_LDO_3V3: C?.1, C?.1, C?.1, C?.1, R?.1, R?.1, R?.1, R?.1, U?.10 (VPWR), U?.10 (VPWR), U?.5 (V+), U?.5 (V+)
- new net TCP_PA_EXT_EN: R?.1
- new net TCP_PB_EXT_EN: R?.1
- new net TCP_SPI_3V3: C?.1, C?.1, R?.1, R?.1, R?.1, R?.1, R?.1, U?.8 (VCC)
- new net TCP_SPI_CLK: U?.38 (SPI_CLK_(GPIO10)), U?.6 (CLK)
- new net TCP_SPI_CS: R?.2, U?.1 (~{CS}), U?.39 (SPI_SS_(GPIO11))
- new net TCP_SPI_HOLD: R?.2, U?.7 (IO3)
- new net TCP_SPI_MISO: R?.2, U?.2 (DO(IO1)), U?.36 (SPI_MISO_(GPIO8))
- new net TCP_SPI_MOSI: R?.2, U?.37 (SPI_MOSI_(GPIO9)), U?.5 (DI(IO0))
- new net TCP_SPI_WP: R?.2, U?.3 (IO2)
- new net VBUS: D?.3 (K), D?.3 (K)
- new net VSYS: U?.1 (IN), U?.1 (IN), U?.15 (VS)
- new net VSYS_SW_DEN: R?.2
- new net VSYS_SW_EN: R?.2
Other:
- note added: "0x62"
- note added: "0x64"
- note added: "2025-03-23 - 2025-04-02"
- note added: "CTCL 2021-2025"
- note added: "MP8859 Address Selection - From MP8859 Rev 1.0 VCC-ADD ADD-GND Address NC NC 0x60 499 301 0x62 301 499 0x64 100 NC 0x66"
- note added: "MediaCow Touch 2 Lite - Power"
- note added: "TCP0_PPHV"
- note added: "TCP1_PPHV"

Commit message: 20250410-2
Parts:
- U?: now fitted
Connections:
- net TCP_ADCIN2: now reaches U?.10 (ADCIN2)
- net TCP_DRAIN1: now reaches U?.15 (DRAIN1)
- net TCP_DRAIN1: now also U?.19 (DRAIN1), U?.58 (DRAIN1), U?.8 (DRAIN1)
- net TCP_DRAIN2: now reaches U?.52 (DRAIN2)
- net TCP_DRAIN2: now also U?.56 (DRAIN2), U?.57 (DRAIN2), U?.7 (DRAIN2)
- net TCP_ADCIN1: now reaches U?.6 (ADCIN1)
- net SYS_I2C_ALT renamed EC_PM_I2C_ALT
- net SYS_I2C_SCL renamed EC_PM_I2C_SCL
- net SYS_I2C_SDA renamed EC_PM_I2C_SDA
Other:
- note added: "2025-03-23 - 2025-04-10"
- note added: "MediaCow Touch 2 Lite "Curitiba" - CTCL 2021-2025"
- note added: "Optional - TCP Config Flash"
- note removed: "2025-03-23 - 2025-04-02"
- note removed: "CTCL 2021-2025"
- moved on the sheet: C?, R?

Commit message: 20250414-1
Other:
- note added: "2025-03-23 - 2025-04-14"
- note removed: "2025-03-23 - 2025-04-10"
- moved on the sheet: C?, R?, U?

Commit message: 20250415-1
Parts:
- J? (x2): footprint (none) -> Connector_USB:USB_C_Receptacle_Molex_105450-0101
Connections:
- net EC_PM_I2C_ALT: now also U?.29 (I2C1_IRQ)
- net EC_PM_I2C_SCL: now also U?.27 (I2C1_SCL)
- net EC_PM_I2C_SDA: now also U?.28 (I2C1_SDA)
- net TCP0_DN: now also U?.53 (C1_USB_N_(GPIO19))
- net TCP0_DP: now also U?.50 (C1_USB_P_(GPIO18))
- net TCP0_VBUS: now also U?.13 (VBUS1), U?.14 (VBUS1)
- net TCP1_DN: now also U?.55 (C2_USB_N_(GPIO21))
- net TCP1_DP: now also U?.54 (C2_USB_P_(GPIO20))
- net TCP1_VBUS: now also U?.3 (VBUS2), U?.4 (VBUS2)
- net TCP_LDO_3V3: now also U?.9 (LDO_3V3)
- net TCP_PP_5V: now reaches U?.25 (PP1_CABLE)
- net TCP_PP_5V: now also U?.46 (PP2_CABLE)
- net TCP_LDO_1V8: now reaches U?.35 (LDO_1V8)
Other:
- note added: "2025-03-23 - 2025-04-15"
- note added: "To-Do: BQ25723 symbol"
- note removed: "2025-03-23 - 2025-04-14"
- moved on the sheet: C?, R?

Commit message: 20250423-1
Changed lines of the file:
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@@
 	(wire
 		(pts
-			(xy 525.78 121.92) (xy 525.78 127)
+			(xy 523.24 121.92) (xy 523.24 127)
 		)
 		(stroke
@@
 	(wire
 		(pts
-			(xy 525.78 121.92) (xy 523.24 121.92)
-		)
-		(stroke
-			(width 0)
-			(type default)
-		)
-	)
-	(wire
-		(pts
 			(xy 532.13 306.07) (xy 543.56 306.07)
 		)
@@
 	(symbol
 		(lib_id "power:GND")
-		(at 525.78 127 0)
+		(at 523.24 127 0)
 		(unit 1)
 		(exclude_from_sim no)
@@
 		(dnp no)
 		(property "Reference" "#PWR034"
-			(at 525.78 133.35 0)
+			(at 523.24 133.35 0)
 			(effects
 				(font
@@
 		)
 		(property "Value" "GND"
-			(at 525.78 130.556 0)
+			(at 523.24 130.556 0)
 			(effects
 				(font
@@
 		)
 		(property "Footprint" ""
-			(at 525.78 127 0)
+			(at 523.24 127 0)
 			(effects
 				(font
@@
 		)
 		(property "Datasheet" ""
-			(at 525.78 127 0)
+			(at 523.24 127 0)
 			(effects
 				(font
@@
 		)
 		(property "Description" "Power symbol creates a global label with name \"GND\" , ground"
-			(at 525.78 127 0)
+			(at 523.24 127 0)
 			(effects
 				(font

Commit message: 20250425-1
Parts:
- added U?: BQ25723, Package_DFN_QFN:Texas_RSN_WQFN-32-1EP_4x4mm_P0.4mm_EP2.8x2.8mm_ThermalVias, symbol mediacow:BQ25723
Other:
- note added: "2025-03-23 - 2025-04-24"
- note removed: "2025-03-23 - 2025-04-15"
- note removed: "To-Do: BQ25723 symbol"
Changed lines of the file:
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@@
 		)
 	)
-	(text "2025-03-23 - 2025-04-15"
+	(text "2025-03-23 - 2025-04-24"
 		(exclude_from_sim no)
 		(at 517.652 403.352 0)
@@
 		)
 	)
-	(text "To-Do: BQ25723 symbol"
-		(exclude_from_sim no)
-		(at 223.774 153.924 0)
-		(effects
-			(font
-				(size 1.27 1.27)
-			)
-		)
-	)
 	(text "MediaCow Touch 2 Lite \"Curitiba\" - CTCL 2021-2025"
 		(exclude_from_sim no)
@@
 					(unit 1)
 				)
+			)
+		)
+	)
+	(symbol
+		(lib_id "mediacow:BQ25723")
+		(at 181.61 151.13 0)
+		(unit 1)
+		(exclude_from_sim no)
+		(in_bom yes)
+		(on_board yes)
+		(dnp no)
+		(property "Reference" "U?"
+			(at 143.002 124.714 0)
+			(effects
+				(font
+					(size 1.27 1.27)
+				)
+				(justify left)
+			)
+		)
+		(property "Value" "BQ25723"
+			(at 211.328 124.46 0)
+			(effects
+				(font
+					(size 1.27 1.27)
+				)
+				(justify left)
+			)
+		)
+		(property "Footprint" "Package_DFN_QFN:Texas_RSN_WQFN-32-1EP_4x4mm_P0.4mm_EP2.8x2.8mm_ThermalVias"
+			(at 140.97 128.27 0)
+			(effects
+				(font
+					(size 1.27 1.27)
+				)
+				(hide yes)
+			)
+		)
+		(property "Datasheet" ""
+			(at 140.97 128.27 0)
+			(effects
+				(font
+					(size 1.27 1.27)
+				)
+				(hide yes)
+			)
+		)
+		(property "Description" ""
+			(at 140.97 128.27 0)
+			(effects
+				(font
+					(size 1.27 1.27)
+				)
+				(hide yes)
+			)
+		)
+		(pin "9"
+		)
+		(pin "32"
+		)
+		(pin "14"
+		)
+		(pin "23"
+		)
+		(pin "26"
+		)
+		(pin "27"
+		)
+		(pin "15"
+		)
+		(pin "13"
+		)
+		(pin "6"
+		)
+		(pin "31"
+		)
+		(pin "17"
+		)
+		(pin "24"
+		)
+		(pin "8"
+		)
+		(pin "11"
+		)
+		(pin "1"
+		)
+		(pin "19"
+		)
+		(pin "5"
+		)
+		(pin "20"
+		)
+		(pin "18"
+		)
+		(pin "4"
+		)
+		(pin "12"
+		)
+		(pin "3"
+		)
+		(pin "28"
+		)
+		(pin "22"
+		)
+		(pin "30"
+		)
+		(pin "2"
+		)
+		(pin "29"
+		)
+		(pin "21"
+		)
+		(pin "10"
+		)
+		(pin "16"
+		)
+		(pin "7"
+		)
+		(pin "25"
+		)
+		(instances
+			(project ""
+				(path "/caf0e9b0-a44c-4a4e-b706-dd9d72690bf9/eb8a2ebe-1a22-48d5-8d40-fed94729eb9b"
+					(reference "U?")
+					(unit 1)
+				)
