File: lite/circuits/mct2_lite/mct2_lite_power.kicad_sch (KiCad schematic)
At the start: 214 parts, among them J5 USB_C_Receptacle, J6 USB_C_Receptacle, Q1 T2N7002BK, Q10 IAUCN04S7L028, Q11 IAUCN04S7L028, Q12 IAUCN04S7L028, Q13 BSC084P03NS3G, Q2 T2N7002BK, Q3 BSZ086P03NS3E, Q4 BSZ086P03NS3E, Q5 NX3008NBKVL, Q6 NX3008NBKVL, Q7 IAUCN04S7L028, Q8 BSZ086P03NS3E, Q9 BSZ086P03NS3E, U10 TLV1701A, U11 TPS65988DHRSHR, U12 TCR3UF105A, U13 BQ25723, U14 TPD6S300A, U15 TPD6S300A, U16 TPD4USB_EXT30, U17 TPD4USB_EXT30, U18 TPD4USB_EXT30, U19 TPD4USB_EXT30, U3 W25Q16JVSS, U4 MPS8859, U5 MPS8859, U6 BTS7006-1EPP, U7 IS31FL3193, U8 TPS560430, U9 TLV1701

Commit message: 20250610-1
Parts:
- L5: value 10uH -> 51uH
- L6: footprint (none) -> Inductor_SMD:L_Chilisin_BMRF00101040
- U8: value TPS560430 -> TPS560430XF
Other:
- moved on the sheet: R46
Changed lines of the file:
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@@
 	)
 	(junction
-		(at 439.42 154.94)
-		(diameter 0)
-		(color 0 0 0 0)
-	)
-	(junction
 		(at 449.58 519.43)
 		(diameter 0)
@@
 	)
 	(junction
+		(at 439.42 154.94)
+		(diameter 0)
+		(color 0 0 0 0)
+	)
+	(junction
 		(at 570.23 283.21)
 		(diameter 0)
@@
 	)
 	(junction
+		(at 530.86 488.95)
+		(diameter 0)
+		(color 0 0 0 0)
+	)
+	(junction
 		(at 562.61 246.38)
 		(diameter 0)
@@
 	)
 	(junction
-		(at 523.24 488.95)
-		(diameter 0)
-		(color 0 0 0 0)
-	)
-	(junction
 		(at 515.62 447.04)
 		(diameter 0)
@@
 	(wire
 		(pts
-			(xy 523.24 495.3) (xy 523.24 488.95)
+			(xy 530.86 495.3) (xy 530.86 488.95)
 		)
 		(stroke
@@
 	(wire
 		(pts
-			(xy 508 488.95) (xy 513.08 488.95)
+			(xy 515.62 488.95) (xy 520.7 488.95)
 		)
 		(stroke
@@
 	(wire
 		(pts
-			(xy 528.32 482.6) (xy 530.86 482.6)
-		)
-		(stroke
-			(width 0)
-			(type default)
-		)
-	)
-	(wire
-		(pts
 			(xy 530.86 436.88) (xy 518.16 436.88)
 		)
@@
 	(wire
 		(pts
-			(xy 508 495.3) (xy 523.24 495.3)
+			(xy 515.62 495.3) (xy 530.86 495.3)
 		)
 		(stroke
@@
 	(wire
 		(pts
-			(xy 528.32 488.95) (xy 528.32 482.6)
+			(xy 530.86 488.95) (xy 530.86 482.6)
 		)
 		(stroke
@@
 	(wire
 		(pts
-			(xy 523.24 488.95) (xy 528.32 488.95)
-		)
-		(stroke
-			(width 0)
-			(type default)
-		)
-	)
-	(wire
-		(pts
 			(xy 693.42 220.98) (xy 704.85 220.98)
 		)
@@
 	(wire
 		(pts
-			(xy 518.16 488.95) (xy 523.24 488.95)
-		)
-		(stroke
-			(width 0)
-			(type default)
-		)
-	)
-	(wire
-		(pts
 			(xy 524.51 410.21) (xy 530.86 410.21)
 		)
@@
 	(wire
 		(pts
-			(xy 439.42 154.94) (xy 443.23 154.94)
-		)
-		(stroke
-			(width 0)
-			(type default)
-		)
-	)
-	(wire
-		(pts
 			(xy 636.27 254) (xy 643.89 254)
 		)
@@
 	(wire
 		(pts
+			(xy 530.86 488.95) (xy 525.78 488.95)
+		)
+		(stroke
+			(width 0)
+			(type default)
+		)
+	)
+	(wire
+		(pts
 			(xy 792.48 330.2) (xy 795.02 330.2)
 		)
@@
 	(wire
 		(pts
+			(xy 439.42 154.94) (xy 443.23 154.94)
+		)
+		(stroke
+			(width 0)
+			(type default)
+		)
+	)
+	(wire
+		(pts
 			(xy 601.98 247.65) (xy 601.98 246.38)
 		)
@@
 	(global_label "SOM_PROCHOT"
 		(shape input)
-		(at 508 495.3 180)
+		(at 515.62 495.3 180)
 		(fields_autoplaced yes)
 		(effects
@@
 		)
 		(property "Intersheetrefs" "${INTERSHEET_REFS}"
-			(at 491.2867 495.3 0)
+			(at 498.9067 495.3 0)
 			(effects
 				(font
@@
 	(global_label "BM_1V05"
 		(shape input)
-		(at 508 488.95 180)
+		(at 515.62 488.95 180)
 		(fields_autoplaced yes)
 		(effects
@@
 		)
 		(property "Intersheetrefs" "${INTERSHEET_REFS}"
-			(at 496.6087 488.95 0)
+			(at 504.2287 488.95 0)
 			(effects
 				(font
@@
 	)
 	(symbol
+		(lib_name "mediacow:TPD4EUSB30")
 		(lib_id "mediacow:TPD4EUSB30")
 		(at 755.65 269.24 0)
@@
 		(dnp no)
 		(property "Reference" "C57"
-			(at 435.61 515.366 0)
+			(at 436.372 515.366 0)
 			(effects
 				(font
@@
 		(dnp no)
 		(property "Reference" "L5"
-			(at 441.96 517.906 90)
+			(at 440.182 520.446 90)
 			(effects
 				(font
@@
 			)
 		)
-		(property "Value" "10uH"
-			(at 445.77 517.906 90)
+		(property "Value" "51uH"
+			(at 445.008 520.446 90)
 			(effects
 				(font
@@
 		)
 		(property "Value" "BTS7006-1EPP"
-			(at 347.726 130.81 0)
+			(at 346.71 130.81 0)
 			(effects
 				(font
@@
 		(dnp no)
 		(property "Reference" "R10"
-			(at 319.024 131.064 0)
+			(at 318.516 131.064 0)
 			(effects
 				(font
@@
 		(dnp no)
 		(property "Reference" "C83"
-			(at 512.572 471.17 90)
+			(at 512.826 473.456 90)
 			(effects
 				(font
@@
 		)
 		(property "Value" "33pF"
-			(at 518.922 471.17 90)
+			(at 518.922 473.456 90)
 			(effects
 				(font
@@
 		(dnp no)
 		(property "Reference" "C79"
-			(at 512.572 481.584 90)
+			(at 507.492 483.616 90)
 			(effects
 				(font
@@
 		)
 		(property "Value" "1.2nF"
-			(at 510.54 485.394 90)
+			(at 514.096 483.616 90)
 			(effects
 				(font
@@
 		(dnp no)
 		(property "Reference" "Q11"
-			(at 592.836 425.704 90)
+			(at 593.344 425.45 90)
 			(effects
 				(font
@@
 		(dnp no)
 		(property "Reference" "C84"
-			(at 512.572 476.25 90)
+			(at 512.826 476.504 90)
 			(effects
 				(font
@@
 		)
 		(property "Value" "15pF"
-			(at 518.922 476.25 90)
+			(at 518.922 476.504 90)
 			(effects
 				(font
@@
 			)
 		)
-		(property "Value" "TPS560430"
+		(property "Value" "TPS560430XF"
 			(at 424.18 510.794 0)
 			(effects
@@
 		(dnp no)
 		(property "Reference" "C78"
-			(at 507.492 466.344 90)
+			(at 507.746 466.344 90)
 			(effects
 				(font
@@
 		)
 		(property "Value" "3.3nF"
-			(at 510.54 464.312 90)
+			(at 514.096 466.344 90)
 			(effects
 				(font
@@
 		(dnp no)
 		(property "Reference" "R49"
-			(at 517.652 481.584 90)
+			(at 520.446 480.822 90)
 			(effects
 				(font
@@
 	)
 	(symbol
+		(lib_name "mediacow:TPD4EUSB30")
 		(lib_id "mediacow:TPD4EUSB30")
 		(at 778.51 269.24 0)
@@
 	)
 	(symbol
+		(lib_name "mediacow:TPD4EUSB30")
 		(lib_id "mediacow:TPD4EUSB30")
 		(at 778.51 157.48 0)
@@
 		(dnp no)
 		(property "Reference" "R48"
-			(at 516.89 466.344 90)
+			(at 520.446 469.392 90)
 			(effects
 				(font
@@
 		)
 		(property "Value" "16.9K"
-			(at 520.7 464.312 90)
+			(at 520.7 465.328 90)
 			(effects
 				(font
@@
 	(symbol
 		(lib_id "Device:R_Small")
-		(at 515.62 488.95 90)
+		(at 523.24 488.95 90)
 		(unit 1)
 		(exclude_from_sim no)
@@
 		(dnp no)
 		(property "Reference" "R46"
-			(at 512.318 490.22 90)
+			(at 519.938 490.22 90)
 			(effects
 				(font
@@
 		)
 		(property "Value" "50"
-			(at 518.668 490.22 90)
+			(at 526.288 490.22 90)
 			(effects
 				(font
@@
 		)
 		(property "Footprint" "Resistor_SMD:R_0603_1608Metric"
-			(at 515.62 488.95 0)
+			(at 523.24 488.95 0)
 			(effects
 				(font
@@
 		)
 		(property "Datasheet" "~"
-			(at 515.62 488.95 0)
+			(at 523.24 488.95 0)
 			(effects
 				(font
@@
 		)
 		(property "Description" "Resistor, small symbol"
-			(at 515.62 488.95 0)
+			(at 523.24 488.95 0)
 			(effects
 				(font
@@
 		(dnp no)
 		(property "Reference" "C98"
-			(at 575.31 421.386 0)
+			(at 573.786 421.386 0)
 			(effects
 				(font
@@
 	)
 	(symbol
+		(lib_name "mediacow:TPD4EUSB30")
 		(lib_id "mediacow:TPD4EUSB30")
 		(at 755.65 157.48 0)
@@
 		(dnp no)
 		(property "Reference" "R13"
-			(at 319.786 120.904 90)
+			(at 318.516 120.904 90)
 			(effects
 				(font
@@
 			)
 		)
-		(property "Footprint" ""
+		(property "Footprint" "Inductor_SMD:L_Chilisin_BMRF00101040"
 			(at 571.5 410.21 0)
 			(effects

Commit message: 20250628-1
Parts:
- renumbered D1 to U?
Connections:
- net EC_IOVDD: now also R62.1
- net GND: now also R63.2
Other:
- moved on the sheet: R58, R59, R60, R61, R62, R63

Commit message: 20250712-1 mv docs from website to repo
Parts:
- removed R10, R13: 4.7K, Resistor_SMD:R_0603_1608Metric, symbol Device:R_Small
- removed R14: 100K, Resistor_SMD:R_0603_1608Metric, symbol Device:R_Small
- removed U6: BTS7006-1EPP, Package_SO:Infineon_PG-TSDSO-14-22, symbol mediacow:BTS7006-1EPP
Other:
- note removed: "SoM Load Switch"
- moved on the sheet: C39, C40, C41, C42, C43, C44, C45, C46, C47, C48, C49, C50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
