File: lite/circuits/mct2_lite/mct2_lite_io.kicad_sch (KiCad schematic)
At the start: 0 parts

Commit message: 20250410-1
Parts:
- added C? (x2): 120uF, symbol Device:C_Small
- added C? (x3): 100nF, symbol Device:C_Small
- added J?: HDMI_A, symbol Connector:HDMI_A
- added J? (x2): USB3_A, symbol Connector:USB3_A
- added R? (x2): 56K, symbol Device:R_Small
- added R? (x2): 20K, symbol Device:R_Small
- added TP?: TestPoint_Alt, symbol Connector:TestPoint_Alt
- added U? (x2): TPS25221, Package_SON:WSON-6-1EP_2x2mm_P0.65mm_EP1x1.6mm, symbol mediacow:TPS25221
- added U?: TPD12S016RKTR, RKT24, symbol mediacow:TPD12S016RKTR
Connections:
- new net: R?.1, U?.5 (ILIM) (x2)
- new net: C?.1, J?.1 (VBUS), U?.6 (OUT) (x2)
- new net GND: C?.2, C?.2, C?.2, C?.2, C?.2, J?.10 (SHIELD), J?.10 (SHIELD), J?.4 (GND), J?.4 (GND), J?.7 (DRAIN), J?.7 (DRAIN), R?.2, R?.2, R?.2, R?.2, U?.13 (GND), U?.18 (GND), U?.2 (GND), U?.2 (GND), U?.5 (GND)
- new net HDMI_5V: U?.10 (VCC5V)
- new net HDMI_5V_CN: C?.1, J?.18 (+5V), U?.12 (5V_OUT)
- new net HDMI_CEC: U?.24 (CEC_A)
- new net HDMI_CLKN: J?.12 (CK-), U?.14 (CLK-)
- new net HDMI_CLKP: J?.10 (CK+), U?.15 (CLK+)
- new net HDMI_CN_CEC: J?.13 (CEC), U?.6 (CEC_B)
- new net HDMI_CN_HPD: J?.19 (HPD), U?.9 (HPD_B)
- new net HDMI_CN_SCL: J?.15 (SCL), U?.7 (SCL_B)
- new net HDMI_CN_SDA: J?.16 (SDA), U?.8 (SDA_B)
- new net HDMI_CT_HPD: U?.11 (CT_HPD)
- new net HDMI_D0N: J?.9 (D0-), U?.16 (D0-)
- new net HDMI_D0P: J?.7 (D0+), U?.17 (D0+)
- new net HDMI_D1N: J?.6 (D1-), U?.19 (D1-)
- new net HDMI_D1P: J?.4 (D1+), U?.20 (D1+)
- new net HDMI_D2N: J?.3 (D2-), U?.21 (D2-)
- new net HDMI_D2P: J?.1 (D2+), U?.22 (D2+)
- new net HDMI_HPD: U?.3 (HPD_A)
- new net HDMI_LS_OE: U?.4 (LS_OE)
- new net HDMI_SCL: U?.1 (SCL_A)
- new net HDMI_SDA: U?.2 (SDA_A)
- new net HDMI_UTILITY: J?.14 (UTILITY), TP?.1
- new net HDMI_VCCA: U?.23 (VCCA)
- new net USB_5V: C?.1, C?.1, U?.1 (IN), U?.1 (IN)
- new net USB_EXT1_EN: R?.1, R?.1, U?.3 (EN), U?.3 (EN)
- new net USB_EXT1_FLT: U?.4 (FAULT), U?.4 (FAULT)
Other:
- note added: "2025-03-23 - 2025-03-29"
- note added: "CTCL 2021-2025"
- note added: "MediaCow Touch 2 Lite - IO"

Commit message: 20250410-2
Other:
- note added: "2025-03-23 - 2025-04-10"
- note added: "HDMI"
- note added: "MediaCow Touch 2 Lite "Curitiba" - CTCL 2021-2025"
- note removed: "2025-03-23 - 2025-03-29"
- note removed: "CTCL 2021-2025"
Changed lines of the file:
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@@
+		)
+	)
+	(rectangle
+		(start 279.4 152.4)
+		(end 406.4 241.3)
+		(stroke
+			(width 0)
+			(type default)
+		)
+		(fill
+			(type none)
 		)
 	)
@@
 		)
 	)
-	(text "2025-03-23 - 2025-03-29"
+	(text "2025-03-23 - 2025-04-10"
 		(exclude_from_sim no)
 		(at 343.916 280.416 0)
@@
 		)
 	)
-	(text "CTCL 2021-2025"
+	(text "MediaCow Touch 2 Lite \"Curitiba\" - CTCL 2021-2025"
 		(exclude_from_sim no)
-		(at 309.118 267.462 0)
+		(at 327.406 266.954 0)
 		(effects
 			(font
@@
 			)
 		)
+	)
+	(text "HDMI"
+		(exclude_from_sim no)
+		(at 284.48 150.368 0)
+		(effects
+			(font
+				(size 2.54 2.54)
+			)
+		)

Commit message: 20250414-1
Parts:
- added C? (x8): 100nF, symbol Device:C_Small
- added R? (x4): 0, symbol Device:R_Small
Connections:
- net USB_EXT1_EN: no longer R?.1, U?.3 (EN)
- net USB_EXT1_FLT: no longer U?.4 (FAULT)
- net USB_EXT1_USB2_N: now reaches J?.2 (D-)
- net USB_EXT1_USB2_N: now also R?.2
- net USB_EXT1_USB2_P: now reaches J?.3 (D+)
- net USB_EXT1_USB2_P: now also R?.2
- net USB_EXT1_SSRX0_N: now reaches J?.5 (SSRX-)
- net USB_EXT1_SSRX0_N: now also C?.2
- net USB_EXT1_SSRX0_P: now reaches J?.6 (SSRX+)
- net USB_EXT1_SSRX0_P: now also C?.2
- net USB_EXT1_SSRX1_N: now reaches J?.8 (SSTX-)
- net USB_EXT1_SSRX1_N: now also C?.2
- net USB_EXT1_SSRX1_P: now reaches J?.9 (SSTX+)
- net USB_EXT1_SSRX1_P: now also C?.2
- net USB_EXT0_USB2_N: now reaches J?.2 (D-)
- net USB_EXT0_USB2_N: now also R?.2
- net USB_EXT0_USB2_P: now reaches J?.3 (D+)
- net USB_EXT0_USB2_P: now also R?.2
- net USB_EXT0_SSRX0_N: now reaches J?.5 (SSRX-)
- net USB_EXT0_SSRX0_N: now also C?.2
- net USB_EXT0_SSRX0_P: now reaches J?.6 (SSRX+)
- net USB_EXT0_SSRX0_P: now also C?.2
- net USB_EXT0_SSRX1_N: now reaches J?.8 (SSTX-)
- net USB_EXT0_SSRX1_N: now also C?.2
- net USB_EXT0_SSRX1_P: now reaches J?.9 (SSTX+)
- net USB_EXT0_SSRX1_P: now also C?.2
- new net SOM_HSIO0_RX_N: C?.1
- new net SOM_HSIO0_RX_P: C?.1
- new net SOM_HSIO0_TX_N: C?.1
- new net SOM_HSIO0_TX_P: C?.1
- new net SOM_HSIO1_RX_N: C?.1
- new net SOM_HSIO1_RX_P: C?.1
- new net SOM_HSIO1_TX_N: C?.1
- new net SOM_HSIO1_TX_P: C?.1
- new net SOM_USB2_P1_N: R?.1
- new net SOM_USB2_P1_P: R?.1
- new net SOM_USB2_P2_N: R?.1
- new net SOM_USB2_P2_P: R?.1
- new net USB_EXT0_EN: R?.1, U?.3 (EN)
- new net USB_EXT0_FLT: U?.4 (FAULT)
Other:
- note added: "2025-03-23 - 2025-04-14"
- note removed: "2025-03-23 - 2025-04-10"
- moved on the sheet: C?, R?, U?

Commit message: 20250415-1
Other:
- note added: "2025-03-23 - 2025-04-15"
- note removed: "2025-03-23 - 2025-04-14"
Changed lines of the file:
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@@
 		)
 	)
-	(text "2025-03-23 - 2025-04-14"
+	(text "2025-03-23 - 2025-04-15"
 		(exclude_from_sim no)
 		(at 343.916 280.416 0)
@@
 	(label "HDMI_CN_SCL"
 		(at 344.17 201.93 0)
+		(fields_autoplaced yes)
 		(effects
 			(font
@@
 	(label "USB_EXT0_USB2_N"
 		(at 349.25 30.48 0)
+		(fields_autoplaced yes)
 		(effects
 			(font
@@
 	(label "USB_EXT1_SSRX0_P"
 		(at 350.52 86.36 0)
+		(fields_autoplaced yes)
 		(effects
 			(font
@@
 	(label "USB_EXT1_SSRX0_N"
 		(at 350.52 83.82 0)
+		(fields_autoplaced yes)
 		(effects
 			(font
@@
 	(label "HDMI_CLKP"
 		(at 344.17 194.31 0)
+		(fields_autoplaced yes)
 		(effects
 			(font
@@
 	(label "HDMI_CLKN"
 		(at 344.17 196.85 0)
+		(fields_autoplaced yes)
 		(effects
 			(font
@@
 	(label "HDMI_CN_SDA"
 		(at 344.17 204.47 0)
+		(fields_autoplaced yes)
 		(effects
 			(font
@@
 	(label "HDMI_D2N"
 		(at 344.17 181.61 0)
+		(fields_autoplaced yes)
 		(effects
 			(font
@@
 	(label "USB_EXT0_SSRX0_P"
 		(at 349.25 40.64 0)
+		(fields_autoplaced yes)
 		(effects
 			(font
@@
 	(label "HDMI_D0P"
 		(at 344.17 189.23 0)
+		(fields_autoplaced yes)
 		(effects
 			(font
@@
 	(label "USB_EXT1_USB2_P"
 		(at 350.52 78.74 0)
+		(fields_autoplaced yes)
 		(effects
 			(font
@@
 	(label "USB_EXT1_SSRX1_P"
 		(at 350.52 93.98 0)
+		(fields_autoplaced yes)
 		(effects
 			(font
@@
 	(label "HDMI_UTILITY"
 		(at 365.76 214.63 0)
+		(fields_autoplaced yes)
 		(effects
 			(font
@@
 	(label "USB_EXT0_SSRX1_P"
 		(at 349.25 48.26 0)
+		(fields_autoplaced yes)
 		(effects
 			(font
@@
 	(label "HDMI_CN_CEC"
 		(at 344.17 199.39 0)
+		(fields_autoplaced yes)
 		(effects
 			(font
@@
 	(label "USB_EXT0_USB2_P"
 		(at 349.25 33.02 0)
+		(fields_autoplaced yes)
 		(effects
 			(font
@@
 	(label "USB_EXT1_USB2_N"
 		(at 350.52 76.2 0)
+		(fields_autoplaced yes)
 		(effects
 			(font
@@
 	(label "USB_EXT1_SSRX1_N"
 		(at 350.52 91.44 0)
+		(fields_autoplaced yes)
 		(effects
 			(font
@@
 	(label "HDMI_D2P"
 		(at 344.17 179.07 0)
+		(fields_autoplaced yes)
 		(effects
 			(font
@@
 	(label "HDMI_CN_HPD"
 		(at 344.17 207.01 0)
+		(fields_autoplaced yes)
 		(effects
 			(font
@@
 	(label "USB_EXT0_SSRX0_N"
 		(at 349.25 38.1 0)
+		(fields_autoplaced yes)
 		(effects
 			(font
@@
 	(label "HDMI_D1P"
 		(at 344.17 184.15 0)
+		(fields_autoplaced yes)
 		(effects
 			(font
@@
 	(label "USB_EXT0_SSRX1_N"
 		(at 349.25 45.72 0)
+		(fields_autoplaced yes)
 		(effects
 			(font
@@
 	(label "HDMI_D1N"
 		(at 344.17 186.69 0)
+		(fields_autoplaced yes)
 		(effects
 			(font
@@
 	(label "HDMI_D0N"
 		(at 344.17 191.77 0)
-		(effects
-			(font
+		(fields_autoplaced yes)
+		(effects
+			(font

Commit message: 20250426-1 Remove current codename
Other:
- note added: "MediaCow Touch 2 Lite - CTCL 2021-2025"
- note removed: "MediaCow Touch 2 Lite "Curitiba" - CTCL 2021-2025"
Changed lines of the file:
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@@
 		)
 	)
-	(text "MediaCow Touch 2 Lite \"Curitiba\" - CTCL 2021-2025"
+	(text "MediaCow Touch 2 Lite - CTCL 2021-2025"
 		(exclude_from_sim no)
-		(at 327.406 266.954 0)
+		(at 322.326 266.7 0)
 		(effects
 			(font
@@
 	(label "HDMI_CN_SCL"
 		(at 344.17 201.93 0)
-		(fields_autoplaced yes)
 		(effects
 			(font
@@
 	(label "USB_EXT0_USB2_N"
 		(at 349.25 30.48 0)
-		(fields_autoplaced yes)
 		(effects
 			(font
@@
 	(label "USB_EXT1_SSRX0_P"
 		(at 350.52 86.36 0)
-		(fields_autoplaced yes)
 		(effects
 			(font
@@
 	(label "USB_EXT1_SSRX0_N"
 		(at 350.52 83.82 0)
-		(fields_autoplaced yes)
 		(effects
 			(font
@@
 	(label "HDMI_CLKP"
 		(at 344.17 194.31 0)
-		(fields_autoplaced yes)
 		(effects
 			(font
@@
 	(label "HDMI_CLKN"
 		(at 344.17 196.85 0)
-		(fields_autoplaced yes)
 		(effects
 			(font
@@
 	(label "HDMI_CN_SDA"
 		(at 344.17 204.47 0)
-		(fields_autoplaced yes)
 		(effects
 			(font
@@
 	(label "HDMI_D2N"
 		(at 344.17 181.61 0)
-		(fields_autoplaced yes)
 		(effects
 			(font
@@
 	(label "USB_EXT0_SSRX0_P"
 		(at 349.25 40.64 0)
-		(fields_autoplaced yes)
 		(effects
 			(font
@@
 	(label "HDMI_D0P"
 		(at 344.17 189.23 0)
-		(fields_autoplaced yes)
 		(effects
 			(font
@@
 	(label "USB_EXT1_USB2_P"
 		(at 350.52 78.74 0)
-		(fields_autoplaced yes)
 		(effects
 			(font
@@
 	(label "USB_EXT1_SSRX1_P"
 		(at 350.52 93.98 0)
-		(fields_autoplaced yes)
 		(effects
 			(font
@@
 	(label "HDMI_UTILITY"
 		(at 365.76 214.63 0)
-		(fields_autoplaced yes)
 		(effects
 			(font
@@
 	(label "USB_EXT0_SSRX1_P"
 		(at 349.25 48.26 0)
-		(fields_autoplaced yes)
 		(effects
 			(font
@@
 	(label "HDMI_CN_CEC"
 		(at 344.17 199.39 0)
-		(fields_autoplaced yes)
 		(effects
 			(font
@@
 	(label "USB_EXT0_USB2_P"
 		(at 349.25 33.02 0)
-		(fields_autoplaced yes)
 		(effects
 			(font
@@
 	(label "USB_EXT1_USB2_N"
 		(at 350.52 76.2 0)
-		(fields_autoplaced yes)
 		(effects
 			(font
@@
 	(label "USB_EXT1_SSRX1_N"
 		(at 350.52 91.44 0)
-		(fields_autoplaced yes)
 		(effects
 			(font
@@
 	(label "HDMI_D2P"
 		(at 344.17 179.07 0)
-		(fields_autoplaced yes)
 		(effects
 			(font
@@
 	(label "HDMI_CN_HPD"
 		(at 344.17 207.01 0)
-		(fields_autoplaced yes)
 		(effects
 			(font
@@
 	(label "USB_EXT0_SSRX0_N"
 		(at 349.25 38.1 0)
-		(fields_autoplaced yes)
 		(effects
 			(font
@@
 	(label "HDMI_D1P"
 		(at 344.17 184.15 0)
-		(fields_autoplaced yes)
 		(effects
 			(font
@@
 	(label "USB_EXT0_SSRX1_N"
 		(at 349.25 45.72 0)
-		(fields_autoplaced yes)
 		(effects
 			(font
@@
 	(label "HDMI_D1N"
 		(at 344.17 186.69 0)
-		(fields_autoplaced yes)
 		(effects
 			(font
@@
 	(label "HDMI_D0N"
 		(at 344.17 191.77 0)
-		(fields_autoplaced yes)
-		(effects
-			(font
+		(effects
+			(font

Commit message: 20250504-1
Other:
- note added: "2025-03-23 - 2025-04-29"
- note added: "MediaCow Touch 2 Lite "Curitiba" - CTCL 2021-2025"
- note removed: "2025-03-23 - 2025-04-15"
- note removed: "MediaCow Touch 2 Lite - CTCL 2021-2025"
Changed lines of the file:
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@@
 		)
 	)
-	(text "2025-03-23 - 2025-04-15"
+	(text "2025-03-23 - 2025-04-29\n"
 		(exclude_from_sim no)
 		(at 343.916 280.416 0)
@@
 		)
 	)
-	(text "MediaCow Touch 2 Lite - CTCL 2021-2025"
+	(text "MediaCow Touch 2 Lite \"Curitiba\" - CTCL 2021-2025"
 		(exclude_from_sim no)
-		(at 322.326 266.7 0)
+		(at 327.406 266.954 0)
 		(effects
 			(font
@@
 	(label "HDMI_CN_SCL"
 		(at 344.17 201.93 0)
+		(fields_autoplaced yes)
 		(effects
 			(font
@@
 	(label "USB_EXT0_USB2_N"
 		(at 349.25 30.48 0)
+		(fields_autoplaced yes)
 		(effects
 			(font
@@
 	(label "USB_EXT1_SSRX0_P"
 		(at 350.52 86.36 0)
+		(fields_autoplaced yes)
 		(effects
 			(font
@@
 	(label "USB_EXT1_SSRX0_N"
 		(at 350.52 83.82 0)
+		(fields_autoplaced yes)
 		(effects
 			(font
@@
 	(label "HDMI_CLKP"
 		(at 344.17 194.31 0)
+		(fields_autoplaced yes)
 		(effects
 			(font
@@
 	(label "HDMI_CLKN"
 		(at 344.17 196.85 0)
+		(fields_autoplaced yes)
 		(effects
 			(font
@@
 	(label "HDMI_CN_SDA"
 		(at 344.17 204.47 0)
+		(fields_autoplaced yes)
 		(effects
 			(font
@@
 	(label "HDMI_D2N"
 		(at 344.17 181.61 0)
+		(fields_autoplaced yes)
 		(effects
 			(font
@@
 	(label "USB_EXT0_SSRX0_P"
 		(at 349.25 40.64 0)
+		(fields_autoplaced yes)
 		(effects
 			(font
@@
 	(label "HDMI_D0P"
 		(at 344.17 189.23 0)
+		(fields_autoplaced yes)
 		(effects
 			(font
@@
 	(label "USB_EXT1_USB2_P"
 		(at 350.52 78.74 0)
+		(fields_autoplaced yes)
 		(effects
 			(font
@@
 	(label "USB_EXT1_SSRX1_P"
 		(at 350.52 93.98 0)
+		(fields_autoplaced yes)
 		(effects
 			(font
@@
 	(label "HDMI_UTILITY"
 		(at 365.76 214.63 0)
+		(fields_autoplaced yes)
 		(effects
 			(font
@@
 	(label "USB_EXT0_SSRX1_P"
 		(at 349.25 48.26 0)
+		(fields_autoplaced yes)
 		(effects
 			(font
@@
 	(label "HDMI_CN_CEC"
 		(at 344.17 199.39 0)
+		(fields_autoplaced yes)
 		(effects
 			(font
@@
 	(label "USB_EXT0_USB2_P"
 		(at 349.25 33.02 0)
+		(fields_autoplaced yes)
 		(effects
 			(font
@@
 	(label "USB_EXT1_USB2_N"
 		(at 350.52 76.2 0)
+		(fields_autoplaced yes)
 		(effects
 			(font
@@
 	(label "USB_EXT1_SSRX1_N"
 		(at 350.52 91.44 0)
+		(fields_autoplaced yes)
 		(effects
 			(font
@@
 	(label "HDMI_D2P"
 		(at 344.17 179.07 0)
+		(fields_autoplaced yes)
 		(effects
 			(font
@@
 	(label "HDMI_CN_HPD"
 		(at 344.17 207.01 0)
+		(fields_autoplaced yes)
 		(effects
 			(font
@@
 	(label "USB_EXT0_SSRX0_N"
 		(at 349.25 38.1 0)
+		(fields_autoplaced yes)
 		(effects
 			(font
@@
 	(label "HDMI_D1P"
 		(at 344.17 184.15 0)
+		(fields_autoplaced yes)
 		(effects
 			(font
@@
 	(label "USB_EXT0_SSRX1_N"
 		(at 349.25 45.72 0)
+		(fields_autoplaced yes)
 		(effects
 			(font
@@
 	(label "HDMI_D1N"
 		(at 344.17 186.69 0)
+		(fields_autoplaced yes)
 		(effects
 			(font
@@
 	(label "HDMI_D0N"
 		(at 344.17 191.77 0)
-		(effects
-			(font
+		(fields_autoplaced yes)
+		(effects
+			(font

Commit message: 20250509-1
Parts:
- added C? (x3): 2.2uF, symbol Device:C_Small
- added C? (x2): 10uF, symbol Device:C_Small
- added C? (x2): 1uF, symbol Device:C_Small
- added C?: 1nF, symbol Device:C_Small
- added C?: 22pF, symbol Device:C_Small
- added R? (x2): 22, symbol Device:R_Small
- added R?: 2.49K, symbol Device:R_Small
- added R?: 10K, symbol Device:R_Small
- added U?: 92HD95, Package_DFN_QFN:QFN-40-1EP_5x5mm_P0.4mm_EP3.6x3.6mm, symbol mediacow:92HD95
Connections:
- net GND: now also C?.2, C?.2, C?.2, C?.2, C?.2, C?.2, C?.2, C?.2, U?.34 (PVSS), U?.35 (PVSS)
- new net: C?.1, U?.26 (VNeg)
- new net: R?.2, U?.5 (SDATA_OUT)
- new net: C?.1, R?.2
- new net: C?.1, U?.1 (DVDD_CORE)
- new net: C?.1, U?.21 (CAP2)
- new net: C?.1, U?.25 (VPos)
- new net: C?.1, U?.20 (VrefFilt)
- new net: C?.1, U?.29 (CPVreg)
- new net: C?.1, U?.28 (FCap1)
- new net: C?.2, U?.27 (FCap2)
- new net AC_AVDD: R?.1
- new net AC_DMIC_CLK: U?.2 (DMIC_CLK/GPIO_1)
- new net AC_DMIC_D0: U?.3 (DMIC_0/GPIO_2)
- new net AC_DMIC_D1: U?.4 (DMIC_1/GPIO_0)
- new net AC_EAPD: R?.2, U?.39 (EAPD)
- new net AC_PCBEEP: U?.12 (PC_Beep)
- new net AC_PORTA_L: U?.23 (PORTA_L)
- new net AC_PORTA_R: U?.24 (PORTA_R)
- new net AC_PORTB_L: U?.17 (PORTB_L)
- new net AC_PORTB_R: U?.18 (PORTB_R)
- new net AC_PORTB_VREF: U?.19 (VrefOut_B)
- new net AC_PORTC_L: U?.14 (PORTC_L)
- new net AC_PORTC_R: U?.15 (PORTC_R)
- new net AC_PORTC_VREF: U?.16 (VrefOut_C)
- new net AC_PORTD_LN: U?.33 (PORTD_-L)
- new net AC_PORTD_LP: U?.32 (PORTD_+L)
- new net AC_PORTD_RN: U?.36 (PORTD_-R)
- new net AC_PORTD_RP: U?.37 (PORTD_+R)
- new net AC_SENSE_A: C?.1, R?.2, U?.13 (SENSE_A)
- new net SOM_HDA_BCLK: R?.1, U?.6 (BITCLK)
- new net SOM_HDA_RST: U?.11 (RESET#)
- new net SOM_HDA_SDIN: R?.1
- new net SOM_HDA_SDOUT: U?.8 (SDATA_IN)
- new net SOM_HDA_SYNC: U?.10 (SYNC)
Other:
- note added: "Audio CODEC"
- note added: "External USB"
- note removed: "2025-03-23 - 2025-04-29"
- note removed: "MediaCow Touch 2 Lite "Curitiba" - CTCL 2021-2025"
- note removed: "MediaCow Touch 2 Lite - IO"
- company: (none) -> CTCL 2021-2025
- title: (none) -> MediaCow Touch 2 Lite "Curitiba" - IO
- moved on the sheet: C?, J?, R?, TP?, U?
