File: lite/circuits/mct2_lite/mct2_lite_io.kicad_sch (KiCad schematic)
At the start: 42 parts

Commit message: 20250524-1
Parts:
- C? (x5): footprint (none) -> Capacitor_SMD:C_0805_2012Metric
- C? (x13): footprint (none) -> Capacitor_SMD:C_0603_1608Metric
- C? (x2): footprint (none) -> Capacitor_SMD:C_1206_3216Metric
- J?: footprint (none) -> Connector_Video:HDMI_A_Molex_208658-1001_Horizontal
- J? (x2): footprint (none) -> Connector_USB:USB3_A_Molex_48393-001
- R? (x12): footprint (none) -> Resistor_SMD:R_0603_1608Metric
- TP?: footprint (none) -> TestPoint:TestPoint_Pad_2.0x2.0mm
- U?: footprint RKT24 -> Package_SO:TSSOP-24_4.4x7.8mm_P0.65mm
Changed lines of the file:
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@@
 	(title_block
 		(title "MediaCow Touch 2 Lite \"Curitiba\" - IO")
-		(date "2025-03-23 - 2025-05-09")
+		(date "2025-03-23 - 2025-05-24")
 		(company "CTCL 2021-2025")
 	)
@@
 			)
 		)
-		(property "Footprint" ""
+		(property "Footprint" "Resistor_SMD:R_0603_1608Metric"
 			(at 445.77 198.12 0)
 			(effects
@@
 			)
 		)
-		(property "Footprint" ""
+		(property "Footprint" "Connector_Video:HDMI_A_Molex_208658-1001_Horizontal"
 			(at 559.435 328.93 0)
 			(effects
@@
 			)
 		)
-		(property "Datasheet" "https://en.wikipedia.org/wiki/HDMI"
+		(property "Datasheet" ""
 			(at 559.435 328.93 0)
 			(effects
@@
 			)
 		)
-		(property "Footprint" ""
+		(property "Footprint" "Capacitor_SMD:C_0805_2012Metric"
 			(at 547.37 157.48 0)
 			(effects
@@
 			)
 		)
-		(property "Footprint" ""
+		(property "Footprint" "Resistor_SMD:R_0603_1608Metric"
 			(at 511.81 203.2 0)
 			(effects
@@
 			)
 		)
-		(property "Footprint" ""
+		(property "Footprint" "Resistor_SMD:R_0603_1608Metric"
 			(at 417.83 248.92 0)
 			(effects
@@
 			)
 		)
-		(property "Footprint" ""
+		(property "Footprint" "Resistor_SMD:R_0603_1608Metric"
 			(at 504.19 246.38 0)
 			(effects
@@
 			)
 		)
-		(property "Footprint" ""
+		(property "Footprint" "Resistor_SMD:R_0603_1608Metric"
 			(at 430.53 127 0)
 			(effects
@@
 			)
 		)
-		(property "Footprint" ""
+		(property "Footprint" "Resistor_SMD:R_0603_1608Metric"
 			(at 407.67 143.51 0)
 			(effects
@@
 			)
 		)
-		(property "Footprint" ""
+		(property "Footprint" "Capacitor_SMD:C_0603_1608Metric"
 			(at 504.19 261.62 0)
 			(effects
@@
 			)
 		)
-		(property "Footprint" ""
+		(property "Footprint" "Resistor_SMD:R_0603_1608Metric"
 			(at 421.64 133.35 0)
 			(effects
@@
 			)
 		)
-		(property "Footprint" ""
+		(property "Footprint" "Resistor_SMD:R_0603_1608Metric"
 			(at 502.92 200.66 0)
 			(effects
@@
 			)
 		)
-		(property "Footprint" ""
+		(property "Footprint" "Capacitor_SMD:C_0603_1608Metric"
 			(at 502.92 208.28 0)
 			(effects
@@
 			)
 		)
-		(property "Footprint" ""
+		(property "Footprint" "Capacitor_SMD:C_0603_1608Metric"
 			(at 511.81 218.44 0)
 			(effects
@@
 			)
 		)
-		(property "Footprint" ""
+		(property "Footprint" "Capacitor_SMD:C_1206_3216Metric"
 			(at 443.23 119.38 0)
 			(effects
@@
 			)
 		)
-		(property "Footprint" ""
+		(property "Footprint" "Connector_USB:USB3_A_Molex_48393-001"
 			(at 552.45 248.92 0)
 			(effects
@@
 			)
 		)
-		(property "Footprint" ""
+		(property "Footprint" "Resistor_SMD:R_0603_1608Metric"
 			(at 445.77 243.84 0)
 			(effects
@@
 			)
 		)
-		(property "Footprint" ""
+		(property "Footprint" "Capacitor_SMD:C_0603_1608Metric"
 			(at 513.08 264.16 0)
 			(effects
@@
 			)
 		)
-		(property "Footprint" ""
+		(property "Footprint" "Resistor_SMD:R_0603_1608Metric"
 			(at 513.08 248.92 0)
 			(effects
@@
 			)
 		)
-		(property "Footprint" ""
+		(property "Footprint" "Capacitor_SMD:C_0603_1608Metric"
 			(at 396.24 200.66 0)
 			(effects
@@
 			)
 		)
-		(property "Footprint" ""
+		(property "Footprint" "Capacitor_SMD:C_0805_2012Metric"
 			(at 513.08 170.18 0)
 			(effects
@@
 			)
 		)
-		(property "Footprint" ""
+		(property "Footprint" "Connector_USB:USB3_A_Molex_48393-001"
 			(at 551.18 203.2 0)
 			(effects
@@
 			)
 		)
-		(property "Footprint" ""
+		(property "Footprint" "Capacitor_SMD:C_0603_1608Metric"
 			(at 504.19 254 0)
 			(effects
@@
 			)
 		)
-		(property "Footprint" ""
+		(property "Footprint" "Capacitor_SMD:C_0603_1608Metric"
 			(at 502.92 215.9 0)
 			(effects
@@
 			)
 		)
-		(property "Footprint" ""
+		(property "Footprint" "Resistor_SMD:R_0603_1608Metric"
 			(at 516.89 114.3 0)
 			(effects
@@
 			)
 		)
-		(property "Footprint" ""
+		(property "Footprint" "Capacitor_SMD:C_0603_1608Metric"
 			(at 513.08 256.54 0)
 			(effects
@@
 			)
 		)
-		(property "Footprint" ""
+		(property "Footprint" "Capacitor_SMD:C_0603_1608Metric"
 			(at 407.67 151.13 0)
 			(effects
@@
 			)
 		)
-		(property "Footprint" ""
+		(property "Footprint" "Capacitor_SMD:C_0805_2012Metric"
 			(at 541.02 157.48 0)
 			(effects
@@
 			)
 		)
-		(property "Footprint" ""
+		(property "Footprint" "Capacitor_SMD:C_0805_2012Metric"
 			(at 467.36 170.18 0)
 			(effects
@@
 			)
 		)
-		(property "Footprint" ""
+		(property "Footprint" "Capacitor_SMD:C_0603_1608Metric"
 			(at 421.64 138.43 0)
 			(effects
@@
 			)
 		)
-		(property "Footprint" "RKT24"
+		(property "Footprint" "Package_SO:TSSOP-24_4.4x7.8mm_P0.65mm"
 			(at 496.57 323.85 0)
 			(effects
@@
 			)
 		)
-		(property "Datasheet" "TPD12S016RKTR"
+		(property "Datasheet" "https://www.ti.com/lit/ds/symlink/tpd12s016.pdf"
 			(at 496.57 323.85 0)
 			(effects
@@
 			)
 		)
-		(property "Footprint" ""
+		(property "Footprint" "Resistor_SMD:R_0603_1608Metric"
 			(at 417.83 203.2 0)
 			(effects
@@
 			)
 		)
-		(property "Footprint" ""
+		(property "Footprint" "Capacitor_SMD:C_0603_1608Metric"
 			(at 537.21 300.99 0)
 			(effects
@@
 			)
 		)
-		(property "Footprint" ""
+		(property "Footprint" "Capacitor_SMD:C_1206_3216Metric"
 			(at 553.72 157.48 0)
 			(effects
@@
 			)
 		)
-		(property "Footprint" ""
+		(property "Footprint" "Capacitor_SMD:C_0805_2012Metric"
 			(at 525.78 148.59 0)
 			(effects
@@
 			)
 		)
-		(property "Footprint" ""
+		(property "Footprint" "Capacitor_SMD:C_0603_1608Metric"
 			(at 396.24 246.38 0)
 			(effects
@@
 			)
 		)
-		(property "Footprint" ""
+		(property "Footprint" "TestPoint:TestPoint_Pad_2.0x2.0mm"
 			(at 534.67 339.09 0)
 			(effects
@@
 			)
 		)
-		(property "Footprint" ""
+		(property "Footprint" "Capacitor_SMD:C_0603_1608Metric"
 			(at 511.81 210.82 0)
 			(effects

Commit message: 20250529-1
Parts:
- removed C?: 120uF, symbol Device:C_Small
- removed C?: 100nF, Capacitor_SMD:C_0603_1608Metric, symbol Device:C_Small
- removed R?: 56K, Resistor_SMD:R_0603_1608Metric, symbol Device:R_Small
- removed R?: 20K, Resistor_SMD:R_0603_1608Metric, symbol Device:R_Small
- removed U?: TPS25221, Package_SON:WSON-6-1EP_2x2mm_P0.65mm_EP1x1.6mm, symbol mediacow:TPS25221
- added C147: 100nF, Capacitor_SMD:C_0603_1608Metric, symbol Device:C_Small
- added C152, C154, C155, C156, C157, C158, C159, C160, C161, C163, C164: 22uF, Capacitor_SMD:C_1206_3216Metric, symbol Device:C_Small
- added C165, C166: 10nF, symbol Device:C_Small
- added C? (x4): 2.2nF, symbol Device:C_Small
- added J7: AudioJack3_SwitchTR, symbol Connector_Audio:AudioJack3_SwitchTR
- added J?: Adafruit 1669 or equivalent, Connector_JST:JST_PH_S4B-PH-K_1x04_P2.00mm_Horizontal, symbol Connector:Conn_01x04_Socket
- added L7, L8: 600@500mA, symbol Device:L_Ferrite_Small
- added Q14: 2N7002, Package_TO_SOT_SMD:SOT-23, symbol Transistor_FET:2N7002
- added R74: 20K, Resistor_SMD:R_0603_1608Metric, symbol Device:R_Small
- added R77: 56K, Resistor_SMD:R_0603_1608Metric, symbol Device:R_Small
- added R80, R81: 5.1, Resistor_SMD:R_0603_1608Metric, symbol Device:R_Small
- added R86: 100K, Resistor_SMD:R_0603_1608Metric, symbol Device:R_Small
- added R88: 39.2K, Resistor_SMD:R_0603_1608Metric, symbol Device:R_Small
- added R? (x4): 3.3, symbol Device:R_Small
- added U20: TPS25221, Package_SON:WSON-6-1EP_2x2mm_P0.65mm_EP1x1.6mm, symbol mediacow:TPS25221
- added U22, U23: TPD2E2U06DCK, Package_TO_SOT_SMD:SOT-323_SC-70, symbol Power_Protection:TPD2E2U06DCK
- added U26, U27: TPD4EUSB30, Package_SON:USON-10_2.5x1.0mm_P0.5mm, symbol mediacow:TPD4EUSB30
- C153: renamed from C?; value 120uF -> 22uF; footprint (none) -> Capacitor_SMD:C_1206_3216Metric
- gave numbers to parts that had none: 36
Connections:
- net AC_AVDD: now also R86.1
- net AC_PORTA_L: now also R81.1
- net AC_PORTA_R: now also R80.1
- net AC_PORTD_LN: now also C?.2, J?.4 (Pin_4)
- net AC_PORTD_LP: now also C?.1, J?.3 (Pin_3)
- net AC_PORTD_RN: now also C?.2, J?.2 (Pin_2)
- net AC_PORTD_RP: now also C?.1, J?.1 (Pin_1)
- net AC_SENSE_A: now also R88.1
- net GND: now also C147.2, C152.2, C154.2, C155.2, C156.2, C157.2, C158.2, C159.2, C160.2, C161.2, C163.2, C164.2, C165.2, C166.2, Q14.2 (S), R74.2, R77.2, R?.2, R?.2, R?.2, R?.2, U20.2 (GND), U22.3, U23.3, U26.3 (GND), U26.7 (NC), U26.8 (GND), U27.3 (GND), U27.7 (NC), U27.8 (GND)
- net USB_5V: now also C147.1, U20.1 (IN)
- net USB_EXT0_SSRX0_N: now also U26.2 (D1-)
- net USB_EXT0_SSRX0_P: now also U26.1 (D1+)
- net USB_EXT0_SSRX1_N: now also U26.4 (D2-)
- net USB_EXT0_SSRX1_P: now also U26.3 (GND)
- net USB_EXT0_USB2_N: now also U22.1
- net USB_EXT0_USB2_P: now also U22.2
- net USB_EXT1_EN: now also R74.1, U20.3 (EN)
- net USB_EXT1_FLT: now also U20.4 (FAULT)
- net USB_EXT1_SSRX0_N: now also U27.2 (D1-)
- net USB_EXT1_SSRX0_P: now also U27.1 (D1+)
- net USB_EXT1_SSRX1_N: now also U27.4 (D2-)
- net USB_EXT1_SSRX1_P: now also U27.3 (GND)
- net USB_EXT1_USB2_N: now also U23.1
- net USB_EXT1_USB2_P: now also U23.2
- net USB_EXT1_VBUS: now reaches C153.1, J9.1 (VBUS), U21.6 (OUT)
- net USB_EXT1_VBUS: now also C152.1, C154.1, C155.1, C156.1, C157.1, C158.1, C159.1, C160.1, C161.1, C163.1, C164.1, U20.6 (OUT)
- net USB_EXT0_VBUS: now reaches J8.1 (VBUS)
- net AC_DVDD: now reaches R87.1
- new net: C?.2, R?.1 (x2)
- new net: L7.1, R80.2
- new net: J7.RN, Q14.1 (G), R86.2
- new net: C?.1, R?.1 (x2)
- new net: Q14.3 (D), R88.2
- new net: C166.1, J7.R, L7.2
- new net: C165.1, J7.T, L8.2
- new net: L8.1, R81.2
- new net: R77.1, U20.5 (ILIM)
Other:
- note added: "Headphone Output"
- note added: "Internal Speaker Header"
- note added: "Snubber circuit components must be placed close to CODEC"
- moved on the sheet: C148, C149, C150, C151, C153, C162, C167, C168, C169, C170, C171, C172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
