File: lite/circuits/mct2_lite/mct2_lite_io.kicad_sch (KiCad schematic)
At the start: 75 parts, among them J10 HDMI_A, J7 AudioJack3_SwitchTR, J8 USB3_A, J9 USB3_A, Q14 2N7002, U20 TPS25221, U21 TPS25221, U22 TPD2E2U06DCK, U23 TPD2E2U06DCK, U24 92HD95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

Commit message: 20250610-1
Parts:
- C? (x4): footprint (none) -> Capacitor_SMD:C_0603_1608Metric
Changed lines of the file:
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@@
 	(wire
 		(pts
-			(xy 494.03 137.16) (xy 496.57 137.16)
+			(xy 492.76 137.16) (xy 496.57 137.16)
 		)
 		(stroke
@@
 	(wire
 		(pts
-			(xy 494.03 132.08) (xy 496.57 132.08)
+			(xy 492.76 132.08) (xy 496.57 132.08)
 		)
 		(stroke
@@
 	(global_label "AC_PORTA_L"
 		(shape input)
-		(at 494.03 137.16 180)
+		(at 492.76 137.16 180)
 		(fields_autoplaced yes)
 		(effects
@@
 		)
 		(property "Intersheetrefs" "${INTERSHEET_REFS}"
-			(at 479.7962 137.16 0)
+			(at 478.5262 137.16 0)
 			(effects
 				(font
@@
 	(global_label "AC_PORTA_R"
 		(shape input)
-		(at 494.03 132.08 180)
+		(at 492.76 132.08 180)
 		(fields_autoplaced yes)
 		(effects
@@
 		)
 		(property "Intersheetrefs" "${INTERSHEET_REFS}"
-			(at 479.5543 132.08 0)
+			(at 478.2843 132.08 0)
 			(effects
 				(font
@@
 			)
 		)
-		(property "Footprint" ""
+		(property "Footprint" "Capacitor_SMD:C_0603_1608Metric"
 			(at 410.21 149.86 0)
 			(effects
@@
 		(dnp no)
 		(property "Reference" "R80"
-			(at 495.808 131.064 90)
+			(at 494.792 131.064 90)
 			(effects
 				(font
@@
 		(on_board yes)
 		(dnp no)
-		(fields_autoplaced yes)
 		(property "Reference" "R86"
-			(at 544.83 148.5899 0)
+			(at 543.306 148.59 0)
 			(effects
 				(font
@@
 		)
 		(property "Value" "100K"
-			(at 544.83 151.1299 0)
+			(at 543.306 151.13 0)
 			(effects
 				(font
@@
 			)
 		)
-		(property "Footprint" ""
+		(property "Footprint" "Capacitor_SMD:C_0603_1608Metric"
 			(at 410.21 137.16 0)
 			(effects
@@
 			)
 		)
-		(property "Footprint" ""
+		(property "Footprint" "Capacitor_SMD:C_0603_1608Metric"
 			(at 410.21 165.1 0)
 			(effects
@@
 		(dnp no)
 		(property "Reference" "R81"
-			(at 495.808 136.144 90)
+			(at 494.792 136.144 90)
 			(effects
 				(font
@@
 			)
 		)
-		(property "Footprint" ""
+		(property "Footprint" "Capacitor_SMD:C_0603_1608Metric"
 			(at 410.21 121.92 0)
 			(effects
