File: lite/circuits/mct2_lite/mct2_lite.kicad_sch (KiCad schematic)
At the start: 10 parts

Commit message: 20250509-1
Parts:
- A?: footprint Module_LattePanda:LattePanda_Module_H8.0mm_Horizontal -> LattePanda Mu:LattePanda_Module_H4.0mm_Horizontal
- J?: footprint (none) -> Package_SO:SOIC-8W_5.3x5.3mm_P1.27mm
- J?: footprint (none) -> Connector_PinHeader_2.54mm:PinHeader_2x05_P2.54mm_Vertical
Other:
- note removed: "2025-03-23 - 2025-04-29"
- note removed: "MediaCow Touch 2 Lite "Curitiba" - CTCL 2021-2025"
- note removed: "MediaCow Touch 2 Lite - Root"
- company: (none) -> CTCL 2021-2025
- title: (none) -> MediaCow Touch 2 Lite "Curitiba"
Changed lines of the file:
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@@
 	(generator_version "8.0")
 	(paper "A2")
+	(title_block
+		(title "MediaCow Touch 2 Lite \"Curitiba\"")
+		(date "2025-03-23 - 2025-05-09")
+		(company "CTCL 2021-2025")
+	)
 	(no_connect
 		(at 303.53 223.52)
@@
 		)
 	)
-	(text "2025-03-23 - 2025-04-29"
-		(exclude_from_sim no)
-		(at 517.906 403.352 0)
-		(effects
-			(font
-				(size 1.27 1.27)
-			)
-		)
-	)
-	(text "MediaCow Touch 2 Lite \"Curitiba\" - CTCL 2021-2025"
-		(exclude_from_sim no)
-		(at 501.904 390.144 0)
-		(effects
-			(font
-				(size 1.27 1.27)
-			)
-		)
-	)
-	(text "MediaCow Touch 2 Lite - Root"
-		(exclude_from_sim no)
-		(at 498.094 400.05 0)
-		(effects
-			(font
-				(size 1.27 1.27)
-			)
-		)
-	)
 	(global_label "HDMI_TX1_N"
 		(shape input)
@@
 			)
 		)
-		(property "Footprint" "Module_LattePanda:LattePanda_Module_H8.0mm_Horizontal"
+		(property "Footprint" "LattePanda Mu:LattePanda_Module_H4.0mm_Horizontal"
 			(at 173.99 166.37 0)
 			(effects
@@
 			)
 		)
-		(property "Footprint" ""
+		(property "Footprint" "Package_SO:SOIC-8W_5.3x5.3mm_P1.27mm"
 			(at 295.91 240.03 0)
 			(effects
@@
 			)
 		)
-		(property "Footprint" ""
+		(property "Footprint" "Connector_PinHeader_2.54mm:PinHeader_2x05_P2.54mm_Vertical"
 			(at 295.91 220.98 0)
 			(effects

Commit message: 20250524-1
Parts:
- added J?: Bus_M.2_Socket_E, symbol Connector:Bus_M.2_Socket_E
- BT?: footprint (none) -> Battery:BatteryHolder_Keystone_1057_1x2032
- TP? (x6): footprint (none) -> TestPoint:TestPoint_Pad_2.0x2.0mm
Connections:
- net GND: now also J?.1 (GND), J?.18 (GND), J?.33 (GND), J?.39 (GND), J?.45 (GND), J?.51 (GND), J?.57 (GND), J?.63 (GND), J?.69 (GND), J?.7 (GND), J?.75 (GND)
- net SOM_SUSCLK: now also J?.50 (SUSCLK)
- net SOM_I2C5_SCL: now reaches A?.142 (I2C5_SCL)
- net SOM_I2C5_SDA: now reaches A?.144 (I2C5_SDA)
- net SOM_I2C4_SCL: now reaches A?.146 (I2C4_SCL)
- net SOM_I2C4_SDA: now reaches A?.148 (I2C4_SDA)
- net SOM_I2C3_SCL: now reaches A?.150 (I2C3_SCL)
- net SOM_I2C3_SCL: now also J?.60 (I2C_CLK)
- net SOM_I2C3_SDA: now reaches A?.152 (I2C3_SDA)
- net SOM_I2C3_SDA: now also J?.58 (I2C_DATA)
- net TCP1_HPD: now reaches A?.185 (TCP1_HPD)
- net TCP0_HPD: now reaches A?.187 (TCP0_HPD)
- new net: J?.2 (3.3V), J?.4 (3.3V), J?.72 (3.3V), J?.74 (3.3V)
- new net M2E_COEX1: J?.48 (COEX1)
- new net M2E_COEX2: J?.46 (COEX2)
- new net M2E_COEX3: J?.44 (COEX3)
- new net M2E_I2C_ALT: J?.62 (~{ALERT})
- new net M2E_SDIO_CLK: J?.9 (SDIO_CLK)
- new net M2E_SDIO_CMD: J?.11 (SDIO_CMD)
- new net M2E_SDIO_DATA0: J?.13 (SDIO_DATA0)
- new net M2E_SDIO_DATA1: J?.15 (SDIO_DATA1)
- new net M2E_SDIO_DATA2: J?.17 (SDIO_DATA2)
- new net M2E_SDIO_DATA3: J?.19 (SDIO_DATA3)
- new net M2E_SDIO_RST: J?.23 (~{SDIO_RESET})
- new net M2E_SDIO_WAKE: J?.21 (~{SDIO_WAKE})
- new net M2E_USB_DN: J?.5 (USB_D-)
- new net M2E_USB_DP: J?.3 (USB_D+)
- new net M2E_VD1: J?.38 (VENDOR_DEFINED)
- new net M2E_VD2: J?.40 (VENDOR_DEFINED)
- new net M2E_VD3: J?.42 (VENDOR_DEFINED)
- new net M2E_WDISABLE1: J?.56 (~{W_DISABLE1})
- new net M2E_WDISABLE2: J?.54 (~{W_DISABLE2})
- no-connect marks 7 -> 5

Commit message: 20250529-1
Parts:
- added C1, C2, C35, C36, C37, C38: 100nF, Capacitor_SMD:C_0603_1608Metric, symbol Device:C_Small
- added C10, C11, C12, C13, C14, C17, C18, C21, C22, C23, C24, C25, C26, C27, C28, C31, C32, C7, C8, C9: 100nF, Capacitor_SMD:C_0402_1005Metric, symbol Device:C_Small
- added C15, C16, C19, C20, C29, C30, C33, C34, C5, C6: 10uF, Capacitor_SMD:C_1206_3216Metric, symbol Device:C_Small
- added C3, C4: 100pF, symbol Device:C_Small
- added J4: Bus_M.2_Socket_M, mediacow:TE_1-2199230-5, symbol Connector:Bus_M.2_Socket_M
- added L1, L2: 6.8uH, Inductor_SMD:L_Chilisin_BMRF00101040, symbol Device:L_Small
- added R1, R3: 182K, Resistor_SMD:R_0603_1608Metric, symbol Device:R_Small
- added R2, R4: 62K, Resistor_SMD:R_0603_1608Metric, symbol Device:R_Small
- added R5: 1K, Resistor_SMD:R_0603_1608Metric, symbol Device:R_Small
- added U1, U2: AP63200WU, Package_TO_SOT_SMD:TSOT-23-6, symbol Regulator_Switching:AP63200WU
- J3: renamed from J?; footprint (none) -> mediacow:TE_21992304
- gave numbers to parts that had none: 10
Connections:
- net GND: now also C15.2, C16.2, C19.2, C20.2, C29.2, C30.2, C33.2, C34.2, C35.2, C36.2, C37.2, C38.2, C5.2, C6.2, J4.1 (GND), J4.15 (GND), J4.21 (GND), J4.27 (GND), J4.3 (GND), J4.33 (GND), J4.39 (GND), J4.45 (GND), J4.51 (GND), J4.57 (GND), J4.71 (GND), J4.73 (GND), J4.75 (GND), J4.9 (GND), R2.2, R4.2, R5.1, U1.4 (GND), U2.4 (GND)
- net SOM_HSIO10_RX_N: now also C11.2
- net SOM_HSIO10_RX_P: now also C25.2
- net SOM_HSIO10_TX_N: now also C12.2
- net SOM_HSIO10_TX_P: now also C26.2
- net SOM_HSIO11_RX_N: now also C13.2
- net SOM_HSIO11_RX_P: now also C27.2
- net SOM_HSIO11_TX_N: now also C14.2
- net SOM_HSIO11_TX_P: now also C28.2
- net SOM_HSIO6_RX_N: now also C17.2
- net SOM_HSIO6_RX_P: now also C31.2
- net SOM_HSIO6_TX_N: now also C18.2
- net SOM_HSIO6_TX_P: now also C32.2
- net SOM_HSIO8_RX_N: now also C7.2
- net SOM_HSIO8_RX_P: now also C21.2
- net SOM_HSIO8_TX_N: now also C8.2
- net SOM_HSIO8_TX_P: now also C22.2
- net SOM_HSIO9_RX_N: now also C9.2
- net SOM_HSIO9_RX_P: now also C23.2
- net SOM_HSIO9_TX_N: now also C10.2
- net SOM_HSIO9_TX_P: now also C24.2
- net SOM_PCIE_REF3_N: now also J3.49 (REFCLKn0)
- net SOM_PCIE_REF3_P: now also J3.47 (REFCLKp0)
- net SOM_PCIE_REF4_N: now also J4.53 (REFCLKn)
- net SOM_PCIE_REF4_P: now also J4.55 (REFCLKp)
- net SOM_SUSCLK: now also J4.68 (SUSCLK)
- net SOM_VSYS: now also U1.2 (EN), U1.3 (IN), U2.2 (EN), U2.3 (IN)
- net M2E_I2S_WS: now reaches J3.10 (PCM_SYNC/I2S_WS)
- net M2E_I2S_SDIN: now reaches J3.12 (PCM_IN/I2S_SD_IN)
- net M2E_I2S_SDOUT: now reaches J3.14 (PCM_OUT/I2S_SD_OUT)
- net M2E_LED2: now reaches J3.16 (~{LED_2})
- net at J3.2 (3.3V), J3.4 (3.3V), J3.72 (3.3V)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: now also C15.1, C19.1, C29.1, C3.1, C33.1, C35.1, C37.1, C5.1, L1.2, R1.1
- net M2E_UART_WAKE: now reaches J3.20 (~{UART_WAKE})
- net M2E_UART_RX: now reaches J3.22 (UART_RXD)
- net M2E_UART_TX: now reaches J3.32 (UART_TXD)
- net M2E_UART_CTS: now reaches J3.34 (UART_CTS)
- net M2E_PCIE_RX_P: now reaches J3.35 (PETp0)
- net M2E_PCIE_RX_P: now also C31.1
- net M2E_UART_RTS: now reaches J3.36 (UART_RTS)
- net M2E_PCIE_RX_N: now reaches J3.37 (PETn0)
- net M2E_PCIE_RX_N: now also C17.1
- net M2E_PCIE_TX_P: now reaches J3.41 (PERp0)
- net M2E_PCIE_TX_P: now also C32.1
- net M2E_PCIE_TX_N: now reaches J3.43 (PERn0)
- net M2E_PCIE_TX_N: now also C18.1
- net M2E_PCIE_RST: now reaches J3.52 (~{PERST0})
- net M2E_PCIE_CLKREQ: now reaches J3.53 (~{CLKREQ0})
- net M2E_PCIE_WAKE: now reaches J3.55 (~{PEWAKE0})
- net M2E_LED1: now reaches J3.6 (~{LED_1})
- net M2E_UIM_SWP: now reaches J3.66 (UIM_SWP/~{PERST1})
- net M2E_POWER_SNK: now reaches J3.68 (UIM_POWER_SNK/~{CLKREQ1})
- net M2E_POWER_SRC: now reaches J3.70 (UIM_POWER_SRC/GPIO1/~{PEWAKE1})
- net M2E_I2S_CLK: now reaches J3.8 (PCM_CLK/I2S_SCK)
- new net: J4.69 (PEDET), R5.2
- new net: C4.2, R3.2, R4.1, U2.1 (FB)
- new net: C2.1, U2.5 (SW)
- new net: C2.2, L2.1, U2.6 (BST)
- new net: C16.1, C20.1, C30.1, C34.1, C36.1, C38.1, C4.1, C6.1, J4.12 (3.3V), J4.14 (3.3V), J4.16 (3.3V), J4.18 (3.3V), J4.2 (3.3V), J4.4 (3.3V), J4.70 (3.3V), J4.72 (3.3V), J4.74 (3.3V), L2.2, R3.1
- new net: C3.2, R1.2, R2.1, U1.1 (FB)
- new net: C1.1, U1.5 (SW)
- new net: C1.2, L1.1, U1.6 (BST)
- new net M2M_DEVSLP: J4.38 (DEVSLP)
- new net M2M_PCIE0_RX_N: C7.1, J4.47 (PETn0/SATA-A-)
- new net M2M_PCIE0_RX_P: C21.1, J4.49 (PETp0/SATA-A+)
- new net M2M_PCIE0_TX_N: C8.1, J4.41 (PERn0/SATA-B+)
- new net M2M_PCIE0_TX_P: C22.1, J4.43 (PERp0/SATA-B-)
- new net M2M_PCIE1_RX_N: C9.1, J4.35 (PETn1)
- new net M2M_PCIE1_RX_P: C23.1, J4.37 (PETp1)
- new net M2M_PCIE1_TX_N: C10.1, J4.29 (PERn1)
- new net M2M_PCIE1_TX_P: C24.1, J4.31 (PERp1)
- new net M2M_PCIE2_RX_N: C11.1, J4.23 (PETn2)
- new net M2M_PCIE2_RX_P: C25.1, J4.25 (PETp2)
- new net M2M_PCIE2_TX_N: C12.1, J4.17 (PERn2)
- new net M2M_PCIE2_TX_P: C26.1, J4.19 (PERp2)
- new net M2M_PCIE3_RX_N: C13.1, J4.11 (PETn3)
- new net M2M_PCIE3_RX_P: C27.1, J4.13 (PETp3)
- new net M2M_PCIE3_TX_N: C14.1, J4.5 (PERn3)
- new net M2M_PCIE3_TX_P: C28.1, J4.7 (PERp3)
- new net M2M_PCIE_CLKREQ: J4.52 (~{CLKREQ})
- new net M2M_PCIE_RST: J4.50 (~{PERST})
- new net M2M_PCIE_WAKE: J4.54 (~{PEWAKE})
- no-connect marks 5 -> 12
