File: lite/circuits/mct2_lite/mct2_lite.kicad_sch (KiCad schematic)
At the start: 59 parts, among them J1 TPM, J2 External BIOS, J3 Bus_M.2_Socket_E, J4 Bus_M.2_Socket_M, U1 AP63200WU, U2 AP63200WU

Commit message: 20250628-1
Parts:
- removed TP5, TP6: TestPoint_Alt, TestPoint:TestPoint_Pad_2.0x2.0mm, symbol Connector:TestPoint_Alt
- added J11: Conn_01x04_Socket, symbol Connector:Conn_01x04_Socket
- added TP10, TP11, TP8, TP9: TestPoint_Alt, TestPoint:TestPoint_Pad_2.0x2.0mm, symbol Connector:TestPoint_Alt
Connections:
- net GND: now also J11.4 (Pin_4)
- net SOM_SIO_UART_RX: now also J11.3 (Pin_3)
- net SOM_SIO_UART_TX: now also J11.2 (Pin_2)
- net TCP1_DDC_SDA: now reaches A1.173 (TCP1_DDC_SDA)
- net TCP1_DDC_SDA: now also TP10.1
- net TCP1_DDC_SCL: now reaches A1.175 (TCP1_DDC_SCL)
- net TCP1_DDC_SCL: now also TP11.1
- net TCP0_DDC_SDA: now reaches A1.177 (TCP0_DDC_SDA)
- net TCP0_DDC_SDA: now also TP8.1
- net TCP0_DDC_SCL: now reaches A1.179 (TCP0_DDC_SCL)
- net TCP0_DDC_SCL: now also TP9.1
- no-connect marks 12 -> 8
Other:
- moved on the sheet: TP1, TP2, TP3, TP4
